File: Hardware/Temp/PFC/PFC.kicad_sch (KiCad schematic)
At the start: 36 parts, among them J1 HB9500M-9.5-3P, J2 Terminal, M1 600V 9.5A, U1 UCC28180D

Commit message: update PFC
Parts:
- removed R10: 18K_1/4W_5%, charge_battery_footprint_lib:Res_18K_1_4W_1, symbol charge_battery_sym_lib:Res_hole_18K_1/4W_5%
- added R11: 16.9K/1%/1_8W, Resistor_SMD:R_0805_2012Metric, symbol charge_battery_sym_lib:Res_10K_0603_1%
- C11: value 1uF 50V -> 4.7uF 50V; footprint charge_battery_footprint_lib:Ceramic_Cap_Hole_1uF_50V -> Resistor_SMD:R_1206_3216Metric; Supply URL https://www.thegioiic.com/tu-gom-multilayer-1uf-50v -> https://www.thegioiic.com/tu-gom-1206-4-7uf-50v; Supply part number Tụ Gốm Multilayer 1uF 50V -> Tụ Gốm 1206 4.7uF 50V
- C9: value 10uF 16V -> 680nF 50V 1206; footprint charge_battery_footprint_lib:Ceramic_Cap_10uF_16V -> Capacitor_SMD:C_1206_3216Metric; Supply URL https://www.thegioiic.com/tu-gom-0603-10uf-16v -> https://www.thegioiic.com/tu-gom-1206-680nf-50v; Supply part number Tụ Gốm 0603 10uF 16V -> Tụ Gốm 1206 680nF 50V
Connections:
- net at C9.2, U1.5 (VCOMP): now also R11.2
- net at C8.2: now also R11.1
Changed lines of the file:
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@@
 	(wire
 		(pts
+			(xy 139.7 146.05) (xy 139.7 149.86)
+		)
+		(stroke
+			(width 0)
+			(type default)
+		)
+	)
+	(wire
+		(pts
 			(xy 127 121.92) (xy 127 74.93)
 		)
@@
 	(wire
 		(pts
-			(xy 139.7 146.05) (xy 139.7 149.86)
-		)
-		(stroke
-			(width 0)
-			(type default)
-		)
-	)
-	(wire
-		(pts
 			(xy 148.59 146.05) (xy 148.59 127)
 		)
@@
 			)
 		)
-		(property "Value" "10uF 16V"
+		(property "Value" "680nF 50V 1206"
 			(at 151.892 151.1299 90)
 			(effects
@@
 			)
 		)
-		(property "Footprint" "charge_battery_footprint_lib:Ceramic_Cap_10uF_16V"
+		(property "Footprint" "Capacitor_SMD:C_1206_3216Metric"
 			(at 141.478 150.114 0)
 			(effects
@@
 			)
 		)
-		(property "Datasheet" "https://www.mouser.vn/datasheet/2/40/KYOCERA_AutoMLCCKAM-3106308.pdf"
+		(property "Datasheet" ""
 			(at 141.478 149.606 0)
 			(effects
@@
 			)
 		)
-		(property "Description" "10%, 0603 (1608 Metric)"
+		(property "Description" "10%, 1206 (3216 Metric)"
 			(at 140.97 148.844 0)
 			(effects
@@
 			)
 		)
-		(property "Supply part number" "Tụ Gốm 0603 10uF 16V"
+		(property "Supply part number" "Tụ Gốm 1206 680nF 50V"
 			(at 140.97 148.59 0)
 			(effects
@@
 			)
 		)
-		(property "Supply URL" "https://www.thegioiic.com/tu-gom-0603-10uf-16v"
+		(property "Supply URL" "https://www.thegioiic.com/tu-gom-1206-680nf-50v"
 			(at 141.478 149.86 0)
 			(effects
@@
 	)
 	(symbol
+		(lib_id "charge_battery_sym_lib:Res_10K_0603_1%")
+		(at 146.05 144.526 90)
+		(unit 1)
+		(exclude_from_sim no)
+		(in_bom yes)
+		(on_board yes)
+		(dnp no)
+		(fields_autoplaced yes)
+		(property "Reference" "R11"
+			(at 142.24 140.9699 90)
+			(effects
+				(font
+					(size 1.27 1.27)
+				)
+				(justify right)
+			)
+		)
+		(property "Value" "16.9K/1%/1_8W"
+			(at 142.24 143.5099 90)
+			(effects
+				(font
+					(size 1.27 1.27)
+				)
+				(justify right)
+			)
+		)
+		(property "Footprint" "Resistor_SMD:R_0805_2012Metric"
+			(at 134.62 104.648 90)
+			(effects
+				(font
+					(size 1.27 1.27)
+				)
+				(hide yes)
+			)
+		)
+		(property "Datasheet" ""
+			(at 145.288 104.902 90)
+			(effects
+				(font
+					(size 1.27 1.27)
+				)
+				(hide yes)
+			)
+		)
+		(property "Description" "Code 1692, 1/8W"
+			(at 139.192 104.14 90)
+			(effects
+				(font
+					(size 1.27 1.27)
+				)
+				(hide yes)
+			)
+		)
+		(property "Supply name" "Thegioiic"
+			(at 133.604 104.394 90)
+			(effects
+				(font
+					(size 1.27 1.27)
+				)
+				(hide yes)
+			)
+		)
+		(property "Supply part number" "Điện Trở 16.9 KOhm 0805 1%"
+			(at 132.588 104.648 90)
+			(effects
+				(font
+					(size 1.27 1.27)
+				)
+				(hide yes)
+			)
+		)
+		(property "Supply URL" "https://www.thegioiic.com/dien-tro-16-9-kohm-0805-1-"
+			(at 125.476 103.378 90)
+			(effects
+				(font
+					(size 1.27 1.27)
+				)
+				(hide yes)
+			)
+		)
+		(pin "1"
+		)
+		(pin "2"
+		)
+		(instances
+			(project "PFC"
+				(path "/3b17fecf-a6c4-4ae7-a684-61da545cc8d4"
+					(reference "R11")
+					(unit 1)
+				)
+			)
+		)
+	)
+	(symbol
 		(lib_name "R_Shunt_10mR_1")
 		(lib_id "charge_battery_sym_lib:R_Shunt_10mR")
@@
 			)
 		)
-		(property "Value" "1uF 50V"
+		(property "Value" "4.7uF 50V"
 			(at 202.438 113.0299 90)
 			(effects
@@
 			)
 		)
-		(property "Footprint" "charge_battery_footprint_lib:Ceramic_Cap_Hole_1uF_50V"
+		(property "Footprint" "Resistor_SMD:R_1206_3216Metric"
 			(at 192.278 112.014 0)
 			(effects
@@
 			)
 		)
-		(property "Description" "1uF ±10%, code 105"
+		(property "Description" "10%, 1206 (3216 Metric)"
 			(at 191.77 110.744 0)
 			(effects
@@
 			)
 		)
-		(property "Supply part number" "Tụ Gốm Multilayer 1uF 50V"
+		(property "Supply part number" "Tụ Gốm 1206 4.7uF 50V"
 			(at 191.77 110.49 0)
 			(effects
@@
 			)
 		)
-		(property "Supply URL" "https://www.thegioiic.com/tu-gom-multilayer-1uf-50v"
+		(property "Supply URL" "https://www.thegioiic.com/tu-gom-1206-4-7uf-50v"
 			(at 192.278 111.76 0)
 			(effects
@@
 					(unit 1)
 				)
-			)
-		)
-	)
-	(symbol
-		(lib_id "charge_battery_sym_lib:Res_hole_18K_1/4W_5%")
-		(at 138.43 143.51 90)
-		(unit 1)
-		(exclude_from_sim no)
-		(in_bom yes)
-		(on_board yes)
-		(dnp no)
-		(fields_autoplaced yes)
-		(property "Reference" "R10"
-			(at 141.478 140.9699 90)
-			(effects
-				(font
-					(size 1.27 1.27)
-				)
-				(justify right)
-			)
-		)
-		(property "Value" "18K_1/4W_5%"
-			(at 141.478 143.5099 90)
-			(effects
-				(font
-					(size 1.27 1.27)
-				)
-				(justify right)
-			)
-		)
-		(property "Footprint" "charge_battery_footprint_lib:Res_18K_1_4W_1"
-			(at 110.236 163.322 0)
-			(effects
-				(font
-					(size 1.27 1.27)
-				)
-				(hide yes)
-			)
-		)
-		(property "Datasheet" "~"
-			(at 110.744 160.782 90)
-			(effects
-				(font
-					(size 1.27 1.27)
-				)
-				(hide yes)
-			)
-		)
-		(property "Description" "Resistor"
-			(at 109.728 160.528 0)
-			(effects
-				(font
-					(size 1.27 1.27)
-				)
-				(hide yes)
-			)
-		)
-		(property "Supply name " "Thegioiic"
-			(at 109.728 153.416 0)
-			(effects
-				(font
-					(size 1.27 1.27)
-				)
-				(hide yes)
-			)
-		)
-		(property "Supply part number" "Điện Trở 18 KOhm 1/4W 5% 4 Vòng Màu"
-			(at 109.982 153.924 0)
-			(effects
-				(font
-					(size 1.27 1.27)
-				)
-				(hide yes)
-			)
-		)
-		(property "Supply URL" "https://www.thegioiic.com/dien-tro-18-kohm-1-4w-5-4-vong-mau"
-			(at 109.982 153.924 0)
-			(effects
-				(font
-					(size 1.27 1.27)
-				)
-				(hide yes)
-			)
-		)
-		(pin "1"
-		)
-		(pin "2"
-		)
-		(instances
-			(project "PFC"
-				(path "/3b17fecf-a6c4-4ae7-a684-61da545cc8d4"
-					(reference "R10")
-					(unit 1)
-				)

Commit message: update: PFC
Parts:
- removed R2, R6: 330K_1/4W_1%, charge_battery_footprint_lib:Res_18K_1_4W_1, symbol charge_battery_sym_lib:Res_hole_18K_1/4W_1%
- added C14: 100nF_50V_3216, Capacitor_SMD:C_1206_3216Metric, symbol charge_battery_sym_lib:Ceramic_Cap_SMD_10uF_16V
- added Q1: MMBT3904, Package_TO_SOT_SMD:SOT-23, symbol Transistor_BJT:MMBT3904
- added R10: 1K/1%/1_4W, Resistor_SMD:R_1206_3216Metric, symbol charge_battery_sym_lib:Res_200K_0603_1%
- added R12: 10K/1%/1_4W, Resistor_SMD:R_1206_3216Metric, symbol charge_battery_sym_lib:Res_200K_0603_1%
- added R13, R14: 330K_1/4W_1%_3216, Resistor_SMD:R_1206_3216Metric, symbol charge_battery_sym_lib:Res_hole_18K_1/4W_1%
- added TP1: TestPoint, symbol Connector:TestPoint
- added U2: SN74LVC1G14DBV, Package_TO_SOT_SMD:SOT-23-5, symbol 74xGxx:SN74LVC1G14DBV
- C11: value 4.7uF 50V -> 4.7uF_50V_3216
- C12, C3: value 1nF 50V -> 1nF_50V_3216; footprint charge_battery_footprint_lib:Ceramic_Cap_Hole_1nF_50V -> Capacitor_SMD:C_1206_3216Metric; Supply URL https://www.thegioiic.com/tu-gom-tron-1nf-50v -> https://www.thegioiic.com/tu-gom-1206-1nf-50v; Supply part number Tụ Gốm Tròn 1nF 50V -> Tụ Gốm 1206 1nF 50V
- C2: value 47uF_16VV -> 47uF_16V
- C7: value 680pF 1000V -> 1000pF_50V_3216; footprint charge_battery_footprint_lib:Ceramic_Cap_Hole_680pF_1000V -> Capacitor_SMD:C_1206_3216Metric; Supply URL https://thegioiic.com/tu-gom-xanh-680pf-1000v -> https://www.thegioiic.com/tu-gom-1206-1nf-50v; Supply part number Tụ Gốm Xanh 680pF 1000V -> Tụ Gốm 1206 1nF 50V
- C8: value 10uF_50V -> 8.2uF 0V; Supply URL https://www.thegioiic.com/tu-gom-0805-10uf-50v -> https://linhkien.cxt.vn/7871-tu-khong-phan-cuc-0805.html; Supply part number Tụ Gốm 0805 10uF 50V -> Tụ Gốm 0805 8.2uF 50V
- C9: value 680nF 50V 1206 -> 680nF_50V_3216
- R7: value 18K_1/4W_1% -> 18K_1/4W_5%_3216; footprint charge_battery_footprint_lib:Res_18K_1_4W_1 -> Resistor_SMD:R_1206_3216Metric; Supply URL https://www.thegioiic.com/dien-tro-18-kohm-1-4w-1-5-vong-mau -> https://www.thegioiic.com/dien-tro-18-kohm-1206-5-; Supply part number Điện Trở 18 KOhm 1/4W 1% 4 Vòng Màu -> Điện Trở 18 KOhm 1206 5%
- R8: value 330K_1/4W_1% -> 330K_1/4W_1%_3216; footprint charge_battery_footprint_lib:Res_18K_1_4W_1 -> Resistor_SMD:R_1206_3216Metric; Supply URL https://www.thegioiic.com/dien-tro-330-kohm-1-4w-1-5-vong-m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 -> https://www.thegioiic.com/dien-tro-330-kohm-1206-1-; Supply part number Điện Trở 330 KOhm 1/4W 1% 4 Vòng Màu -> Điện Trở 330 KOhm 1206 1%
Connections:
- net GND: now also C14.1, Q1.2 (E), R12.1, U2.3 (GND)
- net at C12.2, R1.2, R8.1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: now also Q1.3 (C)
- net at R8.2: now also R13.1
- net V_OUT_PFC renamed PFC_VCC
- net PFC_VCC: now also R14.2, TP1.1
- new net: C14.2, R10.2, R12.2, U2.4
- new net: Q1.1 (B), R10.1
- new net: R13.2, R14.1
- new net +5V: U2.5 (VCC)
- new net PFC_ON/OFF: U2.2
Other:
- moved on the sheet: C1, C10, C11, C12, C13, C2, C4, C5, C6, C7, C8, C9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

Commit message: update PFC
Parts:
- removed C13: 330uF_450V, charge_battery_footprint_lib:Big_Cap_330uF_450V, symbol charge_battery_sym_lib:Cap_Polarized_330uF_450V
- removed C7: 1000pF_50V_3216, Capacitor_SMD:C_1206_3216Metric, symbol charge_battery_sym_lib:Ceramic_Cap_Hole_1nF_2000V
- removed D1: KBPC606, charge_battery_footprint_lib:TO_BPC606_VIS, symbol charge_battery_sym_lib:KBPC606
- added C13: Cap_Polarized_1000uF_450V, charge_battery_footprint_lib:Big_Cap_330uF_450V, symbol charge_battery_sym_lib:Cap_Polarized_1000uF_450V
- added C7: 820pF_50V_0805, Capacitor_SMD:C_0805_2012Metric, symbol charge_battery_sym_lib:Ceramic_Cap_Hole_1nF_50V
- added D5: KBU808, Diode_THT:Diode_Bridge_Vishay_KBU, symbol charge_battery_sym_lib:KBU808
- C1, C10, C6: value 100nF, 275VAC -> 220nF, 275VAC; footprint charge_battery_footprint_lib:CAP_B32671P-10--5x11x13_TDK -> charge_battery_footprint_lib:Candy_Cap_hole_100nF_275V; Supply URL https://www.thegioiic.com/tu-keo-vang-x2-100nf-0-1uf-104k-2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 -> https://www.thegioiic.com/tu-keo-vang-x2-220nf-224k-275vac; Supply part number Tụ Kẹo Vàng X2 100nF (0.1uF) 104K 275VAC -> Tụ Kẹo Vàng X2 220nF 224K 275VAC
- C12: value 1nF_50V_3216 -> 820pF_50V_0805; footprint Capacitor_SMD:C_1206_3216Metric -> Capacitor_SMD:C_0805_2012Metric; Supply URL https://www.thegioiic.com/tu-gom-1206-1nf-50v -> https://www.thegioiic.com/tu-gom-0805-820pf-50v; Supply part number Tụ Gốm 1206 1nF 50V -> Tụ Gốm 0805 820pF 50V Tụ Gốm 0805 820pF 50V
- C8: value 8.2uF 0V -> 8.2uF_50V_0805
- L2: value 680uH -> 330uH; Supply URL https://www.thegioiic.com/cdrh127-cuon-cam-dan-smd-1280-681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 -> https://www.thegioiic.com/cdrh127-cuon-cam-dan-smd-1280-331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; Supply part number CDRH127 Cuộn Cảm Dán SMD 1280-681 680uH 1.03A -> CDRH127 Cuộn Cảm Dán SMD 1280-331 330uH 1.45A
- M1: value 600V 9.5A -> 600V 12A; Supply URL https://www.thegioiic.com/fqpf10n60c-mosfet-kenh-n-600v-9-5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 -> https://www.thegioiic.com/fqpf12n60c-mosfet-kenh-600v-12a-t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; Supply part number FQPF10N60C MOSFET Kênh N 600V 9.5A TO-220F -> FQPF12N60C MOSFET Kênh 600V 12A TO-220-3
- R4: value 3,3K_1/4W_1% -> 3,3R_1/4W_1%
Connections:
- net GND: now also C13.2, C7.1
- net PFC_VCC: now also C13.1
- net at C10.2, D3.1, L2.1: now also D5.1 (+)
- net at C4.2, C6.1, L1.2: now also D5.2
- net at C10.1, R3.2, R9.2: now also D5.4 (-)
- net at TH1.2: now also D5.3
- net at R9.1, U1.3 (ISENSE): now also C7.2
