File: Hardware/Source/System_Control/_autosave-System_Control.kicad_pcb (KiCad board)
At the start: 4 copper layers, 100 x 156.4 mm, 566 parts, among them J1 POWER_CONN, J10 NTC_CONN, J11 NTC_CONN, J12 NTC_CONN, J13 NTC_CONN, J14 NTC_CONN, J15 NTC_CONN, J16 BAL_BAT_CONN2, J17 NTC_CONN, J18 NTC_CONN, J19 NTC_CONN, J2 USB_B_Micro, J20 NTC_CONN, J21 NTC_CONN, J22 NTC_CONN, J23 NTC_CONN, J24 NTC_CONN, J3 SIGNAL_CONN, J4 Conn_01x02_Socket, J5 FLASH_CONN, J6 Conn_01x02_Socket, J7 BAL_BAT_CONN1, J8 NTC_CONN, J9 NTC_CONN, Q1 MMBT2222A, Q10 AO3400A, Q11 AO3400A, Q12 AO3400A, Q13 AO3400A, Q14 AO3400A, Q15 AO3400A, Q16 AO3400A, Q17 AO3400A, Q18 AO3400A, Q19 AO3400A, Q2 MMBT2222A, Q20 AO3400A, Q21 LN2302LT1G, Q22 SQJ211ELP-T1_GE3, Q23 SQJ211ELP-T1_GE3, Q24 LN2302LT1G, Q3 MMBT2222A, Q4 MMBT2222A, Q5 AO3400A, Q6 AO3400A, Q7 AO3400A, Q8 AO3400A, Q9 AO3400A, SW1 SW_Push, SW2 SW_Push, SW3 SW_Push, U1 ESP32-WROOM-32U, U10 NE5532DR, U11 NE5532DR, U12 NE5532DR, U13 NE5532DR, U14 TLP291-4, U15 TLP291-4, U16 TLP291-4, U17 TLP291-4, U18 CD74HC4067SM96, U19 CD74HC4067SM96, U2 CH340C, U20 EL3H7, U21 EL3H7, U3 STM32F407VET6, U4 LCD 5“SSD1963, U5 MAX485CSA, U6 NE5532DR, U7 NE5532DR, U8 NE5532DR, U9 NE5532DR, Y1 Crystal_25MHz_SMD-4PIN

Commit message: update lib lcd
Parts:
- moved Q13 0.55 mm to (217.9, 223.3)
- moved D59 0.53 mm to (216.2, 218.8)
- moved D43 0.49 mm to (212.9, 209.2)
- moved D35 0.44 mm to (216.5, 195.5)
- moved Q5 0.43 mm to (217.5, 199.9)
- moved Q9 0.43 mm to (217.5, 205.0)
- moved R132 0.43 mm to (215.5, 198.5)
- moved R144 0.43 mm to (215.5, 203.5)
- moved D33 0.43 mm to (213.1, 200.2)
- moved D41 0.43 mm to (213.1, 205.3)
- moved R164 0.33 mm to (215.9, 221.8)
- moved D57 0.23 mm to (213.6, 223.5)
- moved D67 0.06 mm to (213.4, 232.6)
Routing:
- net Net-(Q13-D): track 0.00 -> 34.6 mm
- net Net-(Q15-D): track 0.00 -> 14.4 mm, vias 0 -> 1
- net Net-(Q13-G): track 0.00 -> 7.78 mm, vias 0 -> 1
- net Net-(D43-A): track 12.2 -> 15.8 mm
- net Net-(Q5-D): track 35.3 -> 34.5 mm
- net Net-(D67-A): track 15.2 -> 15.8 mm
- net Net-(D35-A): track 15.5 -> 14.9 mm
