File: Hardware/Source/System_Control/connector.kicad_sch (KiCad schematic)
At the start: 35 parts, among them J10 BAL_BAT_CONN2, J11 NTC_CONN, J12 NTC_CONN, J3 SIGNAL_CONN, J4 Conn_01x02_Socket, J5 FLASH_CONN, J6 Conn_01x02_Socket, J7 NTC_CONN, J8 NTC_CONN, J9 BAL_BAT_CONN1

Commit message: pull lib
Connections:
- net NTC_10+: now also J11.3 (Pin_3); no longer J11.6 (Pin_6)
- net NTC_10-: now also J11.4 (Pin_4); no longer J11.5 (Pin_5)
- net NTC_11+: now also J11.5 (Pin_5); no longer J11.4 (Pin_4)
- net NTC_11-: now also J11.6 (Pin_6); no longer J11.3 (Pin_3)
- net NTC_12+: now also J11.7 (Pin_7); no longer J11.2 (Pin_2)
- net NTC_12-: now also J11.8 (Pin_8); no longer J11.1 (Pin_1)
- net NTC_13+: now also J12.1 (Pin_1); no longer J12.8 (Pin_8)
- net NTC_13-: now also J12.2 (Pin_2); no longer J12.7 (Pin_7)
- net NTC_14+: now also J12.3 (Pin_3); no longer J12.6 (Pin_6)
- net NTC_14-: now also J12.4 (Pin_4); no longer J12.5 (Pin_5)
- net NTC_15+: now also J12.5 (Pin_5); no longer J12.4 (Pin_4)
- net NTC_15-: now also J12.6 (Pin_6); no longer J12.3 (Pin_3)
- net NTC_16+: now also J12.7 (Pin_7); no longer J12.2 (Pin_2)
- net NTC_16-: now also J12.8 (Pin_8); no longer J12.1 (Pin_1)
- net NTC_9+: now also J11.1 (Pin_1); no longer J11.8 (Pin_8)
- net NTC_9-: now also J11.2 (Pin_2); no longer J11.7 (Pin_7)
Changed lines of the file:
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@@
+	)
+	(symbol
+		(lib_id "Connector:Conn_01x08_Socket")
+		(at 234.95 107.95 0)
+		(mirror y)
+		(unit 1)
+		(exclude_from_sim no)
+		(in_bom yes)
+		(on_board yes)
+		(dnp no)
+		(property "Reference" "J12"
+			(at 233.68 107.9499 0)
+			(effects
+				(font
+					(size 1.27 1.27)
+				)
+				(justify left)
+			)
+		)
+		(property "Value" "NTC_CONN"
+			(at 239.776 120.65 0)
+			(effects
+				(font
+					(size 1.27 1.27)
+				)
+				(justify left)
+			)
+		)
+		(property "Footprint" "charge_battery_footprint_lib:XH_2.54mm_8_SMD"
+			(at 234.95 107.95 0)
+			(effects
+				(font
+					(size 1.27 1.27)
+				)
+				(hide yes)
+			)
+		)
+		(property "Datasheet" "~"
+			(at 234.95 107.95 0)
+			(effects
+				(font
+					(size 1.27 1.27)
+				)
+				(hide yes)
+			)
+		)
+		(property "Description" "Generic connector, single row, 01x08, script generated"
+			(at 234.95 107.95 0)
+			(effects
+				(font
+					(size 1.27 1.27)
+				)
+				(hide yes)
+			)
+		)
+		(property "Supply name" "Thegioiic"
+			(at 234.95 107.95 0)
+			(effects
+				(font
+					(size 1.27 1.27)
+				)
+				(hide yes)
+			)
+		)
+		(property "Supply URL" "https://www.thegioiic.com/dau-xh2-54mm-8-chan-dan-smd-nam-ngang"
+			(at 234.95 107.95 0)
+			(effects
+				(font
+					(size 1.27 1.27)
+				)
+				(hide yes)
+			)
+		)
+		(pin "6"
+		)
+		(pin "3"
+		)
+		(pin "5"
+		)
+		(pin "1"
+		)
+		(pin "2"
+		)
+		(pin "7"
+		)
+		(pin "8"
+		)
+		(pin "4"
+		)
+		(instances
+			(project "System_Control"
+				(path "/85c53e8c-0403-413d-b6c5-0718d4365b1f/3a5f6f4d-7ae8-4d5e-869b-e74be22e0b12"
+					(reference "J12")
+					(unit 1)
+				)
+			)
+		)
 	)
 	(symbol
@@
 	)
 	(symbol
-		(lib_id "Connector:Conn_01x08_Socket")
-		(at 234.95 86.36 180)
-		(unit 1)
-		(exclude_from_sim no)
-		(in_bom yes)
-		(on_board yes)
-		(dnp no)
-		(property "Reference" "J11"
-			(at 233.68 86.3601 0)
-			(effects
-				(font
-					(size 1.27 1.27)
-				)
-				(justify left)
-			)
-		)
-		(property "Value" "NTC_CONN"
-			(at 238.506 96.266 0)
-			(effects
-				(font
-					(size 1.27 1.27)
-				)
-				(justify left)
-			)
-		)
-		(property "Footprint" "charge_battery_footprint_lib:XH_2.54mm_8_SMD"
-			(at 234.95 86.36 0)
-			(effects
-				(font
-					(size 1.27 1.27)
-				)
-				(hide yes)
-			)
-		)
-		(property "Datasheet" "~"
-			(at 234.95 86.36 0)
-			(effects
-				(font
-					(size 1.27 1.27)
-				)
-				(hide yes)
-			)
-		)
-		(property "Description" "Generic connector, single row, 01x08, script generated"
-			(at 234.95 86.36 0)
-			(effects
-				(font
-					(size 1.27 1.27)
-				)
-				(hide yes)
-			)
-		)
-		(property "Supply name" "Thegioiic"
-			(at 234.95 86.36 0)
-			(effects
-				(font
-					(size 1.27 1.27)
-				)
-				(hide yes)
-			)
-		)
-		(property "Supply URL" "https://www.thegioiic.com/dau-xh2-54mm-8-chan-dan-smd-nam-ngang"
-			(at 234.95 86.36 0)
-			(effects
-				(font
-					(size 1.27 1.27)
-				)
-				(hide yes)
-			)
-		)
-		(pin "6"
-		)
-		(pin "3"
-		)
-		(pin "5"
-		)
-		(pin "1"
-		)
-		(pin "2"
-		)
-		(pin "7"
-		)
-		(pin "8"
-		)
-		(pin "4"
-		)
-		(instances
-			(project "System_Control"
-				(path "/85c53e8c-0403-413d-b6c5-0718d4365b1f/3a5f6f4d-7ae8-4d5e-869b-e74be22e0b12"
-					(reference "J11")
-					(unit 1)
-				)
-			)
-		)
-	)
-	(symbol
 		(lib_id "Connector:Conn_01x07_Socket")
 		(at 233.68 48.26 180)
@@
 	)
 	(symbol
-		(lib_id "Connector:Conn_01x08_Socket")
-		(at 234.95 110.49 180)
-		(unit 1)
-		(exclude_from_sim no)
-		(in_bom yes)
-		(on_board yes)
-		(dnp no)
-		(property "Reference" "J12"
-			(at 233.68 110.4901 0)
-			(effects
-				(font
-					(size 1.27 1.27)
-				)
-				(justify left)
-			)
-		)
-		(property "Value" "NTC_CONN"
-			(at 238.506 120.396 0)
-			(effects
-				(font
-					(size 1.27 1.27)
-				)
-				(justify left)
-			)
-		)
-		(property "Footprint" "charge_battery_footprint_lib:XH_2.54mm_8_SMD"
-			(at 234.95 110.49 0)
-			(effects
-				(font
-					(size 1.27 1.27)
-				)
-				(hide yes)
-			)
-		)
-		(property "Datasheet" "~"
-			(at 234.95 110.49 0)
-			(effects
-				(font
-					(size 1.27 1.27)
-				)
-				(hide yes)
-			)
-		)
-		(property "Description" "Generic connector, single row, 01x08, script generated"
-			(at 234.95 110.49 0)
-			(effects
-				(font
-					(size 1.27 1.27)
-				)
-				(hide yes)
-			)
-		)
-		(property "Supply name" "Thegioiic"
-			(at 234.95 110.49 0)
-			(effects
-				(font
-					(size 1.27 1.27)
-				)
-				(hide yes)
-			)
-		)
-		(property "Supply URL" "https://www.thegioiic.com/dau-xh2-54mm-8-chan-dan-smd-nam-ngang"
-			(at 234.95 110.49 0)
-			(effects
-				(font
-					(size 1.27 1.27)
-				)
-				(hide yes)
-			)
-		)
-		(pin "6"
-		)
-		(pin "3"
-		)
-		(pin "5"
-		)
-		(pin "1"
-		)
-		(pin "2"
-		)
-		(pin "7"
-		)
-		(pin "8"
-		)
-		(pin "4"
-		)
-		(instances
-			(project "System_Control"
-				(path "/85c53e8c-0403-413d-b6c5-0718d4365b1f/3a5f6f4d-7ae8-4d5e-869b-e74be22e0b12"
-					(reference "J12")
-					(unit 1)
-				)
-			)
-		)
-	)
-	(symbol
 		(lib_id "Connector:Conn_01x05_Socket")
 		(at 76.2 113.03 0)
@@
 					(unit 1)
 				)
+			)
+		)
+	)
+	(symbol
+		(lib_id "Connector:Conn_01x08_Socket")
+		(at 234.95 83.82 0)
+		(mirror y)
+		(unit 1)
+		(exclude_from_sim no)
+		(in_bom yes)
+		(on_board yes)
+		(dnp no)
+		(property "Reference" "J11"
+			(at 233.68 83.8199 0)
+			(effects
+				(font
+					(size 1.27 1.27)
+				)
+				(justify left)
+			)
+		)
+		(property "Value" "NTC_CONN"
+			(at 240.03 96.266 0)
+			(effects
+				(font
+					(size 1.27 1.27)
+				)
+				(justify left)
+			)
+		)
+		(property "Footprint" "charge_battery_footprint_lib:XH_2.54mm_8_SMD"
+			(at 234.95 83.82 0)
+			(effects
+				(font
+					(size 1.27 1.27)
+				)
+				(hide yes)
+			)
+		)
+		(property "Datasheet" "~"
+			(at 234.95 83.82 0)
+			(effects
+				(font
+					(size 1.27 1.27)
+				)
+				(hide yes)
+			)
+		)
+		(property "Description" "Generic connector, single row, 01x08, script generated"
+			(at 234.95 83.82 0)
+			(effects
+				(font
+					(size 1.27 1.27)
+				)
+				(hide yes)
+			)
+		)
+		(property "Supply name" "Thegioiic"
+			(at 234.95 83.82 0)
+			(effects
+				(font
+					(size 1.27 1.27)
+				)
+				(hide yes)
+			)
+		)
+		(property "Supply URL" "https://www.thegioiic.com/dau-xh2-54mm-8-chan-dan-smd-nam-ngang"
+			(at 234.95 83.82 0)
+			(effects
+				(font
+					(size 1.27 1.27)
+				)
+				(hide yes)
+			)
+		)
+		(pin "6"
+		)
+		(pin "3"
+		)
+		(pin "5"
+		)
+		(pin "1"
+		)
+		(pin "2"
+		)
+		(pin "7"
+		)
+		(pin "8"
+		)
+		(pin "4"
+		)
+		(instances
+			(project "System_Control"
+				(path "/85c53e8c-0403-413d-b6c5-0718d4365b1f/3a5f6f4d-7ae8-4d5e-869b-e74be22e0b12"
+					(reference "J11")
+					(unit 1)
+				)

Commit message: pull
Parts:
- renumbered C173 to C167, C174 to C168, D77 to D75, D78 to D76, R206 to R202, R207 to R203, TP13 to TP12, TP14 to TP13, TP15 to TP14, TP16 to TP15, TP17 to TP16, TP18 to TP17, TP19 to TP18, TP20 to TP19, TP21 to TP20, TP22 to TP21, TP23 to TP22, TP24 to TP23, TP25 to TP24, TP26 to TP25, TP27 to TP26, TP28 to TP27, TP29 to TP28, TP30 to TP29, TP31 to TP30

Commit message: check
Parts:
- removed C167: 10uF/16V, charge_battery_footprint_lib:Ceramic_Cap_0603, symbol charge_battery_sym_lib:Ceramic_Cap_SMD_10uF_16V
- removed C168: 100nF/16V, charge_battery_footprint_lib:Ceramic_Cap_0603, symbol charge_battery_sym_lib:Ceramic_Cap_SMD_100nF_16V
- removed TP12, TP13, TP14, TP15, TP16, TP17, TP18, TP19, TP20, TP21, TP22, TP23, TP24, TP25, TP26, TP27, TP28, TP29, TP30: TestPoint_Small, TestPoint:TestPoint_Pad_D1.0mm, symbol Connector:TestPoint_Small
- added R202, R203: 20R/5%/1_16W, charge_battery_footprint_lib:Res_0402, symbol charge_battery_sym_lib:Res_20R_0402_5%
- renumbered D75 to D74, D76 to D75, R202 to R200, R203 to R201
Connections:
- net SWCLK: now also R203.2; no longer D75.1, J5.3 (Pin_3)
- net SWDIO: now also R202.2; no longer D75.2, J5.2 (Pin_2)
- net UART3_RX renamed UART2_RX
- net UART3_TX renamed UART2_TX
- new net: D75.1, J5.2 (Pin_2), R202.1
- new net: D75.2, J5.3 (Pin_3), R203.1
Other:
- moved on the sheet: D75
