File: Hardware/Source/System_Control/signalkicad_sch.kicad_sch (KiCad schematic)
At the start: 15 parts, among them Q4 MMBT2222A, U5 MAX485CSA

Commit message: pcb,lib,sche: PFC, lib: update pcb PFC, lib
Parts:
- renumbered C42 to C47, C43 to C48, C44 to C49, C45 to C50, D25 to D24, R32 to R34, R33 to R35, R34 to R36, R35 to R37, R36 to R38, R37 to R39, R38 to R40, R39 to R41
Changed lines of the file:
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@@
 		(on_board yes)
 		(dnp no)
-		(property "Reference" "C43"
+		(property "Reference" "C48"
 			(at 121.92 123.952 90)
 			(effects
@@
 			(project "System_Control"
 				(path "/85c53e8c-0403-413d-b6c5-0718d4365b1f/eadc6d73-e2ad-4643-bc1f-3abdfd5d95f1"
-					(reference "C43")
+					(reference "C48")
 					(unit 1)
 				)
@@
 		(on_board yes)
 		(dnp no)
-		(property "Reference" "R39"
+		(property "Reference" "R41"
 			(at 196.596 97.79 0)
 			(effects
@@
 			(project "System_Control"
 				(path "/85c53e8c-0403-413d-b6c5-0718d4365b1f/eadc6d73-e2ad-4643-bc1f-3abdfd5d95f1"
-					(reference "R39")
+					(reference "R41")
 					(unit 1)
 				)
@@
 		(on_board yes)
 		(dnp no)
-		(property "Reference" "R34"
+		(property "Reference" "R36"
 			(at 92.71 89.408 0)
 			(effects
@@
 			(project "System_Control"
 				(path "/85c53e8c-0403-413d-b6c5-0718d4365b1f/eadc6d73-e2ad-4643-bc1f-3abdfd5d95f1"
-					(reference "R34")
+					(reference "R36")
 					(unit 1)
 				)
@@
 		(on_board yes)
 		(dnp no)
-		(property "Reference" "R32"
+		(property "Reference" "R34"
 			(at 72.136 83.058 90)
 			(effects
@@
 			(project "System_Control"
 				(path "/85c53e8c-0403-413d-b6c5-0718d4365b1f/eadc6d73-e2ad-4643-bc1f-3abdfd5d95f1"
-					(reference "R32")
+					(reference "R34")
 					(unit 1)
 				)
@@
 		(on_board yes)
 		(dnp no)
-		(property "Reference" "C44"
+		(property "Reference" "C49"
 			(at 161.29 99.822 90)
 			(effects
@@
 			(project "System_Control"
 				(path "/85c53e8c-0403-413d-b6c5-0718d4365b1f/eadc6d73-e2ad-4643-bc1f-3abdfd5d95f1"
-					(reference "C44")
+					(reference "C49")
 					(unit 1)
 				)
@@
 		(on_board yes)
 		(dnp no)
-		(property "Reference" "R33"
+		(property "Reference" "R35"
 			(at 92.71 75.438 0)
 			(effects
@@
 			(project ""
 				(path "/85c53e8c-0403-413d-b6c5-0718d4365b1f/eadc6d73-e2ad-4643-bc1f-3abdfd5d95f1"
-					(reference "R33")
+					(reference "R35")
 					(unit 1)
 				)
@@
 		(on_board yes)
 		(dnp no)
-		(property "Reference" "R38"
+		(property "Reference" "R40"
 			(at 196.85 58.42 0)
 			(effects
@@
 			(project "System_Control"
 				(path "/85c53e8c-0403-413d-b6c5-0718d4365b1f/eadc6d73-e2ad-4643-bc1f-3abdfd5d95f1"
-					(reference "R38")
+					(reference "R40")
 					(unit 1)
 				)
@@
 		(on_board yes)
 		(dnp no)
-		(property "Reference" "D25"
+		(property "Reference" "D24"
 			(at 208.026 76.708 0)
 			(effects
@@
 			(project "System_Control"
 				(path "/85c53e8c-0403-413d-b6c5-0718d4365b1f/eadc6d73-e2ad-4643-bc1f-3abdfd5d95f1"
-					(reference "D25")
+					(reference "D24")
 					(unit 1)
 				)
@@
 		(on_board yes)
 		(dnp no)
-		(property "Reference" "C42"
+		(property "Reference" "C47"
 			(at 110.49 123.952 90)
 			(effects
@@
 			(project "System_Control"
 				(path "/85c53e8c-0403-413d-b6c5-0718d4365b1f/eadc6d73-e2ad-4643-bc1f-3abdfd5d95f1"
-					(reference "C42")
+					(reference "C47")
 					(unit 1)
 				)
@@
 		(on_board yes)
 		(dnp no)
-		(property "Reference" "R37"
+		(property "Reference" "R39"
 			(at 186.944 76.962 90)
 			(effects
@@
 			(project ""
 				(path "/85c53e8c-0403-413d-b6c5-0718d4365b1f/eadc6d73-e2ad-4643-bc1f-3abdfd5d95f1"
-					(reference "R37")
+					(reference "R39")
 					(unit 1)
 				)
@@
 		(on_board yes)
 		(dnp no)
-		(property "Reference" "R35"
+		(property "Reference" "R37"
 			(at 139.7 74.168 0)
 			(effects
@@
 			(project "System_Control"
 				(path "/85c53e8c-0403-413d-b6c5-0718d4365b1f/eadc6d73-e2ad-4643-bc1f-3abdfd5d95f1"
-					(reference "R35")
+					(reference "R37")
 					(unit 1)
 				)
@@
 		(on_board yes)
 		(dnp no)
-		(property "Reference" "C45"
+		(property "Reference" "C50"
 			(at 172.72 99.822 90)
 			(effects
@@
 			(project "System_Control"
 				(path "/85c53e8c-0403-413d-b6c5-0718d4365b1f/eadc6d73-e2ad-4643-bc1f-3abdfd5d95f1"
-					(reference "C45")
+					(reference "C50")
 					(unit 1)
 				)
@@
 		(on_board yes)
 		(dnp no)
-		(property "Reference" "R36"
+		(property "Reference" "R38"
 			(at 139.7 81.788 0)
 			(effects
@@
 			(project "System_Control"
 				(path "/85c53e8c-0403-413d-b6c5-0718d4365b1f/eadc6d73-e2ad-4643-bc1f-3abdfd5d95f1"
-					(reference "R36")
-					(unit 1)
-				)
+					(reference "R38")
+					(unit 1)
+				)

Commit message: pull
Connections:
- net RS485_A renamed RS485_P
- net RS485_P: now also D24.1; no longer D24.2
- net RS485_B renamed RS485_N
- net RS485_N: now also D24.2; no longer D24.1
Changed lines of the file:
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@@
 		)
 	)
-	(global_label "RS485_B"
+	(label "RS485_N"
+		(at 191.77 73.66 0)
+		(fields_autoplaced yes)
+		(effects
+			(font
+				(size 1.27 1.27)
+			)
+			(justify left bottom)
+		)
+	)
+	(label "RS485_P"
+		(at 191.77 86.36 0)
+		(fields_autoplaced yes)
+		(effects
+			(font
+				(size 1.27 1.27)
+			)
+			(justify left bottom)
+		)
+	)
+	(global_label "RS485_N"
 		(shape bidirectional)
 		(at 215.9 73.66 0)
@@
 		)
 		(property "Intersheetrefs" "${INTERSHEET_REFS}"
-			(at 228.3421 73.66 0)
+			(at 228.4026 73.66 0)
 			(effects
 				(font
@@
 		)
 	)
-	(global_label "RS485_A"
+	(global_label "RS485_P"
 		(shape bidirectional)
 		(at 215.9 86.36 0)
@@
 		)
 		(property "Intersheetrefs" "${INTERSHEET_REFS}"
-			(at 228.1607 86.36 0)
+			(at 228.3421 86.36 0)
 			(effects
 				(font
@@
 	(symbol
 		(lib_id "charge_battery_sym_lib:PESD2USB3UXT-QR")
-		(at 208.28 82.55 0)
+		(at 208.28 77.47 0)
+		(mirror x)
 		(unit 1)
 		(exclude_from_sim no)
@@
 		(dnp no)
 		(property "Reference" "D24"
-			(at 208.026 76.708 0)
+			(at 208.026 76.454 0)
 			(effects
 				(font
@@
 		)
 		(property "Value" "PESD2USB3UXT-QR"
-			(at 212.344 82.804 0)
+			(at 212.344 82.55 0)
 			(effects
 				(font
@@
 		)
 		(property "Footprint" "charge_battery_footprint_lib:SOT23"
-			(at 212.852 94.742 0)
+			(at 212.852 65.278 0)
 			(effects
 				(font
@@
 		)
 		(property "Datasheet" "https://www.mouser.vn/datasheet/2/916/PESD2USB3UXT_Q-3435971.pdf"
-			(at 213.868 94.742 0)
+			(at 213.868 65.278 0)
 			(effects
 				(font
@@
 		)
 		(property "Description" "ESD Protection Diodes / TVS Diodes SOT23 3.3V 4A AUTO ESD PROT"
-			(at 209.042 94.742 0)
+			(at 209.042 65.278 0)
 			(effects
 				(font
@@
 		)
 		(property "Supply name" "Mouser"
-			(at 209.55 94.742 0)
+			(at 209.55 65.278 0)
 			(effects
 				(font
@@
 		)
 		(property "Supply part number" "771-PESD2USB3UXT-QR"
-			(at 209.804 94.742 0)
+			(at 209.804 65.278 0)
 			(effects
 				(font
@@
 		)
 		(property "Supply URL" "https://www.mouser.vn/ProductDetail/Nexperia/PESD2USB3UXT-QR?qs=3Rah4i%252BhyCErbBl4ep9%252BDw%3D%3D"
-			(at 209.804 94.742 0)
-			(effects
-				(font
+			(at 209.804 65.278 0)
+			(effects
+				(font

Commit message: pull
Parts:
- renumbered C47 to C45, C48 to C46, C49 to C47, C50 to C48, R34 to R32, R35 to R33, R36 to R34, R37 to R35, R38 to R36, R39 to R37, R40 to R38, R41 to R39
Changed lines of the file:
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@@
 		(dnp no)
 		(fields_autoplaced yes)
-		(property "Reference" "#PWR074"
+		(property "Reference" "#PWR071"
 			(at 110.49 138.43 0)
 			(effects
@@
 			(project "System_Control"
 				(path "/85c53e8c-0403-413d-b6c5-0718d4365b1f/eadc6d73-e2ad-4643-bc1f-3abdfd5d95f1"
-					(reference "#PWR074")
+					(reference "#PWR071")
 					(unit 1)
 				)
@@
 		(dnp no)
 		(fields_autoplaced yes)
-		(property "Reference" "#PWR077"
+		(property "Reference" "#PWR074"
 			(at 176.53 78.74 0)
 			(effects
@@
 			(project "System_Control"
 				(path "/85c53e8c-0403-413d-b6c5-0718d4365b1f/eadc6d73-e2ad-4643-bc1f-3abdfd5d95f1"
-					(reference "#PWR077")
+					(reference "#PWR074")
 					(unit 1)
 				)
@@
 		(dnp no)
 		(fields_autoplaced yes)
-		(property "Reference" "#PWR079"
+		(property "Reference" "#PWR076"
 			(at 200.66 95.25 0)
 			(effects
@@
 			(project "System_Control"
 				(path "/85c53e8c-0403-413d-b6c5-0718d4365b1f/eadc6d73-e2ad-4643-bc1f-3abdfd5d95f1"
-					(reference "#PWR079")
+					(reference "#PWR076")
 					(unit 1)
 				)
@@
 		(dnp no)
 		(fields_autoplaced yes)
-		(property "Reference" "#PWR080"
+		(property "Reference" "#PWR077"
 			(at 212.09 63.5 0)
 			(effects
@@
 			(project "System_Control"
 				(path "/85c53e8c-0403-413d-b6c5-0718d4365b1f/eadc6d73-e2ad-4643-bc1f-3abdfd5d95f1"
-					(reference "#PWR080")
+					(reference "#PWR077")
 					(unit 1)
 				)
@@
 		(dnp no)
 		(fields_autoplaced yes)
-		(property "Reference" "#PWR075"
+		(property "Reference" "#PWR072"
 			(at 161.29 99.06 0)
 			(effects
@@
 			(project "System_Control"
 				(path "/85c53e8c-0403-413d-b6c5-0718d4365b1f/eadc6d73-e2ad-4643-bc1f-3abdfd5d95f1"
-					(reference "#PWR075")
+					(reference "#PWR072")
 					(unit 1)
 				)
@@
 		(on_board yes)
 		(dnp no)
-		(property "Reference" "C48"
+		(property "Reference" "C46"
 			(at 121.92 123.952 90)
 			(effects
@@
 			(project "System_Control"
 				(path "/85c53e8c-0403-413d-b6c5-0718d4365b1f/eadc6d73-e2ad-4643-bc1f-3abdfd5d95f1"
-					(reference "C48")
+					(reference "C46")
 					(unit 1)
 				)
@@
 		(on_board yes)
 		(dnp no)
-		(property "Reference" "R41"
+		(property "Reference" "R39"
 			(at 196.596 97.79 0)
 			(effects
@@
 			(project "System_Control"
 				(path "/85c53e8c-0403-413d-b6c5-0718d4365b1f/eadc6d73-e2ad-4643-bc1f-3abdfd5d95f1"
-					(reference "R41")
+					(reference "R39")
 					(unit 1)
 				)
@@
 		(dnp no)
 		(fields_autoplaced yes)
-		(property "Reference" "#PWR078"
+		(property "Reference" "#PWR075"
 			(at 176.53 91.44 0)
 			(effects
@@
 			(project "System_Control"
 				(path "/85c53e8c-0403-413d-b6c5-0718d4365b1f/eadc6d73-e2ad-4643-bc1f-3abdfd5d95f1"
-					(reference "#PWR078")
+					(reference "#PWR075")
 					(unit 1)
 				)
@@
 		(dnp no)
 		(fields_autoplaced yes)
-		(property "Reference" "#PWR073"
+		(property "Reference" "#PWR070"
 			(at 110.49 123.19 0)
 			(effects
@@
 			(project "System_Control"
 				(path "/85c53e8c-0403-413d-b6c5-0718d4365b1f/eadc6d73-e2ad-4643-bc1f-3abdfd5d95f1"
-					(reference "#PWR073")
+					(reference "#PWR070")
 					(unit 1)
 				)
@@
 		(on_board yes)
 		(dnp no)
-		(property "Reference" "R36"
+		(property "Reference" "R34"
 			(at 92.71 89.408 0)
 			(effects
@@
 			(project "System_Control"
 				(path "/85c53e8c-0403-413d-b6c5-0718d4365b1f/eadc6d73-e2ad-4643-bc1f-3abdfd5d95f1"
-					(reference "R36")
+					(reference "R34")
 					(unit 1)
 				)
@@
 		(on_board yes)
 		(dnp no)
-		(property "Reference" "#PWR072"
+		(property "Reference" "#PWR069"
 			(at 110.49 107.95 0)
 			(effects
@@
 			(project ""
 				(path "/85c53e8c-0403-413d-b6c5-0718d4365b1f/eadc6d73-e2ad-4643-bc1f-3abdfd5d95f1"
-					(reference "#PWR072")
+					(reference "#PWR069")
 					(unit 1)
 				)
@@
 		(on_board yes)
 		(dnp no)
-		(property "Reference" "R34"
+		(property "Reference" "R32"
 			(at 72.136 83.058 90)
 			(effects
@@
 			(project "System_Control"
 				(path "/85c53e8c-0403-413d-b6c5-0718d4365b1f/eadc6d73-e2ad-4643-bc1f-3abdfd5d95f1"
-					(reference "R34")
+					(reference "R32")
 					(unit 1)
 				)
@@
 		(on_board yes)
 		(dnp no)
-		(property "Reference" "C49"
+		(property "Reference" "C47"
 			(at 161.29 99.822 90)
 			(effects
@@
 			(project "System_Control"
 				(path "/85c53e8c-0403-413d-b6c5-0718d4365b1f/eadc6d73-e2ad-4643-bc1f-3abdfd5d95f1"
-					(reference "C49")
+					(reference "C47")
 					(unit 1)
 				)
@@
 		(on_board yes)
 		(dnp no)
-		(property "Reference" "R35"
+		(property "Reference" "R33"
 			(at 92.71 75.438 0)
 			(effects
@@
 			(project ""
 				(path "/85c53e8c-0403-413d-b6c5-0718d4365b1f/eadc6d73-e2ad-4643-bc1f-3abdfd5d95f1"
-					(reference "R35")
+					(reference "R33")
 					(unit 1)
 				)
@@
 		(dnp no)
 		(fields_autoplaced yes)
-		(property "Reference" "#PWR076"
+		(property "Reference" "#PWR073"
 			(at 161.29 113.03 0)
 			(effects
@@
 			(project "System_Control"
 				(path "/85c53e8c-0403-413d-b6c5-0718d4365b1f/eadc6d73-e2ad-4643-bc1f-3abdfd5d95f1"
-					(reference "#PWR076")
+					(reference "#PWR073")
 					(unit 1)
 				)
@@
 		(on_board yes)
 		(dnp no)
-		(property "Reference" "R40"
+		(property "Reference" "R38"
 			(at 196.85 58.42 0)
 			(effects
@@
 			(project "System_Control"
 				(path "/85c53e8c-0403-413d-b6c5-0718d4365b1f/eadc6d73-e2ad-4643-bc1f-3abdfd5d95f1"
-					(reference "R40")
+					(reference "R38")
 					(unit 1)
 				)
@@
 		(on_board yes)
 		(dnp no)
-		(property "Reference" "C47"
+		(property "Reference" "C45"
 			(at 110.49 123.952 90)
 			(effects
@@
 			(project "System_Control"
 				(path "/85c53e8c-0403-413d-b6c5-0718d4365b1f/eadc6d73-e2ad-4643-bc1f-3abdfd5d95f1"
-					(reference "C47")
+					(reference "C45")
 					(unit 1)
 				)
@@
 		(on_board yes)
 		(dnp no)
-		(property "Reference" "R39"
+		(property "Reference" "R37"
 			(at 186.944 76.962 90)
 			(effects
@@
 			(project ""
 				(path "/85c53e8c-0403-413d-b6c5-0718d4365b1f/eadc6d73-e2ad-4643-bc1f-3abdfd5d95f1"
-					(reference "R39")
+					(reference "R37")
 					(unit 1)
 				)
@@
 		(on_board yes)
 		(dnp no)
-		(property "Reference" "R37"
+		(property "Reference" "R35"
 			(at 139.7 74.168 0)
 			(effects
@@
 			(project "System_Control"
 				(path "/85c53e8c-0403-413d-b6c5-0718d4365b1f/eadc6d73-e2ad-4643-bc1f-3abdfd5d95f1"
-					(reference "R37")
+					(reference "R35")
 					(unit 1)
 				)
@@
 		(dnp no)
 		(fields_autoplaced yes)
-		(property "Reference" "#PWR071"
+		(property "Reference" "#PWR068"
 			(at 69.85 82.55 0)
 			(effects
@@
 			(project "System_Control"
 				(path "/85c53e8c-0403-413d-b6c5-0718d4365b1f/eadc6d73-e2ad-4643-bc1f-3abdfd5d95f1"
-					(reference "#PWR071")
+					(reference "#PWR068")
 					(unit 1)
 				)
@@
 		(on_board yes)
 		(dnp no)
-		(property "Reference" "C50"
+		(property "Reference" "C48"
 			(at 172.72 99.822 90)
 			(effects
@@
 			(project "System_Control"
 				(path "/85c53e8c-0403-413d-b6c5-0718d4365b1f/eadc6d73-e2ad-4643-bc1f-3abdfd5d95f1"
-					(reference "C50")
+					(reference "C48")
 					(unit 1)
 				)
@@
 		(on_board yes)
 		(dnp no)
-		(property "Reference" "R38"
+		(property "Reference" "R36"
 			(at 139.7 81.788 0)
 			(effects
@@
 			(project "System_Control"
 				(path "/85c53e8c-0403-413d-b6c5-0718d4365b1f/eadc6d73-e2ad-4643-bc1f-3abdfd5d95f1"
-					(reference "R38")
+					(reference "R36")
 					(unit 1)
 				)
@@
 		(dnp no)
 		(fields_autoplaced yes)
-		(property "Reference" "#PWR081"
+		(property "Reference" "#PWR078"
 			(at 223.52 80.01 0)
 			(effects
@@
 			(project "System_Control"
 				(path "/85c53e8c-0403-413d-b6c5-0718d4365b1f/eadc6d73-e2ad-4643-bc1f-3abdfd5d95f1"
-					(reference "#PWR081")
-					(unit 1)
-				)
+					(reference "#PWR078")
+					(unit 1)
+				)

Commit message: check
Parts:
- removed D24: PESD2USB3UXT-QR, charge_battery_footprint_lib:SOT23, symbol charge_battery_sym_lib:PESD2USB3UXT-QR
- added D23: SMF05C, charge_battery_footprint_lib:SOT-363, symbol charge_battery_sym_lib:SMF05C
- renumbered C45 to C38, C46 to C39, C47 to C40, C48 to C41, R32 to R30, R33 to R31, R34 to R32, R35 to R33, R36 to R34, R37 to R35, R38 to R36, R39 to R37
Connections:
- net GNDD: now also D23.2
- net RS485_N: now also D23.4
- net RS485_P: now also D23.3
- net UART6_RX renamed UART4_RX
- net UART6_TX renamed UART4_TX

Commit message: check
Parts:
- renumbered D23 to D11, R30 to R31, R31 to R32, R32 to R33, R33 to R34, R34 to R35, R35 to R36, R36 to R37, R37 to R38
Changed lines of the file:
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@@
 		(dnp no)
 		(fields_autoplaced yes)
-		(property "Reference" "#PWR072"
+		(property "Reference" "#PWR070"
 			(at 110.49 138.43 0)
 			(effects
@@
 			(project "System_Control"
 				(path "/85c53e8c-0403-413d-b6c5-0718d4365b1f/eadc6d73-e2ad-4643-bc1f-3abdfd5d95f1"
-					(reference "#PWR072")
+					(reference "#PWR070")
 					(unit 1)
 				)
@@
 		(dnp no)
 		(fields_autoplaced yes)
-		(property "Reference" "#PWR075"
+		(property "Reference" "#PWR073"
 			(at 176.53 78.74 0)
 			(effects
@@
 			(project "System_Control"
 				(path "/85c53e8c-0403-413d-b6c5-0718d4365b1f/eadc6d73-e2ad-4643-bc1f-3abdfd5d95f1"
-					(reference "#PWR075")
+					(reference "#PWR073")
 					(unit 1)
 				)
@@
 		(dnp no)
 		(fields_autoplaced yes)
-		(property "Reference" "#PWR077"
+		(property "Reference" "#PWR075"
 			(at 200.66 95.25 0)
 			(effects
@@
 			(project "System_Control"
 				(path "/85c53e8c-0403-413d-b6c5-0718d4365b1f/eadc6d73-e2ad-4643-bc1f-3abdfd5d95f1"
-					(reference "#PWR077")
+					(reference "#PWR075")
 					(unit 1)
 				)
@@
 		(dnp no)
 		(fields_autoplaced yes)
-		(property "Reference" "#PWR078"
+		(property "Reference" "#PWR076"
 			(at 212.09 63.5 0)
 			(effects
@@
 			(project "System_Control"
 				(path "/85c53e8c-0403-413d-b6c5-0718d4365b1f/eadc6d73-e2ad-4643-bc1f-3abdfd5d95f1"
-					(reference "#PWR078")
+					(reference "#PWR076")
 					(unit 1)
 				)
@@
 		(dnp no)
 		(fields_autoplaced yes)
-		(property "Reference" "#PWR073"
+		(property "Reference" "#PWR071"
 			(at 161.29 99.06 0)
 			(effects
@@
 			(project "System_Control"
 				(path "/85c53e8c-0403-413d-b6c5-0718d4365b1f/eadc6d73-e2ad-4643-bc1f-3abdfd5d95f1"
-					(reference "#PWR073")
+					(reference "#PWR071")
 					(unit 1)
 				)
@@
 		(on_board yes)
 		(dnp no)
-		(property "Reference" "R37"
+		(property "Reference" "R38"
 			(at 196.596 97.79 0)
 			(effects
@@
 			(project "System_Control"
 				(path "/85c53e8c-0403-413d-b6c5-0718d4365b1f/eadc6d73-e2ad-4643-bc1f-3abdfd5d95f1"
-					(reference "R37")
+					(reference "R38")
 					(unit 1)
 				)
@@
 		(dnp no)
 		(fields_autoplaced yes)
-		(property "Reference" "#PWR076"
+		(property "Reference" "#PWR074"
 			(at 176.53 91.44 0)
 			(effects
@@
 			(project "System_Control"
 				(path "/85c53e8c-0403-413d-b6c5-0718d4365b1f/eadc6d73-e2ad-4643-bc1f-3abdfd5d95f1"
-					(reference "#PWR076")
+					(reference "#PWR074")
 					(unit 1)
 				)
@@
 		(dnp no)
 		(fields_autoplaced yes)
-		(property "Reference" "#PWR071"
+		(property "Reference" "#PWR069"
 			(at 110.49 123.19 0)
 			(effects
@@
 			(project "System_Control"
 				(path "/85c53e8c-0403-413d-b6c5-0718d4365b1f/eadc6d73-e2ad-4643-bc1f-3abdfd5d95f1"
-					(reference "#PWR071")
+					(reference "#PWR069")
 					(unit 1)
 				)
@@
 		(on_board yes)
 		(dnp no)
-		(property "Reference" "R32"
+		(property "Reference" "R33"
 			(at 92.71 89.408 0)
 			(effects
@@
 			(project "System_Control"
 				(path "/85c53e8c-0403-413d-b6c5-0718d4365b1f/eadc6d73-e2ad-4643-bc1f-3abdfd5d95f1"
-					(reference "R32")
+					(reference "R33")
 					(unit 1)
 				)
@@
 		(on_board yes)
 		(dnp no)
-		(property "Reference" "#PWR070"
+		(property "Reference" "#PWR068"
 			(at 110.49 107.95 0)
 			(effects
@@
 			(project ""
 				(path "/85c53e8c-0403-413d-b6c5-0718d4365b1f/eadc6d73-e2ad-4643-bc1f-3abdfd5d95f1"
-					(reference "#PWR070")
+					(reference "#PWR068")
 					(unit 1)
 				)
@@
 		(on_board yes)
 		(dnp no)
-		(property "Reference" "R30"
+		(property "Reference" "R31"
 			(at 72.136 83.058 90)
 			(effects
@@
 			(project "System_Control"
 				(path "/85c53e8c-0403-413d-b6c5-0718d4365b1f/eadc6d73-e2ad-4643-bc1f-3abdfd5d95f1"
-					(reference "R30")
+					(reference "R31")
 					(unit 1)
 				)
@@
 		(on_board yes)
 		(dnp no)
-		(property "Reference" "R31"
+		(property "Reference" "R32"
 			(at 92.71 75.438 0)
 			(effects
@@
 			(project ""
 				(path "/85c53e8c-0403-413d-b6c5-0718d4365b1f/eadc6d73-e2ad-4643-bc1f-3abdfd5d95f1"
-					(reference "R31")
+					(reference "R32")
 					(unit 1)
 				)
@@
 		(dnp no)
 		(fields_autoplaced yes)
-		(property "Reference" "#PWR074"
+		(property "Reference" "#PWR072"
 			(at 161.29 113.03 0)
 			(effects
@@
 			(project "System_Control"
 				(path "/85c53e8c-0403-413d-b6c5-0718d4365b1f/eadc6d73-e2ad-4643-bc1f-3abdfd5d95f1"
-					(reference "#PWR074")
+					(reference "#PWR072")
 					(unit 1)
 				)
@@
 		(on_board yes)
 		(dnp no)
-		(property "Reference" "R36"
+		(property "Reference" "R37"
 			(at 196.85 58.42 0)
 			(effects
@@
 			(project "System_Control"
 				(path "/85c53e8c-0403-413d-b6c5-0718d4365b1f/eadc6d73-e2ad-4643-bc1f-3abdfd5d95f1"
-					(reference "R36")
+					(reference "R37")
 					(unit 1)
 				)
@@
 		(on_board yes)
 		(dnp no)
-		(property "Reference" "D23"
+		(property "Reference" "D11"
 			(at 208.026 104.14 0)
 			(effects
@@
 			(project "System_Control"
 				(path "/85c53e8c-0403-413d-b6c5-0718d4365b1f/eadc6d73-e2ad-4643-bc1f-3abdfd5d95f1"
-					(reference "D23")
+					(reference "D11")
 					(unit 1)
 				)
@@
 		(on_board yes)
 		(dnp no)
-		(property "Reference" "R35"
+		(property "Reference" "R36"
 			(at 186.944 76.962 90)
 			(effects
@@
 			(project ""
 				(path "/85c53e8c-0403-413d-b6c5-0718d4365b1f/eadc6d73-e2ad-4643-bc1f-3abdfd5d95f1"
-					(reference "R35")
+					(reference "R36")
 					(unit 1)
 				)
@@
 		(on_board yes)
 		(dnp no)
-		(property "Reference" "R33"
+		(property "Reference" "R34"
 			(at 139.7 74.168 0)
 			(effects
@@
 			(project "System_Control"
 				(path "/85c53e8c-0403-413d-b6c5-0718d4365b1f/eadc6d73-e2ad-4643-bc1f-3abdfd5d95f1"
-					(reference "R33")
+					(reference "R34")
 					(unit 1)
 				)
@@
 		(dnp no)
 		(fields_autoplaced yes)
-		(property "Reference" "#PWR069"
+		(property "Reference" "#PWR067"
 			(at 69.85 82.55 0)
 			(effects
@@
 			(project "System_Control"
 				(path "/85c53e8c-0403-413d-b6c5-0718d4365b1f/eadc6d73-e2ad-4643-bc1f-3abdfd5d95f1"
-					(reference "#PWR069")
+					(reference "#PWR067")
 					(unit 1)
 				)
@@
 		(on_board yes)
 		(dnp no)
-		(property "Reference" "R34"
+		(property "Reference" "R35"
 			(at 139.7 81.788 0)
 			(effects
@@
 			(project "System_Control"
 				(path "/85c53e8c-0403-413d-b6c5-0718d4365b1f/eadc6d73-e2ad-4643-bc1f-3abdfd5d95f1"
-					(reference "R34")
+					(reference "R35")
 					(unit 1)
 				)
@@
 		(dnp no)
 		(fields_autoplaced yes)
-		(property "Reference" "#PWR079"
+		(property "Reference" "#PWR077"
 			(at 223.52 118.11 0)
 			(effects
@@
 			(project "System_Control"
 				(path "/85c53e8c-0403-413d-b6c5-0718d4365b1f/eadc6d73-e2ad-4643-bc1f-3abdfd5d95f1"
-					(reference "#PWR079")
-					(unit 1)
-				)
+					(reference "#PWR077")
+					(unit 1)
+				)
