File: Hardware/Source/System_Control/System_Control.kicad_pcb (KiCad board)
At the start: 4 copper layers, 100 x 100 mm, 507 parts, among them J1 POWER_CONN, J10 BAL_BAT_CONN2, J11 NTC_CONN, J12 NTC_CONN, J2 USB_B_Micro, J3 SIGNAL_CONN, J4 Conn_01x02_Socket, J5 FLASH_CONN, J6 Conn_01x02_Socket, J7 NTC_CONN, J8 NTC_CONN, J9 BAL_BAT_CONN1, Q1 MMBT2222A, Q10 AO3400A, Q11 AO3400A, Q12 AO3400A, Q13 AO3400A, Q14 AO3400A, Q15 AO3400A, Q16 AO3400A, Q17 AO3400A, Q18 AO3400A, Q19 AO3400A, Q2 MMBT2222A, Q20 AO3400A, Q21 MMBT2222A, Q22 SQJ211ELP-T1_GE3, Q23 SQJ211ELP-T1_GE3, Q24 MMBT2222A, Q3 MMBT2222A, Q4 MMBT2222A, Q5 AO3400A, Q6 AO3400A, Q7 AO3400A, Q8 AO3400A, Q9 AO3400A, SW1 SW_Push, SW2 SW_Push, SW3 SW_Push, U1 ESP32-WROOM-32U, U10 NE5532DR, U11 NE5532DR, U12 NE5532DR, U13 NE5532DR, U14 TLP291-4, U15 TLP291-4, U16 TLP291-4, U17 TLP291-4, U18 CD74HC4067SM96, U19 CD74HC4067SM96, U2 CH340C, U3 STM32F407VET6, U4 LCD 5“SSD1963, U5 MAX485CSA, U6 NE5532DR, U7 NE5532DR, U8 NE5532DR, U9 NE5532DR, Y1 Crystal_25MHz_SMD-4PIN

Commit message: check
Parts:
- removed the D10 at (161.8, 154.0)
- removed the D11 at (160.6, 146.7)
- removed the D12 at (162.3, 139.2)
- removed the D13 at (143.2, 127.9)
- removed the D14 at (143.5, 122.8)
- removed the D15 at (143.8, 115.8)
- removed the D16 at (161.8, 150.3)
- removed the D17 at (160.6, 142.9)
- removed the D18 at (141.2, 155.1)
- removed the D19 at (138.2, 128.1)
- removed the D20 at (138.3, 123.0)
- removed the D21 at (134.8, 109.2)
- removed the D22 at (159.6, 109.2)
- removed REF** (x2): Heat sink 14x14, charge_battery_footprint_lib:Heat sink 14x14
- removed the TP2 at (261.3, 102.7)
- removed the TP3 at (261.3, 105.8)
- removed the TP4 at (258.3, 96.6)
- removed TP5, TP6: TestPoint_Small, TestPoint:TestPoint_Pad_D1.0mm
- added D7: LED_0805, charge_battery_footprint_lib:LED_0805, B.Cu at (173.0, 91.5)
- added D8: LED_0805, charge_battery_footprint_lib:LED_0805, B.Cu at (175.0, 91.5)
- added R6: 1K/1%/1_10W, charge_battery_footprint_lib:Res_0603, B.Cu at (171.9, 90.0)
- added R9: 20R/1%/1_10W, charge_battery_footprint_lib:Res_0603, F.Cu at (193.1, 96.5)
- R7: value 20R/5%/1_16W -> 1K/1%/1_10W; footprint charge_battery_footprint_lib:Res_0402 -> charge_battery_footprint_lib:Res_0603; moved to B.Cu
- R8: value 20R/5%/1_16W -> 20R/1%/1_10W; footprint charge_battery_footprint_lib:Res_0402 -> charge_battery_footprint_lib:Res_0603
- TP1: value TestPoint_Small -> GND
- moved TP1 94.9 mm to (217.4, 183.8)
- moved TP2 65.1 mm to (175.3, 114.2)
- moved D63 52.0 mm to (181.9, 143.8), turned to 180 degrees
- moved TP3 48.9 mm to (173.0, 112.8)
- moved R27 42.8 mm to (179.0, 116.7), turned to -90 degrees
- moved R28 42.1 mm to (175.6, 116.7), turned to -90 degrees
- moved D9 41.3 mm to (176.7, 118.2), turned to -90 degrees
- moved D10 41.1 mm to (173.3, 118.2), turned to -90 degrees
- moved R7 14.8 mm to (177.3, 90.0)
- moved C10 11.7 mm to (241.0, 104.9)
- moved C7 11.0 mm to (230.7, 104.9), turned to 180 degrees
- moved C9 8.00 mm to (230.7, 102.6), turned to 180 degrees
- moved C8 7.18 mm to (241.0, 102.6)
- moved R5 6.13 mm to (244.7, 104.9)
- moved D5 6.12 mm to (249.3, 105.5)
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- renumbered D9 to D10, D23 to D11, D24 to D12, D25 to D13, D26 to D14, D27 to D15, D28 to D16, D29 to D17, D30 to D18, D31 to D19, D32 to D20, D33 to D21, D34 to D22, D35 to D23, D36 to D24, D37 to D25, D38 to D26, D39 to D27, D40 to D28, D41 to D29, D42 to D30, D43 to D31, D44 to D32, D45 to D33, D46 to D34, D47 to D35, D48 to D36, D49 to D37, D50 to D38, D51 to D39, D52 to D40, D53 to D41, D54 to D42, D55 to D43, D56 to D44, D57 to D45, D58 to D46, D59 to D47, D60 to D48, D61 to D49, D62 to D50, D63 to D51, D64 to D52, D65 to D53, D66 to D54, D67 to D55, D68 to D56, D69 to D57, D70 to D58, D71 to D59, D72 to D60, D73 to D61, D74 to D62, D75 to D63, D8 to D9, R9 to R10, R99 to R100, R100 to R101, R101 to R102, R102 to R103, R103 to R104, R104 to R105, R105 to R106, R106 to R107, R107 to R108, R108 to R109, R10 to R11, R109 to R110, R110 to R111, R111 to R112, R112 to R113, R113 to R114, R114 to R115, R115 to R116, R116 to R117, R117 to R118, R118 to R119, R11 to R12, R119 to R120, R120 to R121, R121 to R122, R122 to R123, R123 to R124, R124 to R125, R125 to R126, R126 to R127, R127 to R128, R128 to R129, R12 to R13, R129 to R130, R130 to R131, R131 to R132, R132 to R133, R133 to R134, R134 to R135, R135 to R136, R136 to R137, R137 to R138, R138 to R139, R13 to R14, R139 to R140, R140 to R141, R141 to R142, R142 to R143, R143 to R144, R144 to R145, R145 to R146, R146 to R147, R147 to R148, R148 to R149, R14 to R15, R149 to R150, R150 to R151, R151 to R152, R152 to R153, R153 to R154, R154 to R155, R155 to R156, R156 to R157, R157 to R158, R158 to R159, R15 to R16, R159 to R160, R160 to R161, R161 to R162, R162 to R163, R163 to R164, R164 to R165, R165 to R166, R166 to R167, R167 to R168, R168 to R169, R16 to R17, R169 to R170, R170 to R171, R171 to R172, R172 to R173, R173 to R174, R174 to R175, R175 to R176, R176 to R177, R177 to R178, R178 to R179, R17 to R18, R179 to R180, R180 to R181, R181 to R182, R182 to R183, R183 to R184, R184 to R185, R185 to R186, R186 to R187, R187 to R188, R188 to R189, R18 to R19, R189 to R190, R190 to R191, R191 to R192, R192 to R193, R193 to R194, R194 to R195, R195 to R196, R196 to R197, R197 to R198, R198 to R199, R19 to R20, R199 to R200, R200 to R201, R201 to R202, R202 to R203, R203 to R204, R20 to R21, R21 to R22, R22 to R23, R23 to R24, R24 to R25, R25 to R26, R26 to R27, R27 to R28, R28 to R29, R29 to R30, R30 to R31, R31 to R32, R32 to R33, R33 to R34, R34 to R35, R35 to R36, R36 to R37, R37 to R38, R38 to R39, R39 to R40, R40 to R41, R41 to R42, R42 to R43, R43 to R44, R44 to R45, R45 to R46, R46 to R47, R47 to R48, R48 to R49, R49 to R50, R50 to R51, R51 to R52, R52 to R53, R53 to R54, R54 to R55, R55 to R56, R56 to R57, R57 to R58, R58 to R59, R59 to R60, R60 to R61, R61 to R62, R62 to R63, R63 to R64, R64 to R65, R65 to R66, R66 to R67, R67 to R68, R68 to R69, R69 to R70, R70 to R71, R71 to R72, R72 to R73, R73 to R74, R74 to R75, R75 to R76, R76 to R77, R77 to R78, R78 to R79, R79 to R80, R80 to R81, R81 to R82, R82 to R83, R83 to R84, R84 to R85, R85 to R86, R86 to R87, R87 to R88, R88 to R89, R89 to R90, R90 to R91, R91 to R92, R92 to R93, R93 to R94, R94 to R95, R95 to R96, R96 to R97, R97 to R98, R98 to R99, TP7 to TP2, TP8 to TP3, TP9 to TP4
Connections:
- net UART2_RX renamed UART5_RX
- net UART2_TX renamed UART5_TX
- C100 pad 2: NTC_1+ -> +3V3_O
- C101 pad 2: NTC_1+ -> +3V3_O
- C102 pad 2: NTC_1+ -> +3V3_O
- C103 pad 2: NTC_1+ -> +3V3_O
- C104 pad 2: NTC_1+ -> +3V3_O
- C105 pad 2: NTC_1+ -> +3V3_O
- C155 pad 2: VBAT -> +3V3_O
- C156 pad 2: VBAT -> +3V3_O
- C158 pad 2: VBAT -> +3V3_O
- C159 pad 2: VBAT -> +3V3_O
- C36 pad 2: +3V3_D -> +3V3_O
- C37 pad 2: +3V3_D -> +3V3_O
- C42 pad 2: NTC_1+ -> +3V3_O
- C43 pad 2: NTC_1+ -> +3V3_O
- C44 pad 2: NTC_1+ -> +3V3_O
- C45 pad 2: NTC_1+ -> +3V3_O
- C46 pad 2: NTC_1+ -> +3V3_O
- C47 pad 2: NTC_1+ -> +3V3_O
- C48 pad 2: NTC_1+ -> +3V3_O
- C49 pad 2: NTC_1+ -> +3V3_O
- C50 pad 2: NTC_1+ -> +3V3_O
- C51 pad 2: NTC_1+ -> +3V3_O
- C52 pad 2: NTC_1+ -> +3V3_O
- C53 pad 2: NTC_1+ -> +3V3_O
- C54 pad 2: NTC_1+ -> +3V3_O
- C55 pad 2: NTC_1+ -> +3V3_O
- C56 pad 2: NTC_1+ -> +3V3_O
- C57 pad 2: NTC_1+ -> +3V3_O
- C7 pad 1: +3V3_D -> +3V3_O
- C9 pad 1: +3V3_D -> +3V3_O
- C90 pad 2: NTC_1+ -> +3V3_O
- C91 pad 2: NTC_1+ -> +3V3_O
- C92 pad 2: NTC_1+ -> +3V3_O
- C93 pad 2: NTC_1+ -> +3V3_O
- C94 pad 2: NTC_1+ -> +3V3_O
- C95 pad 2: NTC_1+ -> +3V3_O
- C96 pad 2: NTC_1+ -> +3V3_O
- C97 pad 2: NTC_1+ -> +3V3_O
- C98 pad 2: NTC_1+ -> +3V3_O
- C99 pad 2: NTC_1+ -> +3V3_O
- D63 pad 1: Net-(J5-Pin_2) -> Net-(J5-Pin_3)
- D63 pad 2: Net-(J5-Pin_3) -> Net-(J5-Pin_2)
- J1 pad 4: +3V3_D -> +3V3_O
- J11 pad 1: NTC_1+ -> +3V3_O
- J11 pad 3: NTC_1+ -> +3V3_O
- J11 pad 5: NTC_1+ -> +3V3_O
- J11 pad 7: NTC_1+ -> +3V3_O
- J12 pad 1: NTC_1+ -> +3V3_O
- J12 pad 3: NTC_1+ -> +3V3_O
- J12 pad 5: NTC_1+ -> +3V3_O
- J12 pad 7: NTC_1+ -> +3V3_O
- J7 pad 2: NTC_1+ -> +3V3_O
- J7 pad 4: NTC_1+ -> +3V3_O
- J7 pad 6: NTC_1+ -> +3V3_O
- J7 pad 8: NTC_1+ -> +3V3_O
- J8 pad 2: NTC_1+ -> +3V3_O
- J8 pad 4: NTC_1+ -> +3V3_O
- J8 pad 6: NTC_1+ -> +3V3_O
- J8 pad 8: NTC_1+ -> +3V3_O
- R30 pad 2: +3V3_D -> +3V3_O
- R4 pad 1: +3V3_D -> +3V3_O
- R47 pad 2: NTC_1+ -> +3V3_O
- R48 pad 2: NTC_1+ -> +3V3_O
- R49 pad 2: NTC_1+ -> +3V3_O
- R50 pad 2: NTC_1+ -> +3V3_O
- R59 pad 2: NTC_1+ -> +3V3_O
- R60 pad 2: NTC_1+ -> +3V3_O
- R61 pad 2: NTC_1+ -> +3V3_O
- R62 pad 2: NTC_1+ -> +3V3_O
- R7 pad 1: /ESP32/D_P -> Net-(D8-K)
- R7 pad 2: /ESP32/U_P -> GNDA
- R71 pad 2: NTC_1+ -> +3V3_O
- R72 pad 2: NTC_1+ -> +3V3_O
- R73 pad 2: NTC_1+ -> +3V3_O
- R74 pad 2: NTC_1+ -> +3V3_O
- R8 pad 1: /ESP32/D_N -> /ESP32/D_P
- R8 pad 2: /ESP32/U_N -> /ESP32/U_P
- R83 pad 2: NTC_1+ -> +3V3_O
- R84 pad 2: NTC_1+ -> +3V3_O
- R85 pad 2: NTC_1+ -> +3V3_O
- R86 pad 2: NTC_1+ -> +3V3_O
- TP1 pad 1: +5V -> GNDA
- U1 pad 31: unconnected-(U1-IO19-Pad31) -> /ESP32/LED_TEST
- U1 pad 33: unconnected-(U1-IO21-Pad33) -> /ESP32/LED_STATUS
- U18 pad 24: VBAT -> +3V3_O
- U19 pad 24: VBAT -> +3V3_O
- U3 pad 15: ADC1_IN1_S0 -> /STM32F407VET6/LED_TEST
- U3 pad 16: ADC1_IN1_S1 -> /STM32F407VET6/LED_STATUS
- U3 pad 7: unconnected-(U3A-PC13-Pad7) -> ADC1_IN1_S0
- U3 pad 8: unconnected-(U3A-PC14-Pad8) -> ADC1_IN1_S1
Routing:
- net +3V3_O: track 0.00 -> 687.1 mm, vias 0 -> 35
- net GNDA: track 81.6 -> 483.1 mm, vias 15 -> 307
- net VBAT: track 33.0 -> 318.7 mm, vias 1 -> 19
- net +5V: track 5.92 -> 170.4 mm, vias 0 -> 7
- net +3V3_D: track 84.2 -> 0.00 mm, vias 1 -> 0
- net -9V: track 135.7 -> 212.7 mm, vias 4 -> 10
- net NTC_1+: track 52.4 -> 0.00 mm, vias 5 -> 0
- net +9V: track 151.8 -> 177.2 mm, vias 6 -> 10
- net /ESP32/LED_TEST: track 0.00 -> 20.8 mm, vias 0 -> 1
- net RS485_P: track 6.06 -> 24.9 mm
- net RS485_N: track 6.10 -> 24.2 mm
- net /ESP32/LED_STATUS: track 0.00 -> 14.9 mm, vias 0 -> 1
- net FSMC_D15: track 44.3 -> 32.4 mm
- net FSMC_D13: track 42.9 -> 32.3 mm
- net FSMC_D11: track 44.4 -> 33.9 mm, vias 1 -> 0
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- added copper zone on B.Cu, net +3V3_O
- added copper zone on In2.Cu, net +3V3_O
- added copper zone on B.Cu, net +5V
- added copper zone on In2.Cu, net +5V
- added copper zone on B.Cu, net +9V
- added copper zone on In2.Cu, net +9V
- added copper zone on B.Cu, net -9V
- added copper zone on In2.Cu, net -9V
- added copper zone on F.Cu, net GNDA
- added copper zone on B.Cu, net Net-(D22-A)
- added copper zone on B.Cu, net Net-(D23-A)
- added copper zone on B.Cu, net Net-(D26-A)
- added copper zone on B.Cu, net Net-(D27-A)
- added copper zone on B.Cu, net Net-(D30-A)
- added copper zone on B.Cu, net Net-(D31-A)
- added copper zone on B.Cu, net Net-(D34-A)
- added copper zone on B.Cu, net Net-(D46-A)
- added copper zone on B.Cu, net Net-(D47-A)
- added copper zone on B.Cu, net Net-(D50-A)
- added copper zone on B.Cu, net Net-(D54-A)
- added copper zone on B.Cu, net Net-(D55-A)
- added copper zone on B.Cu, net Net-(D58-A)
- added copper zone on B.Cu, net VBAT
- added copper zone on F.Cu, net VBAT
- added copper zone on In2.Cu, net VBAT
- added copper zone on F.Cu, net VDDA
Other:
- outline, holes or cut-outs redrawn
- board text added: "+5V"
- board text added: "+9V"
- board text added: "-9V"
- board text added: "1"
- board text added: "10"
- board text added: "11"
- board text added: "12"
- board text added: "13"
- board text added: "14"
- board text added: "15"
- board text added: "16"
- board text added: "2"
- board text added: "3"
- board text added: "3V3"
- board text added: "4"
- board text added: "5"
- board text added: "6"
- board text added: "7"
- board text added: "8"
- board text added: "9"
- board text added: "A"
- board text added: "B"
- board text added: "GND"
- board text added: "NTC"
- board text added: "RX"
- board text added: "TX"

Commit message: check
Parts:
- SW1: value SW_Push -> FLASH
- SW2: value SW_Push -> EN
- SW3: value SW_Push -> RST
- moved C2 12.3 mm to (215.7, 102.9)
- moved C1 8.23 mm to (215.7, 100.6)
Routing:
- net +5V: track 170.4 -> 160.1 mm, vias 7 -> 8
- net GNDA: vias 307 -> 301
- net (no net): vias 0 -> 24
Other:
- board text added: "->"
- board text added: "BALLANCE"
- board text added: "DISPLAY"
- board text added: "IN"
- board text added: "OUT"

Commit message: check
Parts:
- SW1: value FLASH -> SW_Push
- SW2: value EN -> SW_Push
- SW3: value RST -> SW_Push
Connections:
- U3 pad 87: FSMC_RESET -> unconnected-(U3A-PD6-Pad87)
- U4 pad 7: FSMC_RESET -> unconnected-(U4-E/RESET_NC-Pad7)
Routing:
- net FSMC_RESET: track 32.4 -> 0.00 mm, vias 1 -> 0
- net GNDA: vias 301 -> 304
