File: Hardware/Source/System_Control/ESP32.kicad_sch (KiCad schematic)
At the start: 28 parts, among them J2 USB_B_Micro, Q1 MMBT2222A, Q2 MMBT2222A, SW1 SW_Push, SW2 SW_Push, U1 ESP32-WROOM-32U, U2 CH340C

Commit message: footprint:lib:update header xh2.54 8pin smd
Parts:
- renumbered R11 to R10, R10 to R11, R9 to R8, R8 to R9
Connections:
- net U_N: now reaches R10.1, U2.6 (UD-)
- net U_P: now reaches R8.2, U2.5 (UD+)
- net at J2.1 (VBUS), R7.1: no longer D7.5
- no-connect marks 33 -> 34
Other:
- moved on the sheet: R10, R8
Changed lines of the file:
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@@
 	)
 	(junction
-		(at 71.12 22.86)
-		(diameter 0)
-		(color 0 0 0 0)
-	)
-	(junction
 		(at 55.88 27.94)
 		(diameter 0)
@@
 	)
 	(no_connect
+		(at 71.12 34.29)
+	)
+	(no_connect
 		(at 64.77 113.03)
 	)
@@
 	(wire
 		(pts
-			(xy 123.19 36.83) (xy 119.38 36.83)
+			(xy 123.19 36.83) (xy 114.3 36.83)
 		)
 		(stroke
@@
 	(wire
 		(pts
-			(xy 123.19 34.29) (xy 119.38 34.29)
+			(xy 123.19 34.29) (xy 114.3 34.29)
 		)
 		(stroke
@@
 	(wire
 		(pts
-			(xy 102.87 34.29) (xy 111.76 34.29)
+			(xy 97.79 34.29) (xy 106.68 34.29)
 		)
 		(stroke
@@
 	(wire
 		(pts
-			(xy 102.87 36.83) (xy 111.76 36.83)
+			(xy 97.79 36.83) (xy 106.68 36.83)
 		)
 		(stroke
@@
 	(wire
 		(pts
-			(xy 52.07 22.86) (xy 71.12 22.86)
-		)
-		(stroke
-			(width 0)
-			(type default)
-		)
-	)
-	(wire
-		(pts
 			(xy 40.64 91.44) (xy 40.64 92.71)
 		)
@@
 	(wire
 		(pts
-			(xy 71.12 22.86) (xy 78.74 22.86)
+			(xy 52.07 22.86) (xy 78.74 22.86)
 		)
 		(stroke
@@
 	(wire
 		(pts
-			(xy 71.12 22.86) (xy 71.12 34.29)
-		)
-		(stroke
-			(width 0)
-			(type default)
-		)
-	)
-	(wire
-		(pts
 			(xy 165.1 44.45) (xy 157.48 44.45)
 		)
@@
 	)
 	(label "D_N"
-		(at 102.87 36.83 0)
+		(at 97.79 36.83 0)
+		(fields_autoplaced yes)
+		(effects
+			(font
+				(size 1.27 1.27)
+			)
+			(justify left bottom)
+		)
+	)
+	(label "U_N"
+		(at 118.11 36.83 0)
 		(fields_autoplaced yes)
 		(effects
@@
 		)
 	)
+	(label "U_P"
+		(at 118.11 34.29 0)
+		(fields_autoplaced yes)
+		(effects
+			(font
+				(size 1.27 1.27)
+			)
+			(justify left bottom)
+		)
+	)
 	(label "D_P"
-		(at 102.87 34.29 0)
+		(at 97.79 34.29 0)
 		(fields_autoplaced yes)
 		(effects
@@
 		(lib_name "Res_20R_0603_1%_3")
 		(lib_id "charge_battery_sym_lib:Res_20R_0603_1%")
-		(at 119.38 36.83 0)
+		(at 114.3 36.83 0)
 		(mirror y)
 		(unit 1)
@@
 		(on_board yes)
 		(dnp no)
-		(property "Reference" "R11"
-			(at 115.57 39.116 0)
+		(property "Reference" "R10"
+			(at 110.49 39.116 0)
 			(effects
 				(font
@@
 		)
 		(property "Value" "20R/1%/1_10W"
-			(at 116.078 40.894 0)
+			(at 110.998 40.894 0)
 			(effects
 				(font
@@
 		)
 		(property "Footprint" "charge_battery_footprint_lib:Res_0603"
-			(at 79.502 25.4 90)
+			(at 74.422 25.4 90)
 			(effects
 				(font
@@
 		)
 		(property "Datasheet" "https://fscdn.rohm.com/en/products/databook/datasheet/passive/resistor/chip_resistor/esr-e.pdf"
-			(at 79.756 36.068 90)
+			(at 74.676 36.068 90)
 			(effects
 				(font
@@
 		)
 		(property "Description" "Res 20 Ohm 0603 1%"
-			(at 78.994 29.972 90)
+			(at 73.914 29.972 90)
 			(effects
 				(font
@@
 		)
 		(property "Supply name" "Thegioiic"
-			(at 79.248 24.384 90)
+			(at 74.168 24.384 90)
 			(effects
 				(font
@@
 		)
 		(property "Supply part number" "Điện Trở 20 Ohm 0603 1%"
-			(at 79.502 23.368 90)
+			(at 74.422 23.368 90)
 			(effects
 				(font
@@
 		)
 		(property "Supply URL" "https://www.thegioiic.com/dien-tro-20-ohm-0603-1-"
-			(at 78.232 16.256 90)
+			(at 73.152 16.256 90)
 			(effects
 				(font
@@
 			(project "System_Control"
 				(path "/85c53e8c-0403-413d-b6c5-0718d4365b1f/bc09c168-950d-49ef-aa8a-d95b0b1387ca"
-					(reference "R11")
+					(reference "R10")
 					(unit 1)
 				)
@@
 		(lib_name "Res_20R_0603_1%_3")
 		(lib_id "charge_battery_sym_lib:Res_20R_0603_1%")
-		(at 111.76 34.29 0)
+		(at 106.68 34.29 0)
 		(unit 1)
 		(exclude_from_sim no)
@@
 		(on_board yes)
 		(dnp no)
-		(property "Reference" "R9"
-			(at 115.57 29.718 0)
+		(property "Reference" "R8"
+			(at 110.49 29.718 0)
 			(effects
 				(font
@@
 		)
 		(property "Value" "20R/1%/1_10W"
-			(at 115.316 32.004 0)
+			(at 110.236 32.004 0)
 			(effects
 				(font
@@
 		)
 		(property "Footprint" "charge_battery_footprint_lib:Res_0603"
-			(at 151.638 22.86 90)
+			(at 146.558 22.86 90)
 			(effects
 				(font
@@
 		)
 		(property "Datasheet" "https://fscdn.rohm.com/en/products/databook/datasheet/passive/resistor/chip_resistor/esr-e.pdf"
-			(at 151.384 33.528 90)
+			(at 146.304 33.528 90)
 			(effects
 				(font
@@
 		)
 		(property "Description" "Res 20 Ohm 0603 1%"
-			(at 152.146 27.432 90)
+			(at 147.066 27.432 90)
 			(effects
 				(font
@@
 		)
 		(property "Supply name" "Thegioiic"
-			(at 151.892 21.844 90)
+			(at 146.812 21.844 90)
 			(effects
 				(font
@@
 		)
 		(property "Supply part number" "Điện Trở 20 Ohm 0603 1%"
-			(at 151.638 20.828 90)
+			(at 146.558 20.828 90)
 			(effects
 				(font
@@
 		)
 		(property "Supply URL" "https://www.thegioiic.com/dien-tro-20-ohm-0603-1-"
-			(at 152.908 13.716 90)
+			(at 147.828 13.716 90)
 			(effects
 				(font
@@
 			(project "System_Control"
 				(path "/85c53e8c-0403-413d-b6c5-0718d4365b1f/bc09c168-950d-49ef-aa8a-d95b0b1387ca"
-					(reference "R9")
+					(reference "R8")
 					(unit 1)
 				)
@@
 		(on_board yes)
 		(dnp no)
-		(property "Reference" "R10"
+		(property "Reference" "R11"
 			(at 111.76 91.186 0)
 			(effects
@@
 			(project "System_Control"
 				(path "/85c53e8c-0403-413d-b6c5-0718d4365b1f/bc09c168-950d-49ef-aa8a-d95b0b1387ca"
-					(reference "R10")
+					(reference "R11")
 					(unit 1)
 				)
@@
 		(on_board yes)
 		(dnp no)
-		(property "Reference" "R8"
+		(property "Reference" "R9"
 			(at 111.76 81.788 0)
 			(effects
@@
 			(project "System_Control"
 				(path "/85c53e8c-0403-413d-b6c5-0718d4365b1f/bc09c168-950d-49ef-aa8a-d95b0b1387ca"
-					(reference "R8")
+					(reference "R9")
 					(unit 1)
 				)

Commit message: pull
Parts:
- renumbered C13 to C11, C14 to C12, C15 to C13, C16 to C14, C17 to C15, C18 to C16, C19 to C17
Changed lines of the file:
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@@
 		(dnp no)
 		(fields_autoplaced yes)
-		(property "Reference" "#PWR031"
+		(property "Reference" "#PWR028"
 			(at 40.64 107.95 0)
 			(effects
@@
 			(project "System_Control"
 				(path "/85c53e8c-0403-413d-b6c5-0718d4365b1f/bc09c168-950d-49ef-aa8a-d95b0b1387ca"
-					(reference "#PWR031")
+					(reference "#PWR028")
 					(unit 1)
 				)
@@
 		(dnp no)
 		(fields_autoplaced yes)
-		(property "Reference" "#PWR032"
+		(property "Reference" "#PWR029"
 			(at 44.45 45.72 0)
 			(effects
@@
 			(project "System_Control"
 				(path "/85c53e8c-0403-413d-b6c5-0718d4365b1f/bc09c168-950d-49ef-aa8a-d95b0b1387ca"
-					(reference "#PWR032")
+					(reference "#PWR029")
 					(unit 1)
 				)
@@
 		(on_board yes)
 		(dnp no)
-		(property "Reference" "#PWR041"
+		(property "Reference" "#PWR038"
 			(at 166.37 22.86 0)
 			(effects
@@
 			(project "System_Control"
 				(path "/85c53e8c-0403-413d-b6c5-0718d4365b1f/bc09c168-950d-49ef-aa8a-d95b0b1387ca"
-					(reference "#PWR041")
+					(reference "#PWR038")
 					(unit 1)
 				)
@@
 		(dnp no)
 		(fields_autoplaced yes)
-		(property "Reference" "#PWR042"
+		(property "Reference" "#PWR039"
 			(at 166.37 38.1 0)
 			(effects
@@
 			(project "System_Control"
 				(path "/85c53e8c-0403-413d-b6c5-0718d4365b1f/bc09c168-950d-49ef-aa8a-d95b0b1387ca"
-					(reference "#PWR042")
+					(reference "#PWR039")
 					(unit 1)
 				)
@@
 		(dnp no)
 		(fields_autoplaced yes)
-		(property "Reference" "#PWR046"
+		(property "Reference" "#PWR043"
 			(at 186.69 149.86 0)
 			(effects
@@
 			(project "System_Control"
 				(path "/85c53e8c-0403-413d-b6c5-0718d4365b1f/bc09c168-950d-49ef-aa8a-d95b0b1387ca"
-					(reference "#PWR046")
+					(reference "#PWR043")
 					(unit 1)
 				)
@@
 		(dnp no)
 		(fields_autoplaced yes)
-		(property "Reference" "#PWR030"
+		(property "Reference" "#PWR027"
 			(at 40.64 93.98 0)
 			(effects
@@
 			(project "System_Control"
 				(path "/85c53e8c-0403-413d-b6c5-0718d4365b1f/bc09c168-950d-49ef-aa8a-d95b0b1387ca"
-					(reference "#PWR030")
+					(reference "#PWR027")
 					(unit 1)
 				)
@@
 		(dnp no)
 		(fields_autoplaced yes)
-		(property "Reference" "#PWR040"
+		(property "Reference" "#PWR037"
 			(at 157.48 20.32 0)
 			(effects
@@
 			(project "System_Control"
 				(path "/85c53e8c-0403-413d-b6c5-0718d4365b1f/bc09c168-950d-49ef-aa8a-d95b0b1387ca"
-					(reference "#PWR040")
+					(reference "#PWR037")
 					(unit 1)
 				)
@@
 		(dnp no)
 		(fields_autoplaced yes)
-		(property "Reference" "#PWR033"
+		(property "Reference" "#PWR030"
 			(at 66.04 50.8 0)
 			(effects
@@
 			(project "System_Control"
 				(path "/85c53e8c-0403-413d-b6c5-0718d4365b1f/bc09c168-950d-49ef-aa8a-d95b0b1387ca"
-					(reference "#PWR033")
+					(reference "#PWR030")
 					(unit 1)
 				)
@@
 		(on_board yes)
 		(dnp no)
-		(property "Reference" "C19"
+		(property "Reference" "C17"
 			(at 176.53 24.892 90)
 			(effects
@@
 			(project "System_Control"
 				(path "/85c53e8c-0403-413d-b6c5-0718d4365b1f/bc09c168-950d-49ef-aa8a-d95b0b1387ca"
-					(reference "C19")
+					(reference "C17")
 					(unit 1)
 				)
@@
 		(dnp no)
 		(fields_autoplaced yes)
-		(property "Reference" "#PWR043"
+		(property "Reference" "#PWR040"
 			(at 186.69 83.82 0)
 			(effects
@@
 			(project "System_Control"
 				(path "/85c53e8c-0403-413d-b6c5-0718d4365b1f/bc09c168-950d-49ef-aa8a-d95b0b1387ca"
-					(reference "#PWR043")
+					(reference "#PWR040")
 					(unit 1)
 				)
@@
 		(dnp no)
 		(fields_autoplaced yes)
-		(property "Reference" "#PWR036"
+		(property "Reference" "#PWR033"
 			(at 105.41 22.86 0)
 			(effects
@@
 			(project "System_Control"
 				(path "/85c53e8c-0403-413d-b6c5-0718d4365b1f/bc09c168-950d-49ef-aa8a-d95b0b1387ca"
-					(reference "#PWR036")
+					(reference "#PWR033")
 					(unit 1)
 				)
@@
 		(on_board yes)
 		(dnp no)
-		(property "Reference" "C16"
+		(property "Reference" "C14"
 			(at 166.37 24.892 90)
 			(effects
@@
 			(project "System_Control"
 				(path "/85c53e8c-0403-413d-b6c5-0718d4365b1f/bc09c168-950d-49ef-aa8a-d95b0b1387ca"
-					(reference "C16")
+					(reference "C14")
 					(unit 1)
 				)
@@
 		(on_board yes)
 		(dnp no)
-		(property "Reference" "#PWR037"
+		(property "Reference" "#PWR034"
 			(at 130.81 24.13 0)
 			(effects
@@
 			(project "System_Control"
 				(path "/85c53e8c-0403-413d-b6c5-0718d4365b1f/bc09c168-950d-49ef-aa8a-d95b0b1387ca"
-					(reference "#PWR037")
+					(reference "#PWR034")
 					(unit 1)
 				)
@@
 		(dnp no)
 		(fields_autoplaced yes)
-		(property "Reference" "#PWR045"
+		(property "Reference" "#PWR042"
 			(at 186.69 123.19 0)
 			(effects
@@
 			(project "System_Control"
 				(path "/85c53e8c-0403-413d-b6c5-0718d4365b1f/bc09c168-950d-49ef-aa8a-d95b0b1387ca"
-					(reference "#PWR045")
+					(reference "#PWR042")
 					(unit 1)
 				)
@@
 		(dnp no)
 		(fields_autoplaced yes)
-		(property "Reference" "#PWR044"
+		(property "Reference" "#PWR041"
 			(at 186.69 110.49 0)
 			(effects
@@
 			(project "System_Control"
 				(path "/85c53e8c-0403-413d-b6c5-0718d4365b1f/bc09c168-950d-49ef-aa8a-d95b0b1387ca"
-					(reference "#PWR044")
+					(reference "#PWR041")
 					(unit 1)
 				)
@@
 		(dnp no)
 		(fields_autoplaced yes)
-		(property "Reference" "#PWR035"
+		(property "Reference" "#PWR032"
 			(at 80.01 154.94 0)
 			(effects
@@
 			(project "System_Control"
 				(path "/85c53e8c-0403-413d-b6c5-0718d4365b1f/bc09c168-950d-49ef-aa8a-d95b0b1387ca"
-					(reference "#PWR035")
+					(reference "#PWR032")
 					(unit 1)
 				)
@@
 		(on_board yes)
 		(dnp no)
-		(property "Reference" "C14"
+		(property "Reference" "C12"
 			(at 50.8 94.742 90)
 			(effects
@@
 			(project "System_Control"
 				(path "/85c53e8c-0403-413d-b6c5-0718d4365b1f/bc09c168-950d-49ef-aa8a-d95b0b1387ca"
-					(reference "C14")
+					(reference "C12")
 					(unit 1)
 				)
@@
 		(dnp no)
 		(fields_autoplaced yes)
-		(property "Reference" "#PWR039"
+		(property "Reference" "#PWR036"
 			(at 142.24 110.49 0)
 			(effects
@@
 			(project "System_Control"
 				(path "/85c53e8c-0403-413d-b6c5-0718d4365b1f/bc09c168-950d-49ef-aa8a-d95b0b1387ca"
-					(reference "#PWR039")
+					(reference "#PWR036")
 					(unit 1)
 				)
@@
 		(on_board yes)
 		(dnp no)
-		(property "Reference" "C18"
+		(property "Reference" "C16"
 			(at 173.99 134.112 90)
 			(effects
@@
 			(project "System_Control"
 				(path "/85c53e8c-0403-413d-b6c5-0718d4365b1f/bc09c168-950d-49ef-aa8a-d95b0b1387ca"
-					(reference "C18")
+					(reference "C16")
 					(unit 1)
 				)
@@
 		(dnp no)
 		(fields_autoplaced yes)
-		(property "Reference" "C15"
+		(property "Reference" "C13"
 			(at 146.05 13.97 0)
 			(effects
@@
 			(project "System_Control"
 				(path "/85c53e8c-0403-413d-b6c5-0718d4365b1f/bc09c168-950d-49ef-aa8a-d95b0b1387ca"
-					(reference "C15")
+					(reference "C13")
 					(unit 1)
 				)
@@
 		(dnp no)
 		(fields_autoplaced yes)
-		(property "Reference" "#PWR034"
+		(property "Reference" "#PWR031"
 			(at 80.01 80.01 0)
 			(effects
@@
 			(project "System_Control"
 				(path "/85c53e8c-0403-413d-b6c5-0718d4365b1f/bc09c168-950d-49ef-aa8a-d95b0b1387ca"
-					(reference "#PWR034")
+					(reference "#PWR031")
 					(unit 1)
 				)
@@
 		(on_board yes)
 		(dnp no)
-		(property "Reference" "C13"
+		(property "Reference" "C11"
 			(at 40.64 94.742 90)
 			(effects
@@
 			(project "System_Control"
 				(path "/85c53e8c-0403-413d-b6c5-0718d4365b1f/bc09c168-950d-49ef-aa8a-d95b0b1387ca"
-					(reference "C13")
+					(reference "C11")
 					(unit 1)
 				)
@@
 		(on_board yes)
 		(dnp no)
-		(property "Reference" "C17"
+		(property "Reference" "C15"
 			(at 173.99 94.742 90)
 			(effects
@@
 			(project "System_Control"
 				(path "/85c53e8c-0403-413d-b6c5-0718d4365b1f/bc09c168-950d-49ef-aa8a-d95b0b1387ca"
-					(reference "C17")
+					(reference "C15")
 					(unit 1)
 				)
@@
 		(dnp no)
 		(fields_autoplaced yes)
-		(property "Reference" "#PWR038"
+		(property "Reference" "#PWR035"
 			(at 133.35 58.42 0)
 			(effects
@@
 			(project "System_Control"
 				(path "/85c53e8c-0403-413d-b6c5-0718d4365b1f/bc09c168-950d-49ef-aa8a-d95b0b1387ca"
-					(reference "#PWR038")
+					(reference "#PWR035")
 					(unit 1)
 				)

Commit message: check
Parts:
- removed D8: LED_0805, charge_battery_footprint_lib:LED_0805, symbol charge_battery_sym_lib:LED_0805
- removed R10, R11, R13, R14, R8, R9: 20R/1%/1_10W, charge_battery_footprint_lib:Res_0603, symbol charge_battery_sym_lib:Res_20R_0603_1%
- removed R7: 1K/1%/1_10W, charge_battery_footprint_lib:Res_0603, symbol charge_battery_sym_lib:Res_1K_0603_1%
- added R10, R12, R13, R7, R8, R9: 20R/5%/1_16W, charge_battery_footprint_lib:Res_0402, symbol charge_battery_sym_lib:Res_20R_0402_5%
- renumbered D7 to D6, R12 to R11, R15 to R14, R16 to R15, R17 to R16, R18 to R17
Connections:
- net CONTROL_BOOT0: now also U1.16 (IO13); no longer U1.30 (IO18)
- net CONTROL_BOOT1: now also U1.14 (IO12); no longer U1.31 (IO19)
- net DIR: now also R12.2
- net D_N: now also R8.1
- net D_P: now also R7.1
- net RTS: now also R13.2
- net U0_N: now also R10.2
- net U0_P: now also R9.2
- net U_N: now also R8.2
- net U_P: now also R7.2
- net at U1.34 (RXD0/IO3): now also R10.1
- net at U1.35 (TXD0/IO1): now also R9.1
- net at U2.13 (~{DTR}): now also R12.1
- net at U2.14 (~{RTS}): now also R13.1
- no-connect marks 34 -> 35

Commit message: check
Parts:
- removed R7, R8: 20R/5%/1_16W, charge_battery_footprint_lib:Res_0402, symbol charge_battery_sym_lib:Res_20R_0402_5%
- added D7, D8: LED_0805, charge_battery_footprint_lib:LED_0805, symbol charge_battery_sym_lib:LED_0805
- added R6, R7: 1K/1%/1_10W, charge_battery_footprint_lib:Res_0603, symbol charge_battery_sym_lib:Res_1K_0603_1%
- added R8, R9: 20R/1%/1_10W, charge_battery_footprint_lib:Res_0603, symbol charge_battery_sym_lib:Res_20R_0603_1%
- renumbered R9 to R10, R10 to R11, R11 to R12, R12 to R13, R13 to R14, R14 to R15, R15 to R16, R16 to R17, R17 to R18
Connections:
- net D_N: now also R9.1
- net D_P: now also R8.1
- net GNDD: now also R6.2, R7.2
- net U_N: now also R9.2
- net U_P: now also R8.2
- net LED_TEST: now reaches U1.31 (IO19)
- net LED_TEST: now also D7.2 (A)
- net LED_STATUS: now reaches U1.33 (IO21)
- net LED_STATUS: now also D8.2 (A)
- new net: D8.1 (K), R7.1
- new net: D7.1 (K), R6.1
- no-connect marks 35 -> 33

Commit message: pull
Parts:
- SW1: value SW_Push -> FLASH
- SW2: value SW_Push -> EN
Changed lines of the file:
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@@
 			)
 		)
-		(property "Value" "SW_Push"
+		(property "Value" "FLASH"
 			(at 191.77 96.52 0)
 			(effects
@@
 			)
 		)
-		(property "Value" "SW_Push"
+		(property "Value" "EN"
 			(at 191.77 135.89 0)
 			(effects
