File: Hardware/Source/System_Control/adc_mux.kicad_sch (KiCad schematic)
At the start: 20 parts, among them U18 CD74HC4067SM96, U19 CD74HC4067SM96

Commit message: schematic: update connector charger board F4
Parts:
- added TP8, TP9: TestPoint_Small, TestPoint:TestPoint_Pad_D1.0mm, symbol Connector:TestPoint_Small
Connections:
- net ADC1_IN1: now also TP8.1
- net ADC1_IN2: now also TP9.1
Changed lines of the file:
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@@
 	)
 	(junction
+		(at 238.76 52.07)
+		(diameter 0)
+		(color 0 0 0 0)
+	)
+	(junction
 		(at 115.57 50.8)
 		(diameter 0)
@@
 	)
 	(junction
+		(at 129.54 50.8)
+		(diameter 0)
+		(color 0 0 0 0)
+	)
+	(junction
 		(at 224.79 90.17)
 		(diameter 0)
@@
 	(wire
 		(pts
-			(xy 132.08 50.8) (xy 127 50.8)
+			(xy 133.35 50.8) (xy 129.54 50.8)
 		)
 		(stroke
@@
 	(wire
 		(pts
-			(xy 236.22 52.07) (xy 241.3 52.07)
+			(xy 236.22 52.07) (xy 238.76 52.07)
 		)
 		(stroke
@@
 	(wire
 		(pts
+			(xy 238.76 52.07) (xy 243.84 52.07)
+		)
+		(stroke
+			(width 0)
+			(type default)
+		)
+	)
+	(wire
+		(pts
 			(xy 115.57 76.2) (xy 115.57 77.47)
 		)
@@
 	(wire
 		(pts
+			(xy 129.54 50.8) (xy 127 50.8)
+		)
+		(stroke
+			(width 0)
+			(type default)
+		)
+	)
+	(wire
+		(pts
 			(xy 115.57 77.47) (xy 115.57 78.74)
 		)
@@
 	(global_label "ADC1_IN2"
 		(shape output)
-		(at 241.3 52.07 0)
+		(at 243.84 52.07 0)
 		(fields_autoplaced yes)
 		(effects
@@
 		)
 		(property "Intersheetrefs" "${INTERSHEET_REFS}"
-			(at 253.2357 52.07 0)
+			(at 255.7757 52.07 0)
 			(effects
 				(font
@@
 	(global_label "ADC1_IN1"
 		(shape output)
-		(at 132.08 50.8 0)
+		(at 133.35 50.8 0)
 		(fields_autoplaced yes)
 		(effects
@@
 		)
 		(property "Intersheetrefs" "${INTERSHEET_REFS}"
-			(at 144.0157 50.8 0)
+			(at 145.2857 50.8 0)
 			(effects
 				(font
@@
 	)
 	(symbol
+		(lib_id "Connector:TestPoint_Small")
+		(at 238.76 52.07 0)
+		(unit 1)
+		(exclude_from_sim no)
+		(in_bom yes)
+		(on_board yes)
+		(dnp no)
+		(property "Reference" "TP9"
+			(at 236.982 50.546 0)
+			(effects
+				(font
+					(size 1.27 1.27)
+				)
+				(justify left)
+			)
+		)
+		(property "Value" "TestPoint_Small"
+			(at 240.03 53.3399 0)
+			(effects
+				(font
+					(size 1.27 1.27)
+				)
+				(justify left)
+				(hide yes)
+			)
+		)
+		(property "Footprint" "TestPoint:TestPoint_Pad_D1.0mm"
+			(at 243.84 52.07 0)
+			(effects
+				(font
+					(size 1.27 1.27)
+				)
+				(hide yes)
+			)
+		)
+		(property "Datasheet" "~"
+			(at 243.84 52.07 0)
+			(effects
+				(font
+					(size 1.27 1.27)
+				)
+				(hide yes)
+			)
+		)
+		(property "Description" "test point"
+			(at 238.76 52.07 0)
+			(effects
+				(font
+					(size 1.27 1.27)
+				)
+				(hide yes)
+			)
+		)
+		(pin "1"
+		)
+		(instances
+			(project "System_Control"
+				(path "/85c53e8c-0403-413d-b6c5-0718d4365b1f/8a28eaba-921a-4d69-a485-b69da0a1756d"
+					(reference "TP9")
+					(unit 1)
+				)
+			)
+		)
+	)
+	(symbol
 		(lib_id "charge_battery_sym_lib:Ceramic_Cap_SMD_1nF_50V")
 		(at 224.79 60.96 90)
@@
 					(unit 1)
 				)
+			)
+		)
+	)
+	(symbol
+		(lib_id "Connector:TestPoint_Small")
+		(at 129.54 50.8 0)
+		(unit 1)
+		(exclude_from_sim no)
+		(in_bom yes)
+		(on_board yes)
+		(dnp no)
+		(property "Reference" "TP8"
+			(at 127.762 49.276 0)
+			(effects
+				(font
+					(size 1.27 1.27)
+				)
+				(justify left)
+			)
+		)
+		(property "Value" "TestPoint_Small"
+			(at 130.81 52.0699 0)
+			(effects
+				(font
+					(size 1.27 1.27)
+				)
+				(justify left)
+				(hide yes)
+			)
+		)
+		(property "Footprint" "TestPoint:TestPoint_Pad_D1.0mm"
+			(at 134.62 50.8 0)
+			(effects
+				(font
+					(size 1.27 1.27)
+				)
+				(hide yes)
+			)
+		)
+		(property "Datasheet" "~"
+			(at 134.62 50.8 0)
+			(effects
+				(font
+					(size 1.27 1.27)
+				)
+				(hide yes)
+			)
+		)
+		(property "Description" "test point"
+			(at 129.54 50.8 0)
+			(effects
+				(font
+					(size 1.27 1.27)
+				)
+				(hide yes)
+			)
+		)
+		(pin "1"
+		)
+		(instances
+			(project "System_Control"
+				(path "/85c53e8c-0403-413d-b6c5-0718d4365b1f/8a28eaba-921a-4d69-a485-b69da0a1756d"
+					(reference "TP8")
+					(unit 1)
+				)

Commit message: pcb,lib,sche: PFC, lib: update pcb PFC, lib
Parts:
- renumbered C158 to C163, C159 to C164, C160 to C165, C161 to C166, C162 to C167, C163 to C168, D74 to D73, D75 to D74, R184 to R186, R185 to R187, R186 to R188, R187 to R189, R188 to R190, R189 to R191, R190 to R192, R191 to R193, R192 to R194, R193 to R195
Changed lines of the file:
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@@
 		(on_board yes)
 		(dnp no)
-		(property "Reference" "R186"
+		(property "Reference" "R188"
 			(at 62.484 103.124 0)
 			(effects
@@
 			(project "System_Control"
 				(path "/85c53e8c-0403-413d-b6c5-0718d4365b1f/8a28eaba-921a-4d69-a485-b69da0a1756d"
-					(reference "R186")
+					(reference "R188")
 					(unit 1)
 				)
@@
 		(on_board yes)
 		(dnp no)
-		(property "Reference" "C162"
+		(property "Reference" "C167"
 			(at 224.79 83.312 90)
 			(effects
@@
 			(project "System_Control"
 				(path "/85c53e8c-0403-413d-b6c5-0718d4365b1f/8a28eaba-921a-4d69-a485-b69da0a1756d"
-					(reference "C162")
+					(reference "C167")
 					(unit 1)
 				)
@@
 		(on_board yes)
 		(dnp no)
-		(property "Reference" "R189"
+		(property "Reference" "R191"
 			(at 171.704 99.314 0)
 			(effects
@@
 			(project "System_Control"
 				(path "/85c53e8c-0403-413d-b6c5-0718d4365b1f/8a28eaba-921a-4d69-a485-b69da0a1756d"
-					(reference "R189")
+					(reference "R191")
 					(unit 1)
 				)
@@
 		(on_board yes)
 		(dnp no)
-		(property "Reference" "R192"
+		(property "Reference" "R194"
 			(at 171.704 106.934 0)
 			(effects
@@
 			(project "System_Control"
 				(path "/85c53e8c-0403-413d-b6c5-0718d4365b1f/8a28eaba-921a-4d69-a485-b69da0a1756d"
-					(reference "R192")
+					(reference "R194")
 					(unit 1)
 				)
@@
 		(on_board yes)
 		(dnp no)
-		(property "Reference" "R190"
+		(property "Reference" "R192"
 			(at 171.704 101.854 0)
 			(effects
@@
 			(project "System_Control"
 				(path "/85c53e8c-0403-413d-b6c5-0718d4365b1f/8a28eaba-921a-4d69-a485-b69da0a1756d"
-					(reference "R190")
+					(reference "R192")
 					(unit 1)
 				)
@@
 		(on_board yes)
 		(dnp no)
-		(property "Reference" "C163"
+		(property "Reference" "C168"
 			(at 234.95 83.312 90)
 			(effects
@@
 			(project "System_Control"
 				(path "/85c53e8c-0403-413d-b6c5-0718d4365b1f/8a28eaba-921a-4d69-a485-b69da0a1756d"
-					(reference "C163")
+					(reference "C168")
 					(unit 1)
 				)
@@
 		(dnp no)
 		(fields_autoplaced yes)
-		(property "Reference" "D74"
+		(property "Reference" "D73"
 			(at 129.54 55.8799 90)
 			(effects
@@
 			(project ""
 				(path "/85c53e8c-0403-413d-b6c5-0718d4365b1f/8a28eaba-921a-4d69-a485-b69da0a1756d"
-					(reference "D74")
+					(reference "D73")
 					(unit 1)
 				)
@@
 		(dnp no)
 		(fields_autoplaced yes)
-		(property "Reference" "D75"
+		(property "Reference" "D74"
 			(at 238.76 57.1499 90)
 			(effects
@@
 			(project "System_Control"
 				(path "/85c53e8c-0403-413d-b6c5-0718d4365b1f/8a28eaba-921a-4d69-a485-b69da0a1756d"
-					(reference "D75")
+					(reference "D74")
 					(unit 1)
 				)
@@
 		(on_board yes)
 		(dnp no)
-		(property "Reference" "C158"
+		(property "Reference" "C163"
 			(at 117.094 55.372 90)
 			(effects
@@
 			(project "System_Control"
 				(path "/85c53e8c-0403-413d-b6c5-0718d4365b1f/8a28eaba-921a-4d69-a485-b69da0a1756d"
-					(reference "C158")
+					(reference "C163")
 					(unit 1)
 				)
@@
 		(on_board yes)
 		(dnp no)
-		(property "Reference" "R185"
+		(property "Reference" "R187"
 			(at 62.484 100.584 0)
 			(effects
@@
 			(project "System_Control"
 				(path "/85c53e8c-0403-413d-b6c5-0718d4365b1f/8a28eaba-921a-4d69-a485-b69da0a1756d"
-					(reference "R185")
+					(reference "R187")
 					(unit 1)
 				)
@@
 		(on_board yes)
 		(dnp no)
-		(property "Reference" "C161"
+		(property "Reference" "C166"
 			(at 226.314 56.642 90)
 			(effects
@@
 			(project "System_Control"
 				(path "/85c53e8c-0403-413d-b6c5-0718d4365b1f/8a28eaba-921a-4d69-a485-b69da0a1756d"
-					(reference "C161")
+					(reference "C166")
 					(unit 1)
 				)
@@
 		(dnp no)
 		(fields_autoplaced yes)
-		(property "Reference" "R193"
+		(property "Reference" "R195"
 			(at 180.34 116.8399 90)
 			(effects
@@
 			(project "System_Control"
 				(path "/85c53e8c-0403-413d-b6c5-0718d4365b1f/8a28eaba-921a-4d69-a485-b69da0a1756d"
-					(reference "R193")
+					(reference "R195")
 					(unit 1)
 				)
@@
 		(on_board yes)
 		(dnp no)
-		(property "Reference" "R184"
+		(property "Reference" "R186"
 			(at 62.484 98.044 0)
 			(effects
@@
 			(project "System_Control"
 				(path "/85c53e8c-0403-413d-b6c5-0718d4365b1f/8a28eaba-921a-4d69-a485-b69da0a1756d"
-					(reference "R184")
+					(reference "R186")
 					(unit 1)
 				)
@@
 		(on_board yes)
 		(dnp no)
-		(property "Reference" "R191"
+		(property "Reference" "R193"
 			(at 171.704 104.394 0)
 			(effects
@@
 			(project "System_Control"
 				(path "/85c53e8c-0403-413d-b6c5-0718d4365b1f/8a28eaba-921a-4d69-a485-b69da0a1756d"
-					(reference "R191")
+					(reference "R193")
 					(unit 1)
 				)
@@
 		(on_board yes)
 		(dnp no)
-		(property "Reference" "C159"
+		(property "Reference" "C164"
 			(at 115.57 80.772 90)
 			(effects
@@
 			(project "System_Control"
 				(path "/85c53e8c-0403-413d-b6c5-0718d4365b1f/8a28eaba-921a-4d69-a485-b69da0a1756d"
-					(reference "C159")
+					(reference "C164")
 					(unit 1)
 				)
@@
 		(dnp no)
 		(fields_autoplaced yes)
-		(property "Reference" "R188"
+		(property "Reference" "R190"
 			(at 71.12 115.5699 90)
 			(effects
@@
 			(project ""
 				(path "/85c53e8c-0403-413d-b6c5-0718d4365b1f/8a28eaba-921a-4d69-a485-b69da0a1756d"
-					(reference "R188")
+					(reference "R190")
 					(unit 1)
 				)
@@
 		(on_board yes)
 		(dnp no)
-		(property "Reference" "R187"
+		(property "Reference" "R189"
 			(at 62.484 105.664 0)
 			(effects
@@
 			(project "System_Control"
 				(path "/85c53e8c-0403-413d-b6c5-0718d4365b1f/8a28eaba-921a-4d69-a485-b69da0a1756d"
-					(reference "R187")
+					(reference "R189")
 					(unit 1)
 				)
@@
 		(on_board yes)
 		(dnp no)
-		(property "Reference" "C160"
+		(property "Reference" "C165"
 			(at 125.73 80.772 90)
 			(effects
@@
 			(project "System_Control"
 				(path "/85c53e8c-0403-413d-b6c5-0718d4365b1f/8a28eaba-921a-4d69-a485-b69da0a1756d"
-					(reference "C160")
-					(unit 1)
-				)
+					(reference "C165")
+					(unit 1)
+				)

Commit message: pull
Parts:
- renumbered C163 to C161, C164 to C162, C165 to C163, C166 to C164, C167 to C165, C168 to C166, R186 to R184, R187 to R185, R188 to R186, R189 to R187, R190 to R188, R191 to R189, R192 to R190, R193 to R191, R194 to R192, R195 to R193, TP8 to TP7, TP9 to TP8
Connections:
- net NTC_BAT1: now also U19.7 (I2); no longer U19.9 (I0)
- net NTC_BAT10: now also U19.6 (I3); no longer U19.22 (I9)
- net NTC_BAT11: now also U19.4 (I5); no longer U19.21 (I10)
- net NTC_BAT12: now also U19.5 (I4); no longer U19.20 (I11)
- net NTC_BAT13: now also U19.3 (I6); no longer U19.19 (I12)
- net NTC_BAT14: now also U19.2 (I7); no longer U19.18 (I13)
- net NTC_BAT15: now also U19.20 (I11); no longer U19.17 (I14)
- net NTC_BAT16: now also U19.17 (I14); no longer U19.16 (I15)
- net NTC_BAT2: now also U19.9 (I0); no longer U19.8 (I1)
- net NTC_BAT3: now also U19.19 (I12); no longer U19.7 (I2)
- net NTC_BAT4: now also U19.16 (I15); no longer U19.6 (I3)
- net NTC_BAT5: now also U19.21 (I10); no longer U19.5 (I4)
- net NTC_BAT6: now also U19.18 (I13); no longer U19.4 (I5)
- net NTC_BAT7: now also U19.22 (I9); no longer U19.3 (I6)
- net NTC_BAT8: now also U19.23 (I8); no longer U19.2 (I7)
- net NTC_BAT9: now also U19.8 (I1); no longer U19.23 (I8)

Commit message: check
Parts:
- renumbered C161 to C154, C162 to C155, C163 to C156, C164 to C157, C165 to C158, C166 to C159, D73 to D72, D74 to D73, R184 to R182, R185 to R183, R186 to R184, R187 to R185, R188 to R186, R189 to R187, R190 to R188, R191 to R189, R192 to R190, R193 to R191
Connections:
- net VOL_BAT1: now also U18.23 (I8); no longer U18.9 (I0)
- net VOL_BAT10: now also U18.8 (I1); no longer U18.22 (I9)
- net VOL_BAT11: now also U18.7 (I2); no longer U18.21 (I10)
- net VOL_BAT12: now also U18.6 (I3); no longer U18.20 (I11)
- net VOL_BAT13: now also U18.5 (I4); no longer U18.19 (I12)
- net VOL_BAT14: now also U18.4 (I5); no longer U18.18 (I13)
- net VOL_BAT15: now also U18.3 (I6); no longer U18.17 (I14)
- net VOL_BAT16: now also U18.2 (I7); no longer U18.16 (I15)
- net VOL_BAT2: now also U18.22 (I9); no longer U18.8 (I1)
- net VOL_BAT3: now also U18.21 (I10); no longer U18.7 (I2)
- net VOL_BAT4: now also U18.20 (I11); no longer U18.6 (I3)
- net VOL_BAT5: now also U18.19 (I12); no longer U18.5 (I4)
- net VOL_BAT6: now also U18.18 (I13); no longer U18.4 (I5)
- net VOL_BAT7: now also U18.17 (I14); no longer U18.3 (I6)
- net VOL_BAT8: now also U18.16 (I15); no longer U18.2 (I7)
- net VOL_BAT9: now also U18.9 (I0); no longer U18.23 (I8)

Commit message: check
Parts:
- renumbered D72 to D60, D73 to D61, R182 to R183, R183 to R184, R184 to R185, R185 to R186, R186 to R187, R187 to R188, R188 to R189, R189 to R190, R190 to R191, R191 to R192, TP7 to TP2, TP8 to TP3
Connections:
- net +3V3 renamed +3V3_O

Commit message: pull
Parts:
- TP2: value TestPoint_Small -> IN1
- TP3: value TestPoint_Small -> IN2
Changed lines of the file:
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@@
 			)
 		)
-		(property "Value" "TestPoint_Small"
+		(property "Value" "IN2"
 			(at 240.03 53.3399 0)
 			(effects
@@
 			)
 		)
-		(property "Value" "TestPoint_Small"
+		(property "Value" "IN1"
 			(at 130.81 52.0699 0)
 			(effects

Commit message: check
Parts:
- TP2: value IN1 -> VOL
- TP3: value IN2 -> NTC
Changed lines of the file:
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@@
 			)
 		)
-		(property "Value" "IN2"
+		(property "Value" "NTC"
 			(at 240.03 53.3399 0)
 			(effects
@@
 			)
 		)
-		(property "Value" "IN1"
+		(property "Value" "VOL"
 			(at 130.81 52.0699 0)
 			(effects

Commit message: Exported BOM List 4 boards
Parts:
- U18, U19: Supply name mouser -> Mouser
