File: Hardware/Source/System_Control/balance_bat.kicad_sch (KiCad schematic)
At the start: 132 parts, among them Q10 AO3400A, Q11 AO3400A, Q12 AO3400A, Q13 AO3400A, Q14 AO3400A, Q15 AO3400A, Q16 AO3400A, Q17 AO3400A, Q18 AO3400A, Q19 AO3400A, Q20 AO3400A, Q5 AO3400A, Q6 AO3400A, Q7 AO3400A, Q8 AO3400A, Q9 AO3400A, U14 TLP291-4, U15 TLP291-4, U16 TLP291-4, U17 TLP291-4

Commit message: pull
Parts:
- renumbered R122 to R120, R123 to R121, R124 to R122, R125 to R123, R126 to R124, R127 to R125, R128 to R126, R129 to R127, R130 to R128, R131 to R129, R132 to R130, R133 to R131, R134 to R132, R135 to R133, R136 to R134, R137 to R135, R138 to R136, R139 to R137, R140 to R138, R141 to R139, R142 to R140, R143 to R141, R144 to R142, R145 to R143, R146 to R144, R147 to R145, R148 to R146, R149 to R147, R150 to R148, R151 to R149, R152 to R150, R153 to R151, R154 to R152, R155 to R153, R156 to R154, R157 to R155, R158 to R156, R159 to R157, R160 to R158, R161 to R159, R162 to R160, R163 to R161, R164 to R162, R165 to R163, R166 to R164, R167 to R165, R168 to R166, R169 to R167, R170 to R168, R171 to R169, R172 to R170, R173 to R171, R174 to R172, R175 to R173, R176 to R174, R177 to R175, R178 to R176, R179 to R177, R180 to R178, R181 to R179, R182 to R180, R183 to R181, R184 to R182, R185 to R183

Commit message: check
Parts:
- renumbered D25 to D24, D26 to D25, D27 to D26, D28 to D27, D29 to D28, D30 to D29, D31 to D30, D32 to D31, D33 to D32, D34 to D33, D35 to D34, D36 to D35, D37 to D36, D38 to D37, D39 to D38, D40 to D39, D41 to D40, D42 to D41, D43 to D42, D44 to D43, D45 to D44, D46 to D45, D47 to D46, D48 to D47, D49 to D48, D50 to D49, D51 to D50, D52 to D51, D53 to D52, D54 to D53, D55 to D54, D56 to D55, D57 to D56, D58 to D57, D59 to D58, D60 to D59, D61 to D60, D62 to D61, D63 to D62, D64 to D63, D65 to D64, D66 to D65, D67 to D66, D68 to D67, D69 to D68, D70 to D69, D71 to D70, D72 to D71, R120 to R118, R121 to R119, R122 to R120, R123 to R121, R124 to R122, R125 to R123, R126 to R124, R127 to R125, R128 to R126, R129 to R127, R130 to R128, R131 to R129, R132 to R130, R133 to R131, R134 to R132, R135 to R133, R136 to R134, R137 to R135, R138 to R136, R139 to R137, R140 to R138, R141 to R139, R142 to R140, R143 to R141, R144 to R142, R145 to R143, R146 to R144, R147 to R145, R148 to R146, R149 to R147, R150 to R148, R151 to R149, R152 to R150, R153 to R151, R154 to R152, R155 to R153, R156 to R154, R157 to R155, R158 to R156, R159 to R157, R160 to R158, R161 to R159, R162 to R160, R163 to R161, R164 to R162, R165 to R163, R166 to R164, R167 to R165, R168 to R166, R169 to R167, R170 to R168, R171 to R169, R172 to R170, R173 to R171, R174 to R172, R175 to R173, R176 to R174, R177 to R175, R178 to R176, R179 to R177, R180 to R178, R181 to R179, R182 to R180, R183 to R181

Commit message: check
Parts:
- renumbered D24 to D12, D25 to D13, D26 to D14, D27 to D15, D28 to D16, D29 to D17, D30 to D18, D31 to D19, D32 to D20, D33 to D21, D34 to D22, D35 to D23, D36 to D24, D37 to D25, D38 to D26, D39 to D27, D40 to D28, D41 to D29, D42 to D30, D43 to D31, D44 to D32, D45 to D33, D46 to D34, D47 to D35, D48 to D36, D49 to D37, D50 to D38, D51 to D39, D52 to D40, D53 to D41, D54 to D42, D55 to D43, D56 to D44, D57 to D45, D58 to D46, D59 to D47, D60 to D48, D61 to D49, D62 to D50, D63 to D51, D64 to D52, D65 to D53, D66 to D54, D67 to D55, D68 to D56, D69 to D57, D70 to D58, D71 to D59, R118 to R119, R119 to R120, R120 to R121, R121 to R122, R122 to R123, R123 to R124, R124 to R125, R125 to R126, R126 to R127, R127 to R128, R128 to R129, R129 to R130, R130 to R131, R131 to R132, R132 to R133, R133 to R134, R134 to R135, R135 to R136, R136 to R137, R137 to R138, R138 to R139, R139 to R140, R140 to R141, R141 to R142, R142 to R143, R143 to R144, R144 to R145, R145 to R146, R146 to R147, R147 to R148, R148 to R149, R149 to R150, R150 to R151, R151 to R152, R152 to R153, R153 to R154, R154 to R155, R155 to R156, R156 to R157, R157 to R158, R158 to R159, R159 to R160, R160 to R161, R161 to R162, R162 to R163, R163 to R164, R164 to R165, R165 to R166, R166 to R167, R167 to R168, R168 to R169, R169 to R170, R170 to R171, R171 to R172, R172 to R173, R173 to R174, R174 to R175, R175 to R176, R176 to R177, R177 to R178, R178 to R179, R179 to R180, R180 to R181, R181 to R182

Commit message: Exported BOM List 4 boards
Parts:
- R131, R132, R137, R138, R143, R144, R149, R150, R163, R164, R169, R170, R175, R176, R181, R182: Supply name (none) -> Mouser
