File: Hardware/Source/System_Control/temperature.kicad_sch (KiCad schematic)
At the start: 152 parts, among them U10 NE5532DR, U11 NE5532DR, U12 NE5532DR, U13 NE5532DR, U6 NE5532DR, U7 NE5532DR, U8 NE5532DR, U9 NE5532DR

Commit message: pcb,lib,sche: PFC, lib: update pcb PFC, lib
Parts:
- renumbered C95 to C100, C96 to C101, C97 to C102, C98 to C103, C99 to C104, C100 to C105, C101 to C106, C102 to C107, C103 to C108, C104 to C109, C105 to C110, C106 to C111, C107 to C112, C108 to C113, C109 to C114, C110 to C115, C111 to C116, C112 to C117, C113 to C118, C114 to C119, C115 to C120, C116 to C121, C117 to C122, C118 to C123, C119 to C124, C120 to C125, C121 to C126, C122 to C127, C123 to C128, C124 to C129, C125 to C130, C126 to C131, C127 to C132, C128 to C133, C129 to C134, C130 to C135, C131 to C136, C132 to C137, C133 to C138, C134 to C139, C135 to C140, C136 to C141, C137 to C142, C138 to C143, C139 to C144, C140 to C145, C141 to C146, C46 to C51, C47 to C52, C48 to C53, C49 to C54, C50 to C55, C51 to C56, C52 to C57, C53 to C58, C54 to C59, C55 to C60, C56 to C61, C57 to C62, C58 to C63, C59 to C64, C60 to C65, C61 to C66, C62 to C67, C63 to C68, C64 to C69, C65 to C70, C66 to C71, C67 to C72, C68 to C73, C69 to C74, C70 to C75, C71 to C76, C72 to C77, C73 to C78, C74 to C79, C75 to C80, C76 to C81, C77 to C82, C78 to C83, C79 to C84, C80 to C85, C81 to C86, C82 to C87, C83 to C88, C84 to C89, C85 to C90, C86 to C91, C87 to C92, C88 to C93, C89 to C94, C90 to C95, C91 to C96, C92 to C97, C93 to C98, C94 to C99, R40 to R42, R41 to R43, R42 to R44, R43 to R45, R44 to R46, R45 to R47, R46 to R48, R47 to R49, R48 to R50, R49 to R51, R50 to R52, R51 to R53, R52 to R54, R53 to R55, R54 to R56, R55 to R57, R56 to R58, R57 to R59, R58 to R60, R59 to R61, R60 to R62, R61 to R63, R62 to R64, R63 to R65, R64 to R66, R65 to R67, R66 to R68, R67 to R69, R68 to R70, R69 to R71, R70 to R72, R71 to R73, R72 to R74, R73 to R75, R74 to R76, R75 to R77, R76 to R78, R77 to R79, R78 to R80, R79 to R81, R80 to R82, R81 to R83, R82 to R84, R83 to R85, R84 to R86, R85 to R87, R86 to R88, R87 to R89

Commit message: pull
Parts:
- renumbered C102 to C100, C103 to C101, C104 to C102, C105 to C103, C106 to C104, C107 to C105, C108 to C106, C109 to C107, C110 to C108, C111 to C109, C112 to C110, C113 to C111, C114 to C112, C115 to C113, C116 to C114, C117 to C115, C118 to C116, C119 to C117, C120 to C118, C121 to C119, C122 to C120, C123 to C121, C124 to C122, C125 to C123, C126 to C124, C127 to C125, C128 to C126, C129 to C127, C130 to C128, C131 to C129, C132 to C130, C133 to C131, C134 to C132, C135 to C133, C136 to C134, C137 to C135, C138 to C136, C139 to C137, C140 to C138, C141 to C139, C142 to C140, C143 to C141, C144 to C142, C145 to C143, C146 to C144, C51 to C49, C52 to C50, C53 to C51, C54 to C52, C55 to C53, C56 to C54, C57 to C55, C58 to C56, C59 to C57, C60 to C58, C61 to C59, C62 to C60, C63 to C61, C64 to C62, C65 to C63, C66 to C64, C67 to C65, C68 to C66, C69 to C67, C70 to C68, C71 to C69, C72 to C70, C73 to C71, C74 to C72, C75 to C73, C76 to C74, C77 to C75, C78 to C76, C79 to C77, C80 to C78, C81 to C79, C82 to C80, C83 to C81, C84 to C82, C85 to C83, C86 to C84, C87 to C85, C88 to C86, C89 to C87, C90 to C88, C91 to C89, C92 to C90, C93 to C91, C94 to C92, C95 to C93, C96 to C94, C97 to C95, C98 to C96, C99 to C97, C100 to C98, C101 to C99, R42 to R40, R43 to R41, R44 to R42, R45 to R43, R46 to R44, R47 to R45, R48 to R46, R49 to R47, R50 to R48, R51 to R49, R52 to R50, R53 to R51, R54 to R52, R55 to R53, R56 to R54, R57 to R55, R58 to R56, R59 to R57, R60 to R58, R61 to R59, R62 to R60, R63 to R61, R64 to R62, R65 to R63, R66 to R64, R67 to R65, R68 to R66, R69 to R67, R70 to R68, R71 to R69, R72 to R70, R73 to R71, R74 to R72, R75 to R73, R76 to R74, R77 to R75, R78 to R76, R79 to R77, R80 to R78, R81 to R79, R82 to R80, R83 to R81, R84 to R82, R85 to R83, R86 to R84, R87 to R85, R88 to R86, R89 to R87

Commit message: check
Parts:
- renumbered C107 to C100, C108 to C101, C109 to C102, C110 to C103, C111 to C104, C112 to C105, C113 to C106, C114 to C107, C115 to C108, C116 to C109, C117 to C110, C118 to C111, C119 to C112, C120 to C113, C121 to C114, C122 to C115, C123 to C116, C124 to C117, C125 to C118, C126 to C119, C127 to C120, C128 to C121, C129 to C122, C130 to C123, C131 to C124, C132 to C125, C133 to C126, C134 to C127, C135 to C128, C136 to C129, C137 to C130, C138 to C131, C139 to C132, C140 to C133, C141 to C134, C142 to C135, C143 to C136, C144 to C137, C49 to C42, C50 to C43, C51 to C44, C52 to C45, C53 to C46, C54 to C47, C55 to C48, C56 to C49, C57 to C50, C58 to C51, C59 to C52, C60 to C53, C61 to C54, C62 to C55, C63 to C56, C64 to C57, C65 to C58, C66 to C59, C67 to C60, C68 to C61, C69 to C62, C70 to C63, C71 to C64, C72 to C65, C73 to C66, C74 to C67, C75 to C68, C76 to C69, C77 to C70, C78 to C71, C79 to C72, C80 to C73, C81 to C74, C82 to C75, C83 to C76, C84 to C77, C85 to C78, C86 to C79, C87 to C80, C88 to C81, C89 to C82, C90 to C83, C91 to C84, C92 to C85, C93 to C86, C94 to C87, C95 to C88, C96 to C89, C97 to C90, C98 to C91, C99 to C92, C100 to C93, C101 to C94, C102 to C95, C103 to C96, C104 to C97, C105 to C98, C106 to C99, R40 to R38, R41 to R39, R42 to R40, R43 to R41, R44 to R42, R45 to R43, R46 to R44, R47 to R45, R48 to R46, R49 to R47, R50 to R48, R51 to R49, R52 to R50, R53 to R51, R54 to R52, R55 to R53, R56 to R54, R57 to R55, R58 to R56, R59 to R57, R60 to R58, R61 to R59, R62 to R60, R63 to R61, R64 to R62, R65 to R63, R66 to R64, R67 to R65, R68 to R66, R69 to R67, R70 to R68, R71 to R69, R72 to R70, R73 to R71, R74 to R72, R75 to R73, R76 to R74, R77 to R75, R78 to R76, R79 to R77, R80 to R78, R81 to R79, R82 to R80, R83 to R81, R84 to R82, R85 to R83, R86 to R84, R87 to R85

Commit message: check
Parts:
- renumbered R38 to R39, R39 to R40, R40 to R41, R41 to R42, R42 to R43, R43 to R44, R44 to R45, R45 to R46, R46 to R47, R47 to R48, R48 to R49, R49 to R50, R50 to R51, R51 to R52, R52 to R53, R53 to R54, R54 to R55, R55 to R56, R56 to R57, R57 to R58, R58 to R59, R59 to R60, R60 to R61, R61 to R62, R62 to R63, R63 to R64, R64 to R65, R65 to R66, R66 to R67, R67 to R68, R68 to R69, R69 to R70, R70 to R71, R71 to R72, R72 to R73, R73 to R74, R74 to R75, R75 to R76, R76 to R77, R77 to R78, R78 to R79, R79 to R80, R80 to R81, R81 to R82, R82 to R83, R83 to R84, R84 to R85, R85 to R86
Connections:
- net +3V3 renamed +3V3_O

Commit message: Exported BOM List 4 boards
Parts:
- U10, U11, U12, U13, U6, U7, U8, U9: Supply name TME -> tme
