File: Hardware/Source/System_Control/voltage.kicad_sch (KiCad schematic)
At the start: 48 parts

Commit message: pcb,lib,sche: PFC, lib: update pcb PFC, lib
Parts:
- renumbered C142 to C147, C143 to C148, C144 to C149, C145 to C150, C146 to C151, C147 to C152, C148 to C153, C149 to C154, C150 to C155, C151 to C156, C152 to C157, C153 to C158, C154 to C159, C155 to C160, C156 to C161, C157 to C162, R98 to R100, R99 to R101, R100 to R102, R101 to R103, R102 to R104, R103 to R105, R104 to R106, R105 to R107, R106 to R108, R107 to R109, R108 to R110, R109 to R111, R110 to R112, R111 to R113, R112 to R114, R113 to R115, R114 to R116, R115 to R117, R116 to R118, R117 to R119, R118 to R120, R119 to R121, R88 to R90, R89 to R91, R90 to R92, R91 to R93, R92 to R94, R93 to R95, R94 to R96, R95 to R97, R96 to R98, R97 to R99

Commit message: pull
Parts:
- renumbered C147 to C145, C148 to C146, C149 to C147, C150 to C148, C151 to C149, C152 to C150, C153 to C151, C154 to C152, C155 to C153, C156 to C154, C157 to C155, C158 to C156, C159 to C157, C160 to C158, C161 to C159, C162 to C160, R102 to R100, R103 to R101, R104 to R102, R105 to R103, R106 to R104, R107 to R105, R108 to R106, R109 to R107, R110 to R108, R111 to R109, R112 to R110, R113 to R111, R114 to R112, R115 to R113, R116 to R114, R117 to R115, R118 to R116, R119 to R117, R120 to R118, R121 to R119, R90 to R88, R91 to R89, R92 to R90, R93 to R91, R94 to R92, R95 to R93, R96 to R94, R97 to R95, R98 to R96, R99 to R97, R100 to R98, R101 to R99

Commit message: check
Parts:
- renumbered C145 to C138, C146 to C139, C147 to C140, C148 to C141, C149 to C142, C150 to C143, C151 to C144, C152 to C145, C153 to C146, C154 to C147, C155 to C148, C156 to C149, C157 to C150, C158 to C151, C159 to C152, C160 to C153, R102 to R100, R103 to R101, R104 to R102, R105 to R103, R106 to R104, R107 to R105, R108 to R106, R109 to R107, R110 to R108, R111 to R109, R112 to R110, R113 to R111, R114 to R112, R115 to R113, R116 to R114, R117 to R115, R118 to R116, R119 to R117, R88 to R86, R89 to R87, R90 to R88, R91 to R89, R92 to R90, R93 to R91, R94 to R92, R95 to R93, R96 to R94, R97 to R95, R98 to R96, R99 to R97, R100 to R98, R101 to R99
Connections:
- net VOL_BAT1: now also C153.2, R116.1, R117.2; no longer C138.2, R86.1, R87.2
- net VOL_BAT11: now also C143.2, R96.1, R97.2; no longer C148.2, R106.1, R107.2
- net VOL_BAT12: now also C139.2, R88.1, R89.2; no longer C149.2, R108.1, R109.2
- net VOL_BAT14: now also C146.2, R102.1, R103.2; no longer C151.2, R112.1, R113.2
- net VOL_BAT15: now also C142.2, R94.2, R95.2; no longer C152.2, R114.1, R115.2
- net VOL_BAT16: now also C138.2, R86.1, R87.2; no longer C153.2, R116.1, R117.2
- net VOL_BAT2: now also C149.2, R108.1, R109.2; no longer C139.2, R88.1, R89.2
- net VOL_BAT3: now also C145.2, R100.1, R101.2; no longer C140.2, R90.1, R91.2
- net VOL_BAT5: now also C152.2, R114.1, R115.2; no longer C142.2, R94.2, R95.2
- net VOL_BAT6: now also C148.2, R106.1, R107.2; no longer C143.2, R96.1, R97.2
- net VOL_BAT8: now also C140.2, R90.1, R91.2; no longer C145.2, R100.1, R101.2
- net VOL_BAT9: now also C151.2, R112.1, R113.2; no longer C146.2, R102.1, R103.2

Commit message: check
Parts:
- renumbered R99 to R100, R100 to R101, R101 to R102, R102 to R103, R103 to R104, R104 to R105, R105 to R106, R106 to R107, R107 to R108, R108 to R109, R109 to R110, R110 to R111, R111 to R112, R112 to R113, R113 to R114, R114 to R115, R115 to R116, R116 to R117, R117 to R118, R86 to R87, R87 to R88, R88 to R89, R89 to R90, R90 to R91, R91 to R92, R92 to R93, R93 to R94, R94 to R95, R95 to R96, R96 to R97, R97 to R98, R98 to R99
