File: Hardware/Source/Power_Supply/Charge_Pump.kicad_sch (KiCad schematic)
At the start: 1 part, among them U11 ICL7662CBA

Commit message: Fix lib
Parts:
- removed U11: ICL7662CBA, charge_battery_footprint_lib:SOIC-8, symbol charge_battery_sym_lib:ICL7662CBA
Changed lines of the file:
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@@
 	(generator_version "8.0")
 	(paper "A4")
-	(symbol
-		(lib_id "charge_battery_sym_lib:ICL7662CBA")
-		(at 129.54 72.39 0)
-		(unit 1)
-		(exclude_from_sim no)
-		(in_bom yes)
-		(on_board yes)
-		(dnp no)
-		(fields_autoplaced yes)
-		(property "Reference" "U11"
-			(at 137.16 53.34 0)
-			(effects
-				(font
-					(size 1.27 1.27)
-				)
-			)
-		)
-		(property "Value" "ICL7662CBA"
-			(at 137.16 55.88 0)
-			(effects
-				(font
-					(size 1.27 1.27)
-				)
-			)
-		)
-		(property "Footprint" "charge_battery_footprint_lib:SOIC-8"
-			(at 110.49 94.234 0)
-			(effects
-				(font
-					(size 1.27 1.27)
-				)
-				(hide yes)
-			)
-		)
-		(property "Datasheet" "https://www.analog.com/media/en/technical-documentation/data-sheets/icl7662-si7661.pdf"
-			(at 130.048 93.98 0)
-			(effects
-				(font
-					(size 1.27 1.27)
-				)
-				(hide yes)
-			)
-		)
-		(property "Description" "Voltage Input: 4.5V ~ 20V, Voltage Output: -Vin, 8-SOIC"
-			(at 129.54 94.234 0)
-			(effects
-				(font
-					(size 1.27 1.27)
-				)
-				(hide yes)
-			)
-		)
-		(property "Supply name" "Thegioiic"
-			(at 130.81 93.98 0)
-			(effects
-				(font
-					(size 1.27 1.27)
-				)
-				(hide yes)
-			)
-		)
-		(property "Supply part number" "ICL7662CBA"
-			(at 130.81 93.98 0)
-			(effects
-				(font
-					(size 1.27 1.27)
-				)
-				(hide yes)
-			)
-		)
-		(property "Supply URL" "https://www.thegioiic.com/icl7662cba"
-			(at 117.602 94.234 0)
-			(effects
-				(font
-					(size 1.27 1.27)
-				)
-				(hide yes)
-			)
-		)
-		(pin "5"
-		)
-		(pin "4"
-		)
-		(pin "3"
-		)
-		(pin "8"
-		)
-		(pin "7"
-		)
-		(pin "2"
-		)
-		(pin "6"
-		)
-		(pin "1"
-		)
-		(instances
-			(project ""
-				(path "/5c8a7907-026b-4416-b231-5ef9f93b99e1/fc81c86a-849a-473b-a705-41432f1eafdf"
-					(reference "U11")
-					(unit 1)
-				)
-			)
-		)
-	)
 )

Commit message: Update lib
Parts:
- added U11: ICL7662CBA, charge_battery_footprint_lib:SOIC-8, symbol charge_battery_sym_lib:ICL7662CBA
Changed lines of the file:
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@@
 	(generator_version "8.0")
 	(paper "A4")
+	(symbol
+		(lib_id "charge_battery_sym_lib:ICL7662CBA")
+		(at 129.54 72.39 0)
+		(unit 1)
+		(exclude_from_sim no)
+		(in_bom yes)
+		(on_board yes)
+		(dnp no)
+		(fields_autoplaced yes)
+		(property "Reference" "U11"
+			(at 137.16 53.34 0)
+			(effects
+				(font
+					(size 1.27 1.27)
+				)
+			)
+		)
+		(property "Value" "ICL7662CBA"
+			(at 137.16 55.88 0)
+			(effects
+				(font
+					(size 1.27 1.27)
+				)
+			)
+		)
+		(property "Footprint" "charge_battery_footprint_lib:SOIC-8"
+			(at 110.49 94.234 0)
+			(effects
+				(font
+					(size 1.27 1.27)
+				)
+				(hide yes)
+			)
+		)
+		(property "Datasheet" "https://www.analog.com/media/en/technical-documentation/data-sheets/icl7662-si7661.pdf"
+			(at 130.048 93.98 0)
+			(effects
+				(font
+					(size 1.27 1.27)
+				)
+				(hide yes)
+			)
+		)
+		(property "Description" "Voltage Input: 4.5V ~ 20V, Voltage Output: -Vin, 8-SOIC"
+			(at 129.54 94.234 0)
+			(effects
+				(font
+					(size 1.27 1.27)
+				)
+				(hide yes)
+			)
+		)
+		(property "Supply name" "Thegioiic"
+			(at 130.81 93.98 0)
+			(effects
+				(font
+					(size 1.27 1.27)
+				)
+				(hide yes)
+			)
+		)
+		(property "Supply part number" "ICL7662CBA"
+			(at 130.81 93.98 0)
+			(effects
+				(font
+					(size 1.27 1.27)
+				)
+				(hide yes)
+			)
+		)
+		(property "Supply URL" "https://www.thegioiic.com/icl7662cba"
+			(at 117.602 94.234 0)
+			(effects
+				(font
+					(size 1.27 1.27)
+				)
+				(hide yes)
+			)
+		)
+		(pin "5"
+		)
+		(pin "4"
+		)
+		(pin "3"
+		)
+		(pin "8"
+		)
+		(pin "7"
+		)
+		(pin "2"
+		)
+		(pin "6"
+		)
+		(pin "1"
+		)
+		(instances
+			(project ""
+				(path "/5c8a7907-026b-4416-b231-5ef9f93b99e1/fc81c86a-849a-473b-a705-41432f1eafdf"
+					(reference "U11")
+					(unit 1)
+				)
+			)
+		)
+	)
 )
