File: Hardware/Source/Power_Supply/LDO_3V3.kicad_sch (KiCad schematic)
At the start: 33 parts, among them U13 LD1117S33CTR_SOT223, U14 LD1117S33CTR_SOT223, U15 LD1117S33CTR_SOT223, U16 TPS54331DR

Commit message: update
Parts:
- removed C67: 100uF/35V, Capacitor_SMD:CP_Elec_5x5.4, symbol charge_battery_sym_lib:Cap_Polarized_SMD_100uF_35V
- removed C68: 4.7uF/50V, charge_battery_footprint_lib:Ceramic_Cap_0805, symbol charge_battery_sym_lib:Ceramic_Cap_SMD_4.7uF_50V
- removed C69: 10nF/50V, charge_battery_footprint_lib:Ceramic_Cap_0805, symbol charge_battery_sym_lib:Ceramic_Cap_SMD_10nF_50V_0805
- removed C73: 4.7nF/50V, charge_battery_footprint_lib:Ceramic_Cap_0603, symbol charge_battery_sym_lib:Ceramic_Cap_SMD_4.7nF_50V
- removed C77: 39pF/50V, charge_battery_footprint_lib:Ceramic_Cap_0603, symbol charge_battery_sym_lib:Ceramic_Cap_SMD_39pF_50V
- removed C78: 10nF/50V, charge_battery_footprint_lib:Ceramic_Cap_0603, symbol charge_battery_sym_lib:Ceramic_Cap_SMD_10nF_50V
- removed C85: 100nF/16V, charge_battery_footprint_lib:Ceramic_Cap_0603, symbol charge_battery_sym_lib:Ceramic_Cap_SMD_100nF_16V
- removed C86, C87: 47uF/6.3V, charge_battery_footprint_lib:Ceramic_Cap_0805, symbol charge_battery_sym_lib:Ceramic_Cap_SMD_47uF_6.3V
- removed D9: SS54, charge_battery_footprint_lib:D_SMA, symbol charge_battery_sym_lib:SS54
- removed L8: CDRH104 1038-220, charge_battery_footprint_lib:CDRH104, symbol charge_battery_sym_lib:CDRH104 1038-220
- removed R44: 47K/1%/1_10W, charge_battery_footprint_lib:Res_0603, symbol charge_battery_sym_lib:Res_47K_0603_1%
- removed R45: 10K/1%/1_10W, charge_battery_footprint_lib:Res_0603, symbol charge_battery_sym_lib:Res_10K_0603_1%
- removed R46: 30K/1%/1_10W, charge_battery_footprint_lib:Res_0603, symbol charge_battery_sym_lib:Res_30K_0603_1%
- removed R47: 0/1%/1_8W, charge_battery_footprint_lib:Res_0805, symbol charge_battery_sym_lib:Res_0_0805_1%
- removed R48: 56K/1%/1_8W, charge_battery_footprint_lib:Res_0805, symbol charge_battery_sym_lib:Res_56K_0805_1%
- removed R49: 10.5K/1%/1_8W, charge_battery_footprint_lib:Res_0805, symbol charge_battery_sym_lib:Res_10K5_0805_1%
- removed U16: TPS54331DR, charge_battery_footprint_lib:SOIC-8, symbol charge_battery_sym_lib:TPS54331DR
Other:
- moved on the sheet: C70, C71, C72, C74, C75, C76, C79, C80, C81, C82, C83, C84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

Commit message: update lib PSC
Parts:
- removed C71, C72, C80, C81: 10uF/16V, charge_battery_footprint_lib:Tan_Cap_A, symbol charge_battery_sym_lib:Cap_Tantalum_10uF_16V
- removed C75, C76, C83, C84: 1uF/16V, charge_battery_footprint_lib:Tan_Cap_A, symbol charge_battery_sym_lib:Cap_Tantalum_1uF_16V
- removed U14, U15: LD1117S33CTR_SOT223, charge_battery_footprint_lib:SOT-223, symbol charge_battery_sym_lib:LD1117S33CTR_SOT223
Connections:
- net +3.3_1V renamed +3.3V
- net +5_3V renamed +5V
Other:
- moved on the sheet: C70, C74, C79, C82, U13

Commit message: Update Lib PSC
Changed lines of the file:
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@@
 		(on_board yes)
 		(dnp no)
-		(fields_autoplaced yes)
 		(property "Reference" "#PWR070"
 			(at 171.45 88.9 0)
@@
 		)
 		(property "Value" "+3.3V"
-			(at 173.99 83.8199 0)
+			(at 168.656 80.518 0)
 			(effects
 				(font
@@
 		(on_board yes)
 		(dnp no)
-		(fields_autoplaced yes)
 		(property "Reference" "#PWR061"
 			(at 111.76 88.9 0)
@@
 		)
 		(property "Value" "+5V"
-			(at 114.3 83.8199 0)
+			(at 109.474 80.518 0)
 			(effects
 				(font

Commit message: Update Lib ER35 Transformer
Parts:
- added C33, C37: 10uF/16V, charge_battery_footprint_lib:Tan_Cap_A, symbol charge_battery_sym_lib:Cap_Tantalum_10uF_16V
- added C35, C39: 1uF/16V, charge_battery_footprint_lib:Tan_Cap_A, symbol charge_battery_sym_lib:Cap_Tantalum_1uF_16V
- added U9: LD1117S33CTR_SOT223, charge_battery_footprint_lib:SOT-223, symbol charge_battery_sym_lib:LD1117S33CTR_SOT223
- renumbered C70 to C34, C74 to C36, C79 to C38, C82 to C40, U13 to U10
Connections:
- net +5V: now also C33.1, C35.1, U9.3 (INPUT)
- net GND2: now also C33.2, C35.2, C37.2, C39.2, U9.1 (GND)
- net +3.3V renamed +3.3_1V
- new net +3.3_2V: C37.1, C39.1, U9.2 (OUT), U9.4 (OUT)
