File: Hardware/Source/Power_Supply/5V_Isolated.kicad_sch (KiCad schematic)
At the start: 0 parts

Commit message: update flyback co 7V
Parts:
- added C29, C31: 10uF/16V, charge_battery_footprint_lib:Tan_Cap_A, symbol charge_battery_sym_lib:Cap_Tantalum_10uF_16V
- added C30, C32: 1uF/16V, charge_battery_footprint_lib:Tan_Cap_A, symbol charge_battery_sym_lib:Cap_Tantalum_1uF_16V
- added U8: LM1117IMP-5.0, charge_battery_footprint_lib:SOT-223, symbol charge_battery_sym_lib:LM1117IMP-5.0/NOPB
Connections:
- new net +5_1V: C31.1, C32.1, U8.2 (OUT), U8.4 (OUT)
- new net +7V: C29.1, C30.1, U8.3 (INPUT)
- new net GND3: C29.2, C30.2, C31.2, C32.2, U8.1 (GND)
