File: Hardware/Source/Power_Supply/Power_Supply.kicad_sch (KiCad schematic)
At the start: 0 parts

Commit message: update
Other:
- removed sheet Buck Converter 12V
Changed lines of the file:
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@@
 	)
 	(sheet
-		(at 176.53 73.66)
+		(at 140.97 73.66)
 		(size 30.48 26.67)
 		(fields_autoplaced yes)
@@
 		)
 		(property "Sheetname" "Linear Voltage 9V"
-			(at 176.53 72.9484 0)
+			(at 140.97 72.9484 0)
 			(effects
 				(font
@@
 		)
 		(property "Sheetfile" "Linear_Voltage_9V.kicad_sch"
-			(at 176.53 100.9146 0)
+			(at 140.97 100.9146 0)
 			(effects
 				(font
@@
 				(path "/5c8a7907-026b-4416-b231-5ef9f93b99e1"
 					(page "4")
-				)
-			)
-		)
-	)
-	(sheet
-		(at 140.97 73.66)
-		(size 31.75 26.67)
-		(fields_autoplaced yes)
-		(stroke
-			(width 0.1524)
-			(type solid)
-		)
-		(fill
-			(color 0 0 0 0.0000)
-		)
-		(property "Sheetname" "Buck Converter 12V"
-			(at 140.97 72.9484 0)
-			(effects
-				(font
-					(size 1.27 1.27)
-				)
-				(justify left bottom)
-			)
-		)
-		(property "Sheetfile" "Buck_12V.kicad_sch"
-			(at 140.97 100.9146 0)
-			(effects
-				(font
-					(size 1.27 1.27)
-				)
-				(justify left top)
-			)
-		)
-		(instances
-			(project "Power_Supply"
-				(path "/5c8a7907-026b-4416-b231-5ef9f93b99e1"
-					(page "3")
 				)
 			)
@@
 	)
 	(sheet
-		(at 215.9 110.49)
-		(size 27.94 25.4)
+		(at 212.09 73.66)
+		(size 27.94 26.67)
 		(fields_autoplaced yes)
 		(stroke
@@
 		)
 		(property "Sheetname" "Connector & LED"
-			(at 215.9 109.7784 0)
+			(at 212.09 72.9484 0)
 			(effects
 				(font
@@
 		)
 		(property "Sheetfile" "Connector&LED.kicad_sch"
-			(at 215.9 136.4746 0)
+			(at 212.09 100.9146 0)
 			(effects
 				(font
@@
 	)
 	(sheet
-		(at 215.9 73.66)
+		(at 177.8 73.66)
 		(size 27.94 26.67)
 		(fields_autoplaced yes)
@@
 		)
 		(property "Sheetname" "Charge Pump"
-			(at 215.9 72.9484 0)
+			(at 177.8 72.9484 0)
 			(effects
 				(font
@@
 		)
 		(property "Sheetfile" "Charge_Pump.kicad_sch"
-			(at 215.9 100.9146 0)
-			(effects
-				(font
+			(at 177.8 100.9146 0)
+			(effects
+				(font

Commit message: update de sua sche
Other:
- added sheet LDO 5V Isolated (5V_Isolated.kicad_sch)
Changed lines of the file:
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@@
+	)
+	(sheet
+		(at 99.06 110.49)
+		(size 38.1 25.4)
+		(fields_autoplaced yes)
+		(stroke
+			(width 0.1524)
+			(type solid)
+		)
+		(fill
+			(color 0 0 0 0.0000)
+		)
+		(property "Sheetname" "LDO 5V Isolated"
+			(at 99.06 109.7784 0)
+			(effects
+				(font
+					(size 1.27 1.27)
+				)
+				(justify left bottom)
+			)
+		)
+		(property "Sheetfile" "5V_Isolated.kicad_sch"
+			(at 99.06 136.4746 0)
+			(effects
+				(font
+					(size 1.27 1.27)
+				)
+				(justify left top)
+			)
+		)
+		(instances
+			(project "Power_Supply"
+				(path "/5c8a7907-026b-4416-b231-5ef9f93b99e1"
+					(page "8")
+				)
+			)
+		)
 	)
 	(sheet
