File: Hardware/Source/PFC & LLC/PFC & LLC.kicad_pcb (KiCad board)
At the start: 2 copper layers, 116 x 79.3 mm, 232 parts, among them J1 HB9500M-9.5-3P, J2 Conn_01x02_Socket, J3 Conn_01x06_Socket, J4 Conn_01x04_Pin, J5 Conn_01x05_Socket, K1 Relay 12VDC 10A, Q1 MMBT2222A, Q2 IPA60R170CFD7XKSA1, Q2 IPP60R125CP, Q3 MMBT2222A, Q4 IPP60R125CP, Q5 IPP60R125CP, Q6 LN2302LT1G, Q7 LN2302LT1G, Q8 MMBT2222A, SW1 SW_Push, U1 PC817X2NIPW, U10 OPAMP_OP07CSZ, U11 OPAMP_OP07CSZ, U12 ACS712ELCTR-05B-T, U13 ADS1115IDGS, U14 STM32F103C8T6, U15 MAX485CSA, U2 OPAMP_OP07CSZ, U3 UCC28180D, U4 SN74LVC1G14DBVR, U5 6N137M, U6 6N137M, U7 IR2101, U8 OPAMP_OP07CSZ, U9 OPAMP_OP07CSZ, Y1 Crystal_8MHz_SMD-4PIN

Commit message: layout PFC
Parts:
- removed the C37 at (263.3, 55.1)
- L3: moved to B.Cu
- moved J2 222.8 mm to (25.3, 78.9), turned to -90 degrees
- moved D7 207.5 mm to (55.9, 98.8), turned to 180 degrees
- moved L4 197.5 mm to (23.8, 111.7)
- moved D8 196.1 mm to (67.2, 98.8), turned to 180 degrees
- moved C30 142.4 mm to (74.1, 94.5)
- moved L3 98.0 mm to (80.6, 79.0), turned to 180 degrees
- moved C38 74.5 mm to (42.1, 96.7), turned to -90 degrees
- moved C39 61.1 mm to (31.2, 96.7), turned to -90 degrees
- moved C37 60.0 mm to (20.4, 96.7), turned to -90 degrees
- moved R25 17.6 mm to (89.8, 96.4)
- moved R29 3.33 mm to (82.1, 95.1)
- moved Q4 1.53 mm to (78.2, 98.2)
- moved Q5 1.53 mm to (89.2, 98.2)
Routing:
- net R_Shunt_Voltage: track 0.00 -> 38.9 mm

Commit message: Update Lib ER35 Transformer
Parts:
- L3: moved to F.Cu
- L4: footprint charge_battery_footprint_lib:Transformer -> charge_battery_footprint_lib:Transformer_ER35
- moved J5 110.3 mm to (23.5, 94.4), turned to -90 degrees
- moved J3 94.6 mm to (23.0, 115.6)
- moved L4 53.9 mm to (75.1, 95.4), turned to -90 degrees
- moved C37 31.9 mm to (52.1, 93.1), turned to 0 degrees
- moved D7 29.8 mm to (78.6, 118.1)
- moved C24 28.2 mm to (124.6, 113.0), turned to 180 degrees
- moved C30 25.1 mm to (89.5, 114.3)
- moved L3 24.6 mm to (96.0, 98.2)
- moved C39 22.6 mm to (52.2, 105.1), turned to 0 degrees
- moved C38 22.6 mm to (52.1, 116.9), turned to 0 degrees
- moved R25 22.4 mm to (101.1, 115.8)
- moved R24 22.4 mm to (90.1, 115.8)
- moved R28 22.4 mm to (82.4, 114.5)
- moved R29 22.4 mm to (93.3, 114.5)
- moved Q4 22.4 mm to (89.5, 117.7)
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Connections:
- J3 pad 1: +12V -> GND2
- J3 pad 2: +9V -> +3V3
- J3 pad 3: -9V -> +5V
- J3 pad 4: +5V -> -9V
- J3 pad 5: +3V3 -> +9V
- J3 pad 6: GND2 -> +12V
Routing:
- net Net-(L4-SA): track 0.00 -> 46.1 mm
- net R_Shunt_Voltage: track 38.9 -> 0.00 mm
- net Net-(L4-SB): track 0.00 -> 8.14 mm
Other:
- board size 116 x 79.3 mm -> 116.9 x 98.2 mm

Commit message: Update Lib ER35 Transformer
Parts:
- removed the C35 at (263.3, 32.0)
- removed the C36 at (263.3, 43.5)
- removed the Q2 at (-45.7, 78.7)
- removed the Q2 at (123.8, 52.6)
- added Q2: IPP60R125CP, charge_battery_footprint_lib:TO-220-3, F.Cu at (124.0, 52.5)
- added R65: 47/1%/1_10W, charge_battery_footprint_lib:Res_0603, F.Cu at (150.4, 149.5)
- added R66: 47/1%/1_10W, charge_battery_footprint_lib:Res_0603, F.Cu at (150.4, 152.0)
- added R67: 220/1%/1_10W, charge_battery_footprint_lib:Res_0603, F.Cu at (150.4, 154.5)
- C28, C29, C31, C32, C33, C34, C35, C36, C40, C41, C42, C43, C44, C46, C47, C48, C49, C50, C51, C53, C54, C55, C56, C62, D6, R18, R19, R20, R26, R27, R30, R31, R32, R33, R34, R35, R36, R38, U12, U7, U8, U9: moved to B.Cu
- moved R37 229.0 mm to (36.8, 78.9), turned to 180 degrees
- moved U8 226.5 mm to (37.8, 106.9), turned to 180 degrees
- moved R36 222.4 mm to (46.9, 109.2), turned to 90 degrees
- moved U9 222.2 mm to (37.6, 97.5)
- moved R35 222.2 mm to (46.9, 103.9), turned to 90 degrees
- moved U10 222.0 mm to (34.6, 89.1), turned to -90 degrees
- moved U11 212.5 mm to (43.1, 89.1), turned to 90 degrees
- moved R40 208.1 mm to (31.7, 83.8)
- moved R39 208.1 mm to (31.7, 82.4)
- moved U12 204.9 mm to (48.5, 74.7)
- moved R42 203.0 mm to (37.4, 82.5), turned to 180 degrees
- moved R41 202.8 mm to (37.4, 81.2), turned to 180 degrees
- moved C60 199.7 mm to (29.6, 85.6), turned to -90 degrees
- moved C58 194.1 mm to (31.0, 85.6), turned to -90 degrees
- moved R34 192.6 mm to (43.1, 109.7), turned to 90 degrees
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Connections:
- C86 pad 1: Net-(U14A-PD1-OSC_OUT-RCC_OSC_OUT) -> Net-(C86-Pad1)
- J4 pad 2: /STM32F103C8T6/SWDIO -> Net-(J4-Pin_2)
- J4 pad 3: /STM32F103C8T6/SWCLK -> Net-(J4-Pin_3)
- U14 pad 17: L_Gate_Opto -> H_Gate_Opto
- U14 pad 29: H_Gate_Opto -> L_Gate_Opto
- Y1 pad 3: Net-(U14A-PD1-OSC_OUT-RCC_OSC_OUT) -> Net-(C86-Pad1)
Routing:
- net PFC_VCC: track 53.6 -> 222.6 mm
- net R_Shunt_Voltage: track 0.00 -> 100.9 mm
- net /LLC/LOAD_M1_M2: track 0.00 -> 62.0 mm
- net GND2: track 0.00 -> 48.8 mm
- net H_Gate_Driver: track 0.00 -> 32.7 mm
- net /LLC/OUT_M1: track 0.00 -> 28.0 mm, vias 0 -> 2
- net 51.2V: track 0.00 -> 27.7 mm
- net Net-(U9-+IN): track 0.00 -> 26.4 mm
- net Net-(L4-AA): track 0.00 -> 22.8 mm
- net /LLC/OUT_M2: track 0.00 -> 20.2 mm, vias 0 -> 2
- net GND1: track 1.25 -> 19.2 mm
- net L_Gate_Driver: track 0.00 -> 17.4 mm
- net -9V: track 0.00 -> 13.6 mm
- net Net-(U11-+IN): track 0.00 -> 12.4 mm
- net +9V: track 0.00 -> 12.2 mm
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
Commit message: Update
Parts:
- added H1: MountingHole, MountingHole:MountingHole_3.2mm_M3_ISO14580_Pad_TopBottom, F.Cu at (20.7, 119.8)
- added H2: MountingHole, MountingHole:MountingHole_3.2mm_M3_ISO14580_Pad_TopBottom, F.Cu at (22.7, 151.5)
- added H3: MountingHole, MountingHole:MountingHole_3.2mm_M3_ISO14580_Pad_TopBottom, F.Cu at (22.7, 158.6)
- added H4: MountingHole, MountingHole:MountingHole_3.2mm_M3_ISO14580_Pad_TopBottom, F.Cu at (22.7, 165.6)
- C10, C101, C102, C104, C105, C107, C11, C110, C2, C3, C4, C6, C67, C68, C7, C71, C72, C74, C75, C78, C79, C81, C82, C96, C99, D15, R2, R3, R5, R6, U2: moved to B.Cu
- C90: value 1uF/50V -> 1uF/16V; footprint Capacitor_SMD:CP_Elec_4x5.4 -> charge_battery_footprint_lib:Ceramic_Cap_0603
- D14: value PESD2USB3UXT-QR -> SMF05C_1; footprint charge_battery_footprint_lib:SOT23 -> charge_battery_footprint_lib:SOT-363; moved to B.Cu
- moved D12 149.0 mm to (51.4, 54.6), turned to -90 degrees
- moved D11 144.5 mm to (54.9, 54.6), turned to -90 degrees
- moved C111 142.7 mm to (53.5, 62.2), turned to 180 degrees
- moved C90 141.7 mm to (70.9, 59.6), turned to -90 degrees
- moved R6 140.4 mm to (41.5, 56.0), turned to 90 degrees
- moved C109 140.3 mm to (53.5, 60.7), turned to 180 degrees
- moved D10 139.9 mm to (58.3, 54.6), turned to -90 degrees
- moved R46 139.3 mm to (49.1, 53.1), turned to -90 degrees
- moved R3 137.3 mm to (44.1, 53.3), turned to -90 degrees
- moved C99 137.1 mm to (55.1, 58.0), turned to 90 degrees
- moved C102 135.7 mm to (55.4, 66.6), turned to 90 degrees
- moved R45 135.6 mm to (52.5, 53.1), turned to -90 degrees
- moved D9 135.4 mm to (61.8, 54.6), turned to -90 degrees
- moved R5 135.3 mm to (45.9, 56.0), turned to 90 degrees
- moved R2 134.5 mm to (45.8, 53.3), turned to -90 degrees
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Connections:
- C73 pad 2: VAC_IN -> Current_ACS
- C80 pad 2: Current_ACS -> VAC_IN
- C90 pad 1: +3V3 -> GND2
- C90 pad 2: GND2 -> +3V3
- D14 pad 2: RS485_A -> GND2
- D14 pad 3: GND2 -> unconnected-(D14-Pad3)
- D15 pad 1: UART1_RX -> UART1_TX
- D15 pad 2: UART1_TX -> UART1_RX
- J4 pad 1: +3V3 -> GND2
- J4 pad 4: GND2 -> +3V3
- R65 pad 1: Net-(J4-Pin_2) -> Net-(J4-Pin_3)
- R66 pad 1: Net-(J4-Pin_3) -> Net-(J4-Pin_2)
- U13 pad 5: VAC_IN -> Current_ACS
- U13 pad 7: Current_ACS -> VAC_IN
- U14 pad 11: RS485_CONTROL -> unconnected-(U14A-PA1-Pad11)
- U14 pad 14: Voltage_Protection -> unconnected-(U14A-PA4-Pad14)
- U14 pad 16: unconnected-(U14A-PA6-Pad16) -> LED_TEST
- U14 pad 2: LED_TEST -> unconnected-(U14A-PC13-Pad2)
- U14 pad 21: unconnected-(U14A-PB10-Pad21) -> Voltage_Protection
- U14 pad 22: unconnected-(U14A-PB11-Pad22) -> RS485_CONTROL
Routing:
- net RS485_CONTROL: track 0.00 -> 94.9 mm, vias 0 -> 2
- net UART1_TX: track 0.00 -> 89.5 mm, vias 0 -> 2
- net UART2_TX: track 0.00 -> 85.5 mm, vias 0 -> 2
- net UART1_RX: track 0.00 -> 81.2 mm, vias 0 -> 2
- net PFC_VCC: track 222.6 -> 144.4 mm
- net UART2_RX: track 0.00 -> 77.9 mm, vias 0 -> 2
- net L_Gate_Opto: track 0.00 -> 61.6 mm, vias 0 -> 1
- net H_Gate_Opto: track 0.00 -> 48.7 mm, vias 0 -> 1
- net AC1: track 82.1 -> 34.2 mm
- net PFC_ON/OFF: track 1.52 -> 44.1 mm, vias 1 -> 3
- net VAC_IN: track 0.00 -> 41.3 mm, vias 0 -> 1
- net +3V3: track 0.00 -> 33.9 mm, vias 0 -> 4
- net Voltage_Protection: track 0.00 -> 33.9 mm, vias 0 -> 2
- net +5V: track 9.34 -> 37.3 mm, vias 0 -> 3
- net Voltage_LLC: track 7.83 -> 32.7 mm, vias 0 -> 1
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
Commit message: Update
Parts:
- added C112: 10uF/16V, charge_battery_footprint_lib:Ceramic_Cap_0603, B.Cu at (79.3, 76.7)
- added C113: 100nF/16V, charge_battery_footprint_lib:Ceramic_Cap_0603, B.Cu at (80.7, 76.7)
- added C114: 100nF/16V, charge_battery_footprint_lib:Ceramic_Cap_0603, B.Cu at (83.4, 76.7)
- added C115: 10uF/16V, charge_battery_footprint_lib:Ceramic_Cap_0603, B.Cu at (82.0, 76.7)
- added D9: LED_0603, charge_battery_footprint_lib:LED_0603, F.Cu at (30.0, 82.7)
- added Q9: LN2302LT1G, charge_battery_footprint_lib:SOT23, B.Cu at (81.7, 73.2)
- added R39: 10K/1%/1_10W, charge_battery_footprint_lib:Res_0603, F.Cu at (29.1, 84.0)
- added R69: 10K/1%/1_10W, charge_battery_footprint_lib:Res_0603, B.Cu at (79.6, 72.0)
- added R70: 10K/1%/1_10W, charge_battery_footprint_lib:Res_0603, B.Cu at (85.4, 75.3)
- R67: renamed from R63; moved to B.Cu
- R68: renamed from R64; moved to B.Cu
- moved C82 66.6 mm to (28.2, 98.9), turned to 90 degrees
- moved C79 60.7 mm to (25.9, 98.9), turned to 90 degrees
- moved C70 50.1 mm to (95.1, 75.4), turned to 90 degrees
- moved C73 45.8 mm to (92.7, 72.6), turned to 0 degrees
- moved C76 45.0 mm to (92.6, 77.6), turned to 180 degrees
- moved U13 42.3 mm to (91.2, 75.1), turned to 180 degrees
- moved C77 40.2 mm to (89.8, 72.6), turned to 180 degrees
- moved C69 38.8 mm to (89.5, 77.6), turned to 0 degrees
- moved C80 34.7 mm to (87.2, 73.9), turned to -90 degrees
- moved R67 6.10 mm to (36.2, 114.4)
- moved R68 3.93 mm to (40.0, 114.4)
- moved C43 3.48 mm to (44.0, 89.7)
- moved C54 3.48 mm to (44.6, 91.8)
- moved C47 3.48 mm to (33.4, 89.2)
- moved C49 3.48 mm to (32.0, 89.2)
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- renumbered D9 to D10, D10 to D11, D11 to D12, D12 to D13, D13 to D14, D14 to D15, D15 to D16, R39 to R40, R40 to R41, R41 to R42, R42 to R43, R43 to R44, R44 to R45, R45 to R46, R46 to R47, R47 to R48, R48 to R49, R67 to R50, R49 to R51, R50 to R52, R51 to R53, R52 to R54, R53 to R55, R54 to R56, R55 to R57, R56 to R58, R57 to R59, R58 to R60, R59 to R61, R65 to R62, R66 to R63, R60 to R64, R61 to R65, R62 to R66
Connections:
- C42 pad 2: +3.3V -> +3V3
- C44 pad 2: +3.3V -> +3V3
- C73 pad 2: Current_ACS -> Current_Measurement
- C77 pad 2: Current_Measurement -> Current_ACS
- C84 pad 2: +3.3V -> +3V3
- C85 pad 2: +3.3V -> +3V3
- C88 pad 2: +3.3V -> +3V3
- C89 pad 2: +3.3V -> +3V3
- Q6 pad 1: +3.3V -> +3V3
- Q7 pad 1: +3.3V -> +3V3
- R33 pad 1: +3.3V -> +3V3
- R51 pad 2: +3.3V -> +3V3
- R52 pad 2: +3.3V -> +3V3
- U13 pad 2: /STM32F103C8T6/ALERT/RDY -> ALERT_ADS1115
- U13 pad 5: Current_ACS -> Current_Measurement
- U13 pad 6: Current_Measurement -> Current_ACS
- U14 pad 38: unconnected-(U14A-PA15-Pad38) -> I2C_ALERT
Routing:
- net +3V3: track 33.9 -> 243.2 mm, vias 4 -> 18
- net Current_Measurement: track 15.5 -> 81.7 mm, vias 2 -> 4
- net GND2: track 67.5 -> 127.1 mm, vias 0 -> 5
- net AC1: track 34.2 -> 92.1 mm
- net Voltage_LLC: track 32.7 -> 82.8 mm, vias 1 -> 3
- net Current_ACS: track 15.3 -> 63.3 mm, vias 1 -> 3
- net Earth: track 4.41 -> 51.2 mm
- net I2C_ALERT: track 0.00 -> 38.1 mm, vias 0 -> 1
- net VAC_IN: track 41.3 -> 76.9 mm, vias 1 -> 3
- net RS485_CONTROL: track 94.9 -> 68.1 mm
- net SCL_ADS1115: track 12.9 -> 37.1 mm
- net GND1: track 19.2 -> 36.9 mm, vias 0 -> 1
- net ALERT_ADS1115: track 0.00 -> 14.3 mm, vias 0 -> 1
- net +3.3V: track 13.9 -> 0.00 mm, vias 1 -> 0
- net Net-(U11-+IN): track 12.4 -> 25.7 mm
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
Commit message: Update lib
Parts:
- moved C24 11.6 mm to (114.8, 116.9), turned to 90 degrees

Commit message: Update PCB PFC&LLC
Parts:
- C10, C11, C2, C28, C29, C3, C31, C32, C33, C34, C35, C36, C4, C40, C41, C42, C43, C44, C46, C47, C48, C49, C50, C51, C53, C54, C6, C67, C68, C7, C71, C72, C74, C75, C78, C79, C81, C82, D6, R2, R24, R25, R26, R27, R28, R29, R3, R30, R31, R32, R33, R34, R35, R36, R38, R5, R6, U2, U7, U8, U9: moved to F.Cu
- D4: value BYC10-600,127 -> 1N5408; footprint charge_battery_footprint_lib:TO-220-2_MCH -> charge_battery_footprint_lib:DO-201AD-2
- J2: footprint Connector_Phoenix_GMSTB:PhoenixContact_GMSTBA_2,5_2-G_1x02_P7.50mm_Horizontal -> Connector_Phoenix_MC:PhoenixContact_MC_1,5_2-G-3.81_1x02_P3.81mm_Horizontal
- L4: value Transformer -> EER35_Transformer_Horizontal; footprint charge_battery_footprint_lib:Transformer_ER35 -> charge_battery_footprint_lib:Transformer_ER35_Horizontal
- U5, U6: value 6N137M -> 6N137_SMD; footprint charge_battery_footprint_lib:DIP-8 -> charge_battery_footprint_lib:SOIC8_SMD
- moved R26 209.3 mm to (309.2, 77.3)
- moved R27 209.3 mm to (309.2, 88.4)
- moved C30 197.7 mm to (285.6, 108.2), turned to 180 degrees
- moved R28 195.9 mm to (280.7, 92.1), turned to 90 degrees
- moved Q4 195.0 mm to (282.3, 88.7), turned to -90 degrees
- moved C31 194.9 mm to (307.9, 78.7)
- moved C32 194.9 mm to (307.9, 89.7)
- moved C33 192.2 mm to (306.6, 78.7)
- moved C34 192.2 mm to (306.6, 89.7)
- moved R24 190.1 mm to (279.4, 86.5), turned to -90 degrees
- moved R17 187.6 mm to (273.3, 10.3), turned to 0 degrees
- moved R15 184.1 mm to (272.1, 6.88), turned to 0 degrees
- moved R29 184.0 mm to (280.7, 103.1), turned to 90 degrees
- moved Q5 182.8 mm to (282.4, 99.7), turned to -90 degrees
- moved R16 181.5 mm to (272.1, 2.92), turned to 0 degrees
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Connections:
- J2 pad 1: 51.2V -> GND2
- J2 pad 2: GND2 -> 51.2V
- L4 pad 2: GND1 -> (no net)
- L4 pad 3: Net-(L4-SA) -> (no net)
- L4 pad 4: GND2 -> (no net)
- L4 pad 5: Net-(L4-SB) -> (no net)
Routing:
- net Net-(C17-Pad2): track 58.3 -> 106.9 mm
- net Net-(L4-SA): track 45.2 -> 0.00 mm
- net /LLC/LOAD_M1_M2: track 60.7 -> 92.1 mm, vias 0 -> 3
- net Net-(U9-+IN): track 29.8 -> 58.8 mm
- net PFC_VCC: track 144.4 -> 164.2 mm
- net Net-(L4-AA): track 18.9 -> 0.00 mm
- net Net-(C17-Pad1): track 15.3 -> 33.8 mm
- net L_Gate_Driver: track 17.4 -> 35.5 mm
- net /LLC/OUT_M1: track 27.2 -> 40.5 mm
- net +9V: track 26.4 -> 38.9 mm
- net H_Gate_Driver: track 32.7 -> 44.7 mm
- net /LLC/OUT_M2: track 20.2 -> 29.4 mm
- net Voltage_LLC: track 82.8 -> 90.6 mm
- net +3V3: track 243.2 -> 250.6 mm
- net +12V: track 32.2 -> 39.4 mm
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Other:
- board size 116.9 x 98.2 mm -> 288 x 110.3 mm
