File: Hardware/Source/PFC & LLC/llc.kicad_sch (KiCad schematic)
At the start: 74 parts, among them J2 Conn_01x02_Socket, Q4 IPP60R125CP, Q5 IPP60R125CP, U10 OPAMP_OP07CSZ, U11 OPAMP_OP07CSZ, U12 ACS712ELCTR-05B-T, U5 6N137M, U6 6N137M, U7 IR2101, U8 OPAMP_OP07CSZ, U9 OPAMP_OP07CSZ

Commit message: layout PFC
Changed lines of the file:
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@@
 		(dnp no)
 		(property "Reference" "J2"
-			(at 280.67 114.2999 0)
+			(at 280.162 116.84 0)
 			(effects
 				(font
@@
 		)
 		(property "Value" "Conn_01x02_Socket"
-			(at 280.162 116.84 0)
+			(at 276.86 119.126 0)
 			(effects
 				(font

Commit message: Update Lib ER35 Transformer
Parts:
- L4: footprint charge_battery_footprint_lib:Transformer -> charge_battery_footprint_lib:Transformer_ER35
Changed lines of the file:
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@@
 			)
 		)
-		(property "Footprint" "charge_battery_footprint_lib:Transformer"
+		(property "Footprint" "charge_battery_footprint_lib:Transformer_ER35"
 			(at 125.222 127.254 0)
 			(effects

Commit message: Update
Parts:
- added D9: LED_0603, charge_battery_footprint_lib:LED_0603, symbol charge_battery_sym_lib:LED_0603
- added R39: 10K/1%/1_10W, charge_battery_footprint_lib:Res_0603, symbol charge_battery_sym_lib:Res_10K_0603_1%
- renumbered R39 to R40, R40 to R41, R41 to R42, R42 to R43
Connections:
- net 51.2V: now also D9.2 (A)
- net GND2: now also R39.2
- net +3.3V renamed +3V3
- new net: D9.1 (K), R39.1

Commit message: Update lib
Parts:
- removed L4: Transformer, charge_battery_footprint_lib:Transformer_ER35, symbol charge_battery_sym_lib:Transformer
- removed U5, U6: 6N137M, charge_battery_footprint_lib:DIP-8, symbol charge_battery_sym_lib:6N137M
- added L4: EER35_Transformer_Horizontal, charge_battery_footprint_lib:Transformer_ER35_Horizontal, symbol charge_battery_sym_lib:EER35_Transformer_Horizontal
- added U5, U6: 6N137_SMD, charge_battery_footprint_lib:SOIC8_SMD, symbol charge_battery_sym_lib:6N137_SMD
Connections:
- net +5V: now also U5.8 (VCC), U6.8 (VCC)
- net GND1: now also L4.8 (AB), U5.5 (GND), U6.5 (GND)
- net GND2: now also L4.11 (SC), L4.12 (SC), U5.3 (CATHODE), U6.3 (CATHODE)
- net H_Gate_Driver: now also U5.6 (VO)
- net L_Gate_Driver: now also U6.6 (VO)
- net at R27.2: now also U6.2 (ANODE)
- net at L3.2: now also L4.1 (AA)
- net at R26.2: now also U5.2 (ANODE)
- net at D7.2: now also L4.9 (SA)
- net at D8.2: now also L4.16 (SB)
Other:
- moved on the sheet: D8, R26, R27

Commit message: Update PCB PFC&LLC
Parts:
- J2: footprint Connector_Phoenix_GMSTB:PhoenixContact_GMSTBA_2,5_2-G_1x02_P7.50mm_Horizontal -> Connector_Phoenix_MC:PhoenixContact_MC_1,5_2-G-3.81_1x02_P3.81mm_Horizontal
Connections:
- net 51.2V: now also J2.2 (Pin_2); no longer J2.1 (Pin_1)
- net GND2: now also J2.1 (Pin_1); no longer J2.2 (Pin_2)
Other:
- moved on the sheet: D7, D8
Changed lines of the file:
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@@
 	(wire
 		(pts
-			(xy 271.78 114.3) (xy 274.32 114.3)
-		)
-		(stroke
-			(width 0)
-			(type default)
-		)
-	)
-	(wire
-		(pts
 			(xy 439.42 180.34) (xy 439.42 181.61)
 		)
@@
 	(wire
 		(pts
-			(xy 140.97 124.46) (xy 146.05 124.46)
+			(xy 140.97 124.46) (xy 149.86 124.46)
 		)
 		(stroke
@@
 	(wire
 		(pts
-			(xy 156.21 111.76) (xy 166.37 111.76)
+			(xy 160.02 111.76) (xy 166.37 111.76)
 		)
 		(stroke
@@
 	(wire
 		(pts
-			(xy 140.97 111.76) (xy 146.05 111.76)
+			(xy 140.97 111.76) (xy 149.86 111.76)
 		)
 		(stroke
@@
 	(wire
 		(pts
-			(xy 274.32 116.84) (xy 271.78 116.84)
-		)
-		(stroke
-			(width 0)
-			(type default)
-		)
-	)
-	(wire
-		(pts
 			(xy 360.68 158.75) (xy 368.3 158.75)
 		)
@@
 	(wire
 		(pts
-			(xy 156.21 124.46) (xy 166.37 124.46)
+			(xy 160.02 124.46) (xy 166.37 124.46)
 		)
 		(stroke
@@
 	(wire
 		(pts
+			(xy 271.78 114.3) (xy 274.32 114.3)
+		)
+		(stroke
+			(width 0)
+			(type default)
+		)
+	)
+	(wire
+		(pts
 			(xy 497.84 124.46) (xy 497.84 125.73)
 		)
@@
 	(wire
 		(pts
+			(xy 271.78 116.84) (xy 274.32 116.84)
+		)
+		(stroke
+			(width 0)
+			(type default)
+		)
+	)
+	(wire
+		(pts
 			(xy 115.57 236.22) (xy 115.57 238.76)
 		)
@@
 	(symbol
 		(lib_id "Connector:Conn_01x02_Socket")
-		(at 279.4 114.3 0)
+		(at 279.4 116.84 0)
+		(mirror x)
 		(unit 1)
 		(exclude_from_sim no)
@@
 		(dnp no)
 		(property "Reference" "J2"
-			(at 280.162 116.84 0)
+			(at 280.162 114.3 0)
 			(effects
 				(font
@@
 		)
 		(property "Value" "Conn_01x02_Socket"
-			(at 276.86 119.126 0)
+			(at 276.86 112.014 0)
 			(effects
 				(font
@@
 			)
 		)
-		(property "Footprint" "Connector_Phoenix_GMSTB:PhoenixContact_GMSTBA_2,5_2-G_1x02_P7.50mm_Horizontal"
-			(at 279.4 114.3 0)
+		(property "Footprint" "Connector_Phoenix_MC:PhoenixContact_MC_1,5_2-G-3.81_1x02_P3.81mm_Horizontal"
+			(at 279.4 116.84 0)
 			(effects
 				(font
@@
 		)
 		(property "Datasheet" "~"
-			(at 279.4 114.3 0)
+			(at 279.4 116.84 0)
 			(effects
 				(font
@@
 		)
 		(property "Description" "Generic connector, single row, 01x02, script generated"
-			(at 279.4 114.3 0)
+			(at 279.4 116.84 0)
 			(effects
 				(font
@@
 	(symbol
 		(lib_id "charge_battery_sym_lib:IDH06G65C6")
-		(at 151.13 111.76 0)
+		(at 154.94 111.76 0)
 		(unit 1)
 		(exclude_from_sim no)
@@
 		(dnp no)
 		(property "Reference" "D7"
-			(at 151.13 106.426 0)
+			(at 154.94 106.426 0)
 			(effects
 				(font
@@
 		)
 		(property "Value" "IDH06G65C6"
-			(at 151.13 108.712 0)
+			(at 154.94 108.712 0)
 			(effects
 				(font
@@
 		)
 		(property "Footprint" "charge_battery_footprint_lib:TO-220-2_MCH"
-			(at 139.7 94.488 0)
+			(at 143.51 94.488 0)
 			(effects
 				(font
@@
 		)
 		(property "Datasheet" "https://www.mouser.vn/datasheet/2/196/Infineon_IDH06G65C6_DS_v02_00_EN-1131100.pdf"
-			(at 147.066 94.234 0)
+			(at 150.876 94.234 0)
 			(effects
 				(font
@@
 		)
 		(property "Description" "Schottky Diodes & Rectifiers SIC DIODES"
-			(at 148.336 93.98 0)
+			(at 152.146 93.98 0)
 			(effects
 				(font
@@
 		)
 		(property "Supply name" "Mouser"
-			(at 147.32 94.996 0)
+			(at 151.13 94.996 0)
 			(effects
 				(font
@@
 		)
 		(property "Supply part number" "726-IDH06G65C6XKSA1"
-			(at 145.034 94.234 0)
+			(at 148.844 94.234 0)
 			(effects
 				(font
@@
 		)
 		(property "Supply URL" "https://www.mouser.vn/ProductDetail/Infineon-Technologies/IDH06G65C6XKSA1?qs=HXFqYaX1Q2y0Eo%2FTJueHsw%3D%3D"
-			(at 147.066 94.234 0)
+			(at 150.876 94.234 0)
 			(effects
 				(font
@@
 		)
 		(property " Supply part number" ""
-			(at 151.13 111.76 0)
+			(at 154.94 111.76 0)
 			(effects
 				(font
@@
 		)
 		(property "Field7" ""
-			(at 151.13 111.76 0)
+			(at 154.94 111.76 0)
 			(effects
 				(font
@@
 		)
 		(property "Sim.Device" ""
-			(at 151.13 111.76 0)
+			(at 154.94 111.76 0)
 			(effects
 				(font
@@
 		)
 		(property "Sim.Pins" ""
-			(at 151.13 111.76 0)
+			(at 154.94 111.76 0)
 			(effects
 				(font
@@
 		)
 		(property "Supply part name" ""
-			(at 151.13 111.76 0)
+			(at 154.94 111.76 0)
 			(effects
 				(font
@@
 	(symbol
 		(lib_id "charge_battery_sym_lib:IDH06G65C6")
-		(at 151.13 124.46 0)
+		(at 154.94 124.46 0)
 		(unit 1)
 		(exclude_from_sim no)
@@
 		(dnp no)
 		(property "Reference" "D8"
-			(at 151.13 127.508 0)
+			(at 154.94 127.508 0)
 			(effects
 				(font
@@
 		)
 		(property "Value" "IDH06G65C6"
-			(at 151.13 129.794 0)
+			(at 154.94 129.794 0)
 			(effects
 				(font
@@
 		)
 		(property "Footprint" "charge_battery_footprint_lib:TO-220-2_MCH"
-			(at 139.7 107.188 0)
+			(at 143.51 107.188 0)
 			(effects
 				(font
@@
 		)
 		(property "Datasheet" "https://www.mouser.vn/datasheet/2/196/Infineon_IDH06G65C6_DS_v02_00_EN-1131100.pdf"
-			(at 147.066 106.934 0)
+			(at 150.876 106.934 0)
 			(effects
 				(font
@@
 		)
 		(property "Description" "Schottky Diodes & Rectifiers SIC DIODES"
-			(at 148.336 106.68 0)
+			(at 152.146 106.68 0)
 			(effects
 				(font
@@
 		)
 		(property "Supply name" "Mouser"
-			(at 147.32 107.696 0)
+			(at 151.13 107.696 0)
 			(effects
 				(font
@@
 		)
 		(property "Supply part number" "726-IDH06G65C6XKSA1"
-			(at 145.034 106.934 0)
+			(at 148.844 106.934 0)
 			(effects
 				(font
@@
 		)
 		(property "Supply URL" "https://www.mouser.vn/ProductDetail/Infineon-Technologies/IDH06G65C6XKSA1?qs=HXFqYaX1Q2y0Eo%2FTJueHsw%3D%3D"
-			(at 147.066 106.934 0)
+			(at 150.876 106.934 0)
 			(effects
 				(font
@@
 		)
 		(property " Supply part number" ""
-			(at 151.13 124.46 0)
+			(at 154.94 124.46 0)
 			(effects
 				(font
@@
 		)
 		(property "Field7" ""
-			(at 151.13 124.46 0)
+			(at 154.94 124.46 0)
 			(effects
 				(font
@@
 		)
 		(property "Sim.Device" ""
-			(at 151.13 124.46 0)
+			(at 154.94 124.46 0)
 			(effects
 				(font
@@
 		)
 		(property "Sim.Pins" ""
-			(at 151.13 124.46 0)
+			(at 154.94 124.46 0)
 			(effects
 				(font
@@
 		)
 		(property "Supply part name" ""
-			(at 151.13 124.46 0)
+			(at 154.94 124.46 0)
 			(effects
 				(font

Commit message: Update Lib: Res_100mR
Parts:
- removed R37: R_Shunt_50mR, charge_battery_footprint_lib:R_Shunt, symbol charge_battery_sym_lib:R_Shunt_50mR
- added R37: 50mR/2512/1%, charge_battery_footprint_lib:Res_2512, symbol charge_battery_sym_lib:Res_50mR_2512_1%
Connections:
- net 51.2V: now also R37.2
- net R_Shunt_Voltage: now also R37.1
Changed lines of the file:
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@@
 	)
 	(symbol
-		(lib_id "charge_battery_sym_lib:R_Shunt_50mR")
-		(at 233.68 111.76 0)
-		(unit 1)
-		(exclude_from_sim no)
-		(in_bom yes)
-		(on_board yes)
-		(dnp no)
-		(property "Reference" "R37"
-			(at 235.458 114.554 0)
-			(effects
-				(font
-					(size 1.27 1.27)
-				)
-				(justify left)
-			)
-		)
-		(property "Value" "R_Shunt_50mR"
-			(at 230.886 116.84 0)
-			(effects
-				(font
-					(size 1.27 1.27)
-				)
-				(justify left)
-			)
-		)
-		(property "Footprint" "charge_battery_footprint_lib:R_Shunt"
-			(at 215.9 95.25 0)
-			(effects
-				(font
-					(size 1.27 1.27)
-				)
-				(hide yes)
-			)
-		)
-		(property "Datasheet" "~"
-			(at 226.314 96.012 90)
-			(effects
-				(font
-					(size 1.27 1.27)
-				)
-				(hide yes)
-			)
-		)
-		(property "Description" "Shunt resistor"
-			(at 222.504 96.266 0)
-			(effects
-				(font
-					(size 1.27 1.27)
-				)
-				(hide yes)
-			)
-		)
-		(property "Supply name" "BanLinhKien"
-			(at 218.059 96.393 0)
-			(effects
-				(font
-					(size 1.27 1.27)
-				)
-				(hide yes)
-			)
-		)
-		(property "Supply part number" "Trở Shunt 50mR 1.2x10x7MM"
-			(at 218.059 96.393 0)
-			(effects
-				(font
-					(size 1.27 1.27)
-				)
-				(hide yes)
-			)
-		)
-		(property "Supply URL" "https://banlinhkien.com/tro-shunt-50mr-10x6.5mm-p15749443.html"
-			(at 218.059 96.393 0)
-			(effects
-				(font
-					(size 1.27 1.27)
-				)
-				(hide yes)
-			)
-		)
-		(property " Supply part number" ""
-			(at 233.68 111.76 0)
-			(effects
-				(font
-					(size 1.27 1.27)
-				)
-				(hide yes)
-			)
-		)
-		(property "Field7" ""
-			(at 233.68 111.76 0)
-			(effects
-				(font
-					(size 1.27 1.27)
-				)
-				(hide yes)
-			)
-		)
-		(property "Sim.Device" ""
-			(at 233.68 111.76 0)
-			(effects
-				(font
-					(size 1.27 1.27)
-				)
-				(hide yes)
-			)
-		)
-		(property "Sim.Pins" ""
-			(at 233.68 111.76 0)
-			(effects
-				(font
-					(size 1.27 1.27)
-				)
-				(hide yes)
-			)
-		)
-		(property "Supply part name" ""
-			(at 233.68 111.76 0)
-			(effects
-				(font
-					(size 1.27 1.27)
-				)
-				(hide yes)
-			)
-		)
-		(pin "1"
-		)
-		(pin "2"
-		)
-		(instances
-			(project "PFC & LLC"
-				(path "/97d1a1fe-d5a5-4da8-b78a-88a9132d14ad/c86e0501-622e-4a08-a50b-30d27954cac4"
-					(reference "R37")
-					(unit 1)
-				)
-			)
-		)
-	)
-	(symbol
 		(lib_id "power:+9V")
 		(at 389.89 118.11 0)
@@
 					(unit 1)
 				)
+			)
+		)
+	)
+	(symbol
+		(lib_id "charge_battery_sym_lib:Res_50mR_2512_1%")
+		(at 237.49 109.22 0)
+		(unit 1)
+		(exclude_from_sim no)
+		(in_bom yes)
+		(on_board yes)
+		(dnp no)
+		(property "Reference" "R37"
+			(at 237.744 107.188 0)
+			(effects
+				(font
+					(size 1.27 1.27)
+				)
+			)
+		)
+		(property "Value" "50mR/2512/1%"
+			(at 237.744 109.474 0)
+			(effects
+				(font
+					(size 1.27 1.27)
+				)
+			)
+		)
+		(property "Footprint" "charge_battery_footprint_lib:Res_2512"
+			(at 237.49 114.808 0)
+			(effects
+				(font
+					(size 1.27 1.27)
+				)
+				(hide yes)
+			)
+		)
+		(property "Datasheet" ""
+			(at 237.49 109.22 0)
+			(effects
+				(font
+					(size 1.27 1.27)
+				)
+				(hide yes)
+			)
+		)
+		(property "Description" "Current Sense Resistors - SMD 4W 0.05 Ohms 1%"
+			(at 237.49 109.22 0)
+			(effects
+				(font
+					(size 1.27 1.27)
+				)
+				(hide yes)
+			)
+		)
+		(property "Supply Name" "Mouser"
+			(at 237.744 115.062 0)
+			(effects
+				(font
+					(size 1.27 1.27)
+				)
+				(hide yes)
+			)
+		)
+		(property "Supply Part Number" "660-TLRH3APTTE50L0F"
+			(at 237.998 115.062 0)
+			(effects
+				(font
+					(size 1.27 1.27)
+				)
+				(hide yes)
+			)
+		)
+		(property "Supply URL" "https://www.mouser.vn/ProductDetail/KOA-Speer/TLRH3APTTE50L0F?qs=eArw%252Bdd9rguJ2eBTdOyx8Q%3D%3D"
+			(at 237.49 115.316 0)
+			(effects
+				(font
+					(size 1.27 1.27)
+				)
+				(hide yes)
+			)
+		)
+		(pin "2"
+		)
+		(pin "1"
+		)
+		(instances
+			(project ""
+				(path "/97d1a1fe-d5a5-4da8-b78a-88a9132d14ad/c86e0501-622e-4a08-a50b-30d27954cac4"
+					(reference "R37")
+					(unit 1)
+				)

Commit message: Update PFC&LLC
Parts:
- renumbered C28 to C30, C29 to C31, C30 to C32, C31 to C33, C32 to C34, C33 to C35, C34 to C36, C35 to C37, C36 to C38, C37 to C39, C38 to C40, C39 to C41, C40 to C42, C41 to C43, C42 to C44, C43 to C45, C44 to C46, C45 to C47, C46 to C48, C47 to C49, C48 to C50, C49 to C51, C50 to C52, C51 to C53, C52 to C54, C53 to C55, C54 to C56, C55 to C57, C56 to C58, C57 to C59, C58 to C60, C59 to C61, C60 to C62, C61 to C63, C62 to C64, C63 to C65, C64 to C66, C65 to C67, C66 to C68
