File: Hardware/Source/PFC & LLC/detect_battery.kicad_sch (KiCad schematic)
At the start: 9 parts, among them J3 CHARGER, K2 Relay 12VDC 10A, Q9 MMBT2222A, U18 PC817X2NIPW

Commit message: update lib, LLC
Parts:
- added C109, C110, C112: 100nF/16V, charge_battery_footprint_lib:Ceramic_Cap_0603, symbol charge_battery_sym_lib:Ceramic_Cap_SMD_100nF_16V
- added C111, C113: 10uF/16V, charge_battery_footprint_lib:Ceramic_Cap_0603, symbol charge_battery_sym_lib:Ceramic_Cap_SMD_10uF_16V
- added NT12: GNDD_GNDPWR, NetTie:NetTie-2_SMD_Pad0.5mm, symbol Device:NetTie_2
- added R54: 10K/1%/1_10W, charge_battery_footprint_lib:Res_0603, symbol charge_battery_sym_lib:Res_10K_0603_1%
- added R57: 510R/1%/1_10W, charge_battery_footprint_lib:Res_0603, symbol charge_battery_sym_lib:Res_510R_0603_1%
- added R58: 680K/1%/1_10W, charge_battery_footprint_lib:Res_0603, symbol charge_battery_sym_lib:Res_680K_0603_1%
- added R59: 47K/1%/1_10W, charge_battery_footprint_lib:Res_0603, symbol charge_battery_sym_lib:Res_47K_0603_1%
- added U16: SN74LVC1G14DBVR, charge_battery_footprint_lib:SOT-23-5, symbol charge_battery_sym_lib:SN74LVC1G14DBVR
- added U18: PC817X2NIPW, charge_battery_footprint_lib:PC817X2NIPW, symbol charge_battery_sym_lib:PC817X2NIPW
- added U19: MCP601T-I/OT, charge_battery_footprint_lib:SOT-23-5, symbol charge_battery_sym_lib:MCP601T-I_OT
- renumbered D13 to D18, D20 to D19, J3 to J4, K2 to K1, Q9 to Q7, R53 to R55, R54 to R56, R61 to R60, U18 to U17
Connections:
- net +3V3: now also C110.2, C111.2, U16.5 (VCC), U18.4 (C)
- net GND: now also C112.1, C113.1, R59.1, U18.2 (K), U19.2 (V-), U19.3 (IN+)
- net GNDPWR: now also C110.1, C111.1, NT12.2, U16.3 (GND)
- net RELAY_ENABLE_CHARGER renamed DETECT_BATTERY_CONNECTOR
- net DETECT_BATTERY_CONNECTOR: now also R58.2
- new net: R57.1, U18.1 (A)
- new net: R54.2, U16.2, U18.3 (E)
- new net: R58.1, R59.2, U19.4 (IN-)
- new net: R57.2, U19.1
- new net +5V_GND: C112.2, C113.2, U19.5 (V+)
- new net DETECT_BATTERY: C109.2, U16.4
- new net GNDD: C109.1, NT12.1, R54.1
Other:
- moved on the sheet: D18, D19, J4, K1, Q7, R55, R56, R60, U17

Commit message: update lib, LLC
Parts:
- removed R55: 220/1%/1_10W, charge_battery_footprint_lib:Res_0603, symbol charge_battery_sym_lib:Res_220R_0603_1%
- added D19: LED_0805, charge_battery_footprint_lib:LED_0805, symbol charge_battery_sym_lib:LED_0805
- added R59: 1K/1%/1_10W, charge_battery_footprint_lib:Res_0603, symbol charge_battery_sym_lib:Res_1K_0603_1%
- added R61: 220/1%/1_10W, charge_battery_footprint_lib:Res_0603, symbol charge_battery_sym_lib:Res_220R_0603_1%
- renumbered D18 to D20, D19 to D21, R54 to R60, R56 to R62, R57 to R63, R58 to R64, R59 to R65, R60 to R66
Connections:
- net +3V3: now also D19.2 (A), R61.2
- net at U17.1 (A): now also R61.1
- net Voltage_Protection renamed CONTROL_CHARGER
- net CONTROL_CHARGER: now also R59.1
- new net: D19.1 (K), R59.2

Commit message: update LLC
Parts:
- renumbered C109 to C111, C110 to C112, C111 to C113, C112 to C114, C113 to C115, R59 to R58, R60 to R59, R61 to R60, R62 to R61, R63 to R62, R64 to R63, R65 to R64, R66 to R65
