File: Hardware/Source/PFC & LLC/enable_LLC_PFC.kicad_sch (KiCad schematic)
At the start: 17 parts, among them K2 Relay 12VDC 10A, Q8 MMBT2222A, Q9 MMBT2222A, U20 PC817X2NIPW, U21 SN74LVC1G14DBVR, U22 MCP601T-I/OT, U23 SN74LVC1G14DBVR

Commit message: update lib, LLC
Parts:
- removed R69: 1K/1%/1_10W, charge_battery_footprint_lib:Res_0603, symbol charge_battery_sym_lib:Res_1K_0603_1%
- added C124, C128: 100nF/16V, charge_battery_footprint_lib:Ceramic_Cap_0603, symbol charge_battery_sym_lib:Ceramic_Cap_SMD_100nF_16V
- added C125: 10uF/16V, charge_battery_footprint_lib:Ceramic_Cap_0603, symbol charge_battery_sym_lib:Ceramic_Cap_SMD_10uF_16V
- added D28: LED_0805, charge_battery_footprint_lib:LED_0805, symbol charge_battery_sym_lib:LED_0805
- added R73, R77: 1K/1%/1_10W, charge_battery_footprint_lib:Res_0603, symbol charge_battery_sym_lib:Res_1K_0603_1%
- added R76: 10K/1%/1_10W, charge_battery_footprint_lib:Res_0603, symbol charge_battery_sym_lib:Res_10K_0603_1%
- renumbered C127 to C126, C128 to C127, C124 to C129, C125 to C130, C126 to C131, D26 to D29, R67 to R74, R68 to R75, R70 to R78, U22 to U21, U23 to U22, U21 to U23
Connections:
- net +3V3: now also C126.2, C127.2, U21.3 (IN+), U22.5 (VCC), D28.2 (A)
- net +5V: now also U21.5 (V+), C124.2, C125.2; no longer C126.2, C127.2
- net GNDPWR: now also U21.2 (V-), U22.3 (GND), C124.1, C125.1, R76.1
- net Voltage_Protection: now also R73.1
- net at Q9.1 (B): now also R77.1
- net at C129.2, R78.2, U23.4: now also R77.2
- net at U22.2: now also U21.1
- net PFC_OPERATION: now reaches U22.4
- net PFC_OPERATION: now also C128.2
- net UCC_FEEDBACK_ENABLE: now reaches U21.4 (IN-)
- net UCC_FEEDBACK_ENABLE: now also R76.2
- new net: D28.1 (K), R73.2
- new net GNDD: C128.1
Other:
- moved on the sheet: C126, C127, C131, D29, K2, Q8, R74, R75, U20, U21, U22

Commit message: update LLC
Parts:
- renumbered C124 to C126, C125 to C127, C126 to C128, C127 to C129, C128 to C130, C129 to C131, C130 to C132, C131 to C133, R73 to R72, R74 to R73, R75 to R74, R76 to R75, R77 to R76, R78 to R77
