File: Hardware/Source/PFC & LLC/AC_voltage_measurement.kicad_sch (KiCad schematic)
At the start: 17 parts, among them U5 OP07CSZ, U6 MCP1525T-I/TT

Commit message: update FEEDBACK, AC
Parts:
- removed C10: 1nF/50V, charge_battery_footprint_lib:Ceramic_Cap_0603, symbol charge_battery_sym_lib:Ceramic_Cap_SMD_1nF_50V
- removed C11: 100nF/16V, charge_battery_footprint_lib:Ceramic_Cap_0603, symbol charge_battery_sym_lib:Ceramic_Cap_SMD_100nF_16V
- removed C26: 10uF/16V, charge_battery_footprint_lib:Ceramic_Cap_0603, symbol charge_battery_sym_lib:Ceramic_Cap_SMD_10uF_16V
- removed R22, R8: 10K/1%/1_10W, charge_battery_footprint_lib:Res_0603, symbol charge_battery_sym_lib:Res_10K_0603_1%
- removed R6: 1M/1%/1_10W, charge_battery_footprint_lib:Res_0603, symbol charge_battery_sym_lib:Res_1M_0603_1%
- added C47, C53, C57: 100nF/16V, charge_battery_footprint_lib:Ceramic_Cap_0603, symbol charge_battery_sym_lib:Ceramic_Cap_SMD_100nF_16V
- added C48, C54, C59: 10uF/16V, charge_battery_footprint_lib:Ceramic_Cap_0603, symbol charge_battery_sym_lib:Ceramic_Cap_SMD_10uF_16V
- added C55, C56: 10nF/50V, charge_battery_footprint_lib:Ceramic_Cap_0603, symbol charge_battery_sym_lib:Ceramic_Cap_SMD_10nF_50V
- added C58: 1nF/50V, charge_battery_footprint_lib:Ceramic_Cap_0603, symbol charge_battery_sym_lib:Ceramic_Cap_SMD_1nF_50V
- added R30: 1M/1%/1_10W, charge_battery_footprint_lib:Res_0603, symbol charge_battery_sym_lib:Res_1M_0603_1%
- added R31, R32: 18K/1%/1_10W, charge_battery_footprint_lib:Res_0603, symbol charge_battery_sym_lib:Res_18K_0603_1%
- added R33, R34, R35, R36: 100K/1%/1_10W, charge_battery_footprint_lib:Res_0603, symbol charge_battery_sym_lib:Res_100K_0603_1%
- added U7: OP07CSZ, charge_battery_footprint_lib:SOIC-8, symbol charge_battery_sym_lib:OP07CSZ
- renumbered C14 to C49, C6 to C50, C7 to C51, C27 to C52, C28 to C60, C29 to C61, C31 to C62, C30 to C63, R5 to R29, U5 to U6, U6 to U8
Connections:
- net +9V: now also C57.2, C59.2, U7.7 (V+)
- net -9V: now also C47.2, C48.2, C53.2, C54.2, U7.4 (V-)
- net AC1: now also R30.1
- net GNDA: now also C50.2, C47.1, C48.1, C53.1, C54.1, C57.1, C58.1, C59.1, R31.1, R34.1
- net VAC_IN: now also C56.2, C58.2, R36.2, U7.6; no longer C51.2, U6.6
- net at C50.1, R29.2, U6.3 (+): now also R31.2
- net at C51.1, U6.2 (-): now also R30.2, R32.2
- net VREF_2.5V renamed VREF_2.5V_1
- net VREF_2.5V_1: now also C55.2, R35.2; no longer C50.2
- new net: C56.1, R34.2, R36.1, U7.2 (-)
- new net: C55.1, R33.2, R35.1, U7.3 (+)
- new net: C51.2, R32.1, R33.1, U6.6
- no-connect marks 2 -> 4
Other:
- moved on the sheet: C49, C50, C51, C52, C60, C61, C62, C63, R29, U6, U8

Commit message: update lib, LLC
Parts:
- renumbered C47 to C44, C48 to C45, C49 to C46, C50 to C47, C51 to C48, C52 to C49, C53 to C50, C54 to C51, C55 to C52, C56 to C53, C57 to C54, C58 to C55, C59 to C56, C60 to C57, C61 to C58, C62 to C59, C63 to C60, R29 to R30, R30 to R31, R31 to R32, R32 to R33, R33 to R34, R34 to R35, R35 to R36, R36 to R37, U6 to U4, U7 to U5, U8 to U6

Commit message: update lib, LLC
Parts:
- renumbered R30 to R35, R31 to R36, R32 to R37, R33 to R38, R34 to R39, R35 to R40, R36 to R41, R37 to R42
Changed lines of the file:
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@@
 		(on_board yes)
 		(dnp no)
-		(property "Reference" "R35"
+		(property "Reference" "R40"
 			(at 125.476 81.28 0)
 			(effects
@@
 			(project "PFC & LLC"
 				(path "/97d1a1fe-d5a5-4da8-b78a-88a9132d14ad/52d31f6b-fecd-464b-82e3-66e05e655a74"
-					(reference "R35")
+					(reference "R40")
 					(unit 1)
 				)
@@
 		(on_board yes)
 		(dnp no)
-		(property "Reference" "R31"
+		(property "Reference" "R36"
 			(at 60.452 78.994 0)
 			(effects
@@
 			(project "PFC & LLC"
 				(path "/97d1a1fe-d5a5-4da8-b78a-88a9132d14ad/52d31f6b-fecd-464b-82e3-66e05e655a74"
-					(reference "R31")
+					(reference "R36")
 					(unit 1)
 				)
@@
 		(on_board yes)
 		(dnp no)
-		(property "Reference" "#PWR065"
+		(property "Reference" "#PWR066"
 			(at 186.69 102.87 0)
 			(effects
@@
 			(project "PFC & LLC"
 				(path "/97d1a1fe-d5a5-4da8-b78a-88a9132d14ad/52d31f6b-fecd-464b-82e3-66e05e655a74"
-					(reference "#PWR065")
+					(reference "#PWR066")
 					(unit 1)
 				)
@@
 		(on_board yes)
 		(dnp no)
-		(property "Reference" "R32"
+		(property "Reference" "R37"
 			(at 99.314 55.88 0)
 			(effects
@@
 			(project "PFC & LLC"
 				(path "/97d1a1fe-d5a5-4da8-b78a-88a9132d14ad/52d31f6b-fecd-464b-82e3-66e05e655a74"
-					(reference "R32")
+					(reference "R37")
 					(unit 1)
 				)
@@
 		(on_board yes)
 		(dnp no)
-		(property "Reference" "R30"
+		(property "Reference" "R35"
 			(at 60.452 73.914 0)
 			(effects
@@
 			(project "PFC & LLC"
 				(path "/97d1a1fe-d5a5-4da8-b78a-88a9132d14ad/52d31f6b-fecd-464b-82e3-66e05e655a74"
-					(reference "R30")
+					(reference "R35")
 					(unit 1)
 				)
@@
 		(on_board yes)
 		(dnp no)
-		(property "Reference" "#PWR059"
+		(property "Reference" "#PWR060"
 			(at 149.86 127 0)
 			(effects
@@
 			(project "PFC & LLC"
 				(path "/97d1a1fe-d5a5-4da8-b78a-88a9132d14ad/52d31f6b-fecd-464b-82e3-66e05e655a74"
-					(reference "#PWR059")
+					(reference "#PWR060")
 					(unit 1)
 				)
@@
 		(on_board yes)
 		(dnp no)
-		(property "Reference" "#PWR069"
+		(property "Reference" "#PWR070"
 			(at 238.76 114.3 0)
 			(effects
@@
 			(project "PFC & LLC"
 				(path "/97d1a1fe-d5a5-4da8-b78a-88a9132d14ad/52d31f6b-fecd-464b-82e3-66e05e655a74"
-					(reference "#PWR069")
+					(reference "#PWR070")
 					(unit 1)
 				)
@@
 		(on_board yes)
 		(dnp no)
-		(property "Reference" "R33"
+		(property "Reference" "R38"
 			(at 99.314 93.98 0)
 			(effects
@@
 			(project "PFC & LLC"
 				(path "/97d1a1fe-d5a5-4da8-b78a-88a9132d14ad/52d31f6b-fecd-464b-82e3-66e05e655a74"
-					(reference "R33")
+					(reference "R38")
 					(unit 1)
 				)
@@
 		(on_board yes)
 		(dnp no)
-		(property "Reference" "#PWR067"
+		(property "Reference" "#PWR068"
 			(at 238.76 87.63 0)
 			(effects
@@
 			(project "PFC & LLC"
 				(path "/97d1a1fe-d5a5-4da8-b78a-88a9132d14ad/52d31f6b-fecd-464b-82e3-66e05e655a74"
-					(reference "#PWR067")
+					(reference "#PWR068")
 					(unit 1)
 				)
@@
 		(on_board yes)
 		(dnp no)
-		(property "Reference" "R34"
+		(property "Reference" "R39"
 			(at 125.476 76.2 0)
 			(effects
@@
 			(project ""
 				(path "/97d1a1fe-d5a5-4da8-b78a-88a9132d14ad/52d31f6b-fecd-464b-82e3-66e05e655a74"
-					(reference "R34")
+					(reference "R39")
 					(unit 1)
 				)
@@
 		(on_board yes)
 		(dnp no)
-		(property "Reference" "#PWR063"
+		(property "Reference" "#PWR064"
 			(at 185.42 127 0)
 			(effects
@@
 			(project "PFC & LLC"
 				(path "/97d1a1fe-d5a5-4da8-b78a-88a9132d14ad/52d31f6b-fecd-464b-82e3-66e05e655a74"
-					(reference "#PWR063")
+					(reference "#PWR064")
 					(unit 1)
 				)
@@
 		(on_board yes)
 		(dnp no)
-		(property "Reference" "#PWR061"
+		(property "Reference" "#PWR062"
 			(at 156.21 74.93 0)
 			(effects
@@
 			(project "PFC & LLC"
 				(path "/97d1a1fe-d5a5-4da8-b78a-88a9132d14ad/52d31f6b-fecd-464b-82e3-66e05e655a74"
-					(reference "#PWR061")
+					(reference "#PWR062")
 					(unit 1)
 				)
@@
 		(on_board yes)
 		(dnp no)
-		(property "Reference" "#PWR052"
+		(property "Reference" "#PWR053"
 			(at 66.04 143.51 0)
 			(effects
@@
 			(project "PFC & LLC"
 				(path "/97d1a1fe-d5a5-4da8-b78a-88a9132d14ad/52d31f6b-fecd-464b-82e3-66e05e655a74"
-					(reference "#PWR052")
+					(reference "#PWR053")
 					(unit 1)
 				)
@@
 		(on_board yes)
 		(dnp no)
-		(property "Reference" "#PWR058"
+		(property "Reference" "#PWR059"
 			(at 119.38 92.71 0)
 			(effects
@@
 			(project "PFC & LLC"
 				(path "/97d1a1fe-d5a5-4da8-b78a-88a9132d14ad/52d31f6b-fecd-464b-82e3-66e05e655a74"
-					(reference "#PWR058")
+					(reference "#PWR059")
 					(unit 1)
 				)
@@
 		(on_board yes)
 		(dnp no)
-		(property "Reference" "#PWR060"
+		(property "Reference" "#PWR061"
 			(at 149.86 143.51 0)
 			(effects
@@
 			(project "PFC & LLC"
 				(path "/97d1a1fe-d5a5-4da8-b78a-88a9132d14ad/52d31f6b-fecd-464b-82e3-66e05e655a74"
-					(reference "#PWR060")
+					(reference "#PWR061")
 					(unit 1)
 				)
@@
 		(on_board yes)
 		(dnp no)
-		(property "Reference" "#PWR064"
+		(property "Reference" "#PWR065"
 			(at 185.42 143.51 0)
 			(effects
@@
 			(project "PFC & LLC"
 				(path "/97d1a1fe-d5a5-4da8-b78a-88a9132d14ad/52d31f6b-fecd-464b-82e3-66e05e655a74"
-					(reference "#PWR064")
+					(reference "#PWR065")
 					(unit 1)
 				)
@@
 		(dnp no)
 		(fields_autoplaced yes)
-		(property "Reference" "#PWR066"
+		(property "Reference" "#PWR067"
 			(at 238.76 62.23 0)
 			(effects
@@
 			(project "PFC & LLC"
 				(path "/97d1a1fe-d5a5-4da8-b78a-88a9132d14ad/52d31f6b-fecd-464b-82e3-66e05e655a74"
-					(reference "#PWR066")
+					(reference "#PWR067")
 					(unit 1)
 				)
@@
 		(on_board yes)
 		(dnp no)
-		(property "Reference" "#PWR055"
+		(property "Reference" "#PWR056"
 			(at 101.6 127 0)
 			(effects
@@
 			(project "PFC & LLC"
 				(path "/97d1a1fe-d5a5-4da8-b78a-88a9132d14ad/52d31f6b-fecd-464b-82e3-66e05e655a74"
-					(reference "#PWR055")
+					(reference "#PWR056")
 					(unit 1)
 				)
@@
 		(on_board yes)
 		(dnp no)
-		(property "Reference" "R37"
+		(property "Reference" "R42"
 			(at 163.83 102.87 0)
 			(effects
@@
 			(project "PFC & LLC"
 				(path "/97d1a1fe-d5a5-4da8-b78a-88a9132d14ad/52d31f6b-fecd-464b-82e3-66e05e655a74"
-					(reference "R37")
+					(reference "R42")
 					(unit 1)
 				)
@@
 		(on_board yes)
 		(dnp no)
-		(property "Reference" "#PWR057"
+		(property "Reference" "#PWR058"
 			(at 115.57 66.04 0)
 			(effects
@@
 			(project "PFC & LLC"
 				(path "/97d1a1fe-d5a5-4da8-b78a-88a9132d14ad/52d31f6b-fecd-464b-82e3-66e05e655a74"
-					(reference "#PWR057")
+					(reference "#PWR058")
 					(unit 1)
 				)
@@
 		(on_board yes)
 		(dnp no)
-		(property "Reference" "#PWR056"
+		(property "Reference" "#PWR057"
 			(at 101.6 143.51 0)
 			(effects
@@
 			(project "PFC & LLC"
 				(path "/97d1a1fe-d5a5-4da8-b78a-88a9132d14ad/52d31f6b-fecd-464b-82e3-66e05e655a74"
-					(reference "#PWR056")
+					(reference "#PWR057")
 					(unit 1)
 				)
@@
 		(on_board yes)
 		(dnp no)
-		(property "Reference" "#PWR053"
+		(property "Reference" "#PWR054"
 			(at 97.79 72.39 0)
 			(effects
@@
 			(project "PFC & LLC"
 				(path "/97d1a1fe-d5a5-4da8-b78a-88a9132d14ad/52d31f6b-fecd-464b-82e3-66e05e655a74"
-					(reference "#PWR053")
+					(reference "#PWR054")
 					(unit 1)
 				)
@@
 		(on_board yes)
 		(dnp no)
-		(property "Reference" "#PWR051"
+		(property "Reference" "#PWR052"
 			(at 66.04 127 0)
 			(effects
@@
 			(project "PFC & LLC"
 				(path "/97d1a1fe-d5a5-4da8-b78a-88a9132d14ad/52d31f6b-fecd-464b-82e3-66e05e655a74"
-					(reference "#PWR051")
+					(reference "#PWR052")
 					(unit 1)
 				)
@@
 		(on_board yes)
 		(dnp no)
-		(property "Reference" "#PWR054"
+		(property "Reference" "#PWR055"
 			(at 97.79 82.55 0)
 			(effects
@@
 			(project "PFC & LLC"
 				(path "/97d1a1fe-d5a5-4da8-b78a-88a9132d14ad/52d31f6b-fecd-464b-82e3-66e05e655a74"
-					(reference "#PWR054")
+					(reference "#PWR055")
 					(unit 1)
 				)
@@
 		(dnp no)
 		(fields_autoplaced yes)
-		(property "Reference" "#PWR068"
+		(property "Reference" "#PWR069"
 			(at 238.76 99.06 0)
 			(effects
@@
 			(project "PFC & LLC"
 				(path "/97d1a1fe-d5a5-4da8-b78a-88a9132d14ad/52d31f6b-fecd-464b-82e3-66e05e655a74"
-					(reference "#PWR068")
+					(reference "#PWR069")
 					(unit 1)
 				)
@@
 		(on_board yes)
 		(dnp no)
-		(property "Reference" "R36"
+		(property "Reference" "R41"
 			(at 163.83 53.34 0)
 			(effects
@@
 			(project "PFC & LLC"
 				(path "/97d1a1fe-d5a5-4da8-b78a-88a9132d14ad/52d31f6b-fecd-464b-82e3-66e05e655a74"
-					(reference "R36")
+					(reference "R41")
 					(unit 1)
 				)
@@
 		(on_board yes)
 		(dnp no)
-		(property "Reference" "#PWR062"
+		(property "Reference" "#PWR063"
 			(at 156.21 85.09 0)
 			(effects
@@
 			(project "PFC & LLC"
 				(path "/97d1a1fe-d5a5-4da8-b78a-88a9132d14ad/52d31f6b-fecd-464b-82e3-66e05e655a74"
-					(reference "#PWR062")
+					(reference "#PWR063")
 					(unit 1)
 				)

Commit message: update LLC
Parts:
- removed R37, R38: 18K/1%/1_10W, charge_battery_footprint_lib:Res_0603, symbol charge_battery_sym_lib:Res_18K_0603_1%
- added R36, R37: 5k1/1%/1_8W, charge_battery_footprint_lib:Res_0805, symbol charge_battery_sym_lib:Res_5k1_0805_1%
- renumbered C44 to C46, C45 to C47, C46 to C48, C47 to C49, C48 to C50, C49 to C51, C50 to C52, C51 to C53, C52 to C54, C53 to C55, C54 to C56, C55 to C57, C56 to C58, C57 to C59, C58 to C60, C59 to C61, C60 to C62, R35 to R34, R36 to R35, R39 to R38, R40 to R39, R41 to R40, R42 to R41
Connections:
- net GNDA: now also R36.2
- net at C49.1, R34.2, U4.3 (+): now also R36.1
- net at C50.1, R35.2, U4.2 (-): now also R37.1
- net at C50.2, R38.1, U4.6: now also R37.2
