File: Hardware/Source/PFC & LLC/adc_external.kicad_sch (KiCad schematic)
At the start: 9 parts, among them U8 ADS1115IDGS

Commit message: update FEEDBACK, AC
Parts:
- removed C32: 100nF/16V, charge_battery_footprint_lib:Ceramic_Cap_0603, symbol charge_battery_sym_lib:Ceramic_Cap_SMD_100nF_16V
- removed C34, C35, C37: 1nF/50V, charge_battery_footprint_lib:Ceramic_Cap_0603, symbol charge_battery_sym_lib:Ceramic_Cap_SMD_1nF_50V
- removed C36: 10uF/16V, charge_battery_footprint_lib:Ceramic_Cap_0603, symbol charge_battery_sym_lib:Ceramic_Cap_SMD_10uF_16V
- removed TP3: VAC IN, TestPoint:TestPoint_Bridge_Pitch2.0mm_Drill0.7mm, symbol Connector:TestPoint
- removed TP4: Voltage LLC, TestPoint:TestPoint_Bridge_Pitch2.0mm_Drill0.7mm, symbol Connector:TestPoint
- removed TP5: Current ACS, TestPoint:TestPoint_Bridge_Pitch2.0mm_Drill0.7mm, symbol Connector:TestPoint
- removed U8: ADS1115IDGS, charge_battery_footprint_lib:VSSOP-10, symbol charge_battery_sym_lib:ADS1115IDGS
- added C95, C96, C97: 1nF/50V, charge_battery_footprint_lib:Ceramic_Cap_0603, symbol charge_battery_sym_lib:Ceramic_Cap_SMD_1nF_50V
- added C98: 10uF/16V, charge_battery_footprint_lib:Ceramic_Cap_0603, symbol charge_battery_sym_lib:Ceramic_Cap_SMD_10uF_16V
- added C99: 100nF/16V, charge_battery_footprint_lib:Ceramic_Cap_0603, symbol charge_battery_sym_lib:Ceramic_Cap_SMD_100nF_16V
- added U17: ADS1115IDGS, charge_battery_footprint_lib:VSSOP-10, symbol charge_battery_sym_lib:ADS1115IDGS
Connections:
- net +5V: now also C98.2, C99.2, U17.8 (VDD)
- net ALERT_ADS1115: now also U17.2 (ALERT/RDY)
- net Current_ACS: now also C95.2, U17.6 (AIN2)
- net GNDA: now also C95.1, C96.1, C97.1
- net GNDPWR: now also C98.1, C99.1, U17.3 (GND)
- net SCL_ADS1115: now also U17.10 (SCL)
- net SDA_ADS1115: now also U17.9 (SDA)
- net VAC_IN: now also C97.2, U17.4 (AIN0)
- net Voltage_LLC: now also C96.2, U17.5 (AIN1)
- new net GNDD: U17.1 (ADDR)

Commit message: update lib, LLC
Parts:
- added D15, D16, D17: BZT52-C5V1, charge_battery_footprint_lib:Diode_Zener_BZT52H, symbol charge_battery_sym_lib:BZT52-C5V1
- renumbered C95 to C92, C96 to C93, C97 to C94, C98 to C95, C99 to C96, U17 to U15
Connections:
- net Current_ACS: now also D15.1 (K)
- net GNDA: now also D15.2 (A), D16.2 (A), D17.2 (A)
- net VAC_IN: now also D17.1 (K)
- net Voltage_LLC: now also D16.1 (K)
Other:
- moved on the sheet: C92, C93, C94, C95, C96, U15

Commit message: update lib, LLC
Parts:
- renumbered D15 to D16, D16 to D17, D17 to D18
Changed lines of the file:
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@@
 		(on_board yes)
 		(dnp no)
-		(property "Reference" "#PWR0114"
+		(property "Reference" "#PWR0115"
 			(at 116.84 99.06 0)
 			(effects
@@
 			(project "PFC & LLC"
 				(path "/97d1a1fe-d5a5-4da8-b78a-88a9132d14ad/e834f355-1206-4dc4-b161-ae801911fe6e"
-					(reference "#PWR0114")
+					(reference "#PWR0115")
 					(unit 1)
 				)
@@
 		(dnp no)
 		(fields_autoplaced yes)
-		(property "Reference" "#PWR0119"
+		(property "Reference" "#PWR0120"
 			(at 189.23 99.06 0)
 			(effects
@@
 			(project "PFC & LLC"
 				(path "/97d1a1fe-d5a5-4da8-b78a-88a9132d14ad/e834f355-1206-4dc4-b161-ae801911fe6e"
-					(reference "#PWR0119")
+					(reference "#PWR0120")
 					(unit 1)
 				)
@@
 		(on_board yes)
 		(dnp no)
-		(property "Reference" "#PWR0118"
+		(property "Reference" "#PWR0119"
 			(at 189.23 66.04 0)
 			(effects
@@
 			(project "PFC & LLC"
 				(path "/97d1a1fe-d5a5-4da8-b78a-88a9132d14ad/e834f355-1206-4dc4-b161-ae801911fe6e"
-					(reference "#PWR0118")
+					(reference "#PWR0119")
 					(unit 1)
 				)
@@
 		(dnp no)
 		(fields_autoplaced yes)
-		(property "Reference" "#PWR0117"
+		(property "Reference" "#PWR0118"
 			(at 185.42 130.81 0)
 			(effects
@@
 			(project "PFC & LLC"
 				(path "/97d1a1fe-d5a5-4da8-b78a-88a9132d14ad/e834f355-1206-4dc4-b161-ae801911fe6e"
-					(reference "#PWR0117")
+					(reference "#PWR0118")
 					(unit 1)
 				)
@@
 		(on_board yes)
 		(dnp no)
-		(property "Reference" "#PWR0113"
+		(property "Reference" "#PWR0114"
 			(at 85.09 99.06 0)
 			(effects
@@
 			(project "PFC & LLC"
 				(path "/97d1a1fe-d5a5-4da8-b78a-88a9132d14ad/e834f355-1206-4dc4-b161-ae801911fe6e"
-					(reference "#PWR0113")
+					(reference "#PWR0114")
 					(unit 1)
 				)
@@
 		(dnp no)
 		(fields_autoplaced yes)
-		(property "Reference" "#PWR0120"
+		(property "Reference" "#PWR0121"
 			(at 208.28 100.33 0)
 			(effects
@@
 			(project "PFC & LLC"
 				(path "/97d1a1fe-d5a5-4da8-b78a-88a9132d14ad/e834f355-1206-4dc4-b161-ae801911fe6e"
-					(reference "#PWR0120")
+					(reference "#PWR0121")
 					(unit 1)
 				)
@@
 		(on_board yes)
 		(dnp no)
-		(property "Reference" "#PWR0115"
+		(property "Reference" "#PWR0116"
 			(at 149.86 99.06 0)
 			(effects
@@
 			(project "PFC & LLC"
 				(path "/97d1a1fe-d5a5-4da8-b78a-88a9132d14ad/e834f355-1206-4dc4-b161-ae801911fe6e"
-					(reference "#PWR0115")
+					(reference "#PWR0116")
 					(unit 1)
 				)
@@
 		(on_board yes)
 		(dnp no)
-		(property "Reference" "#PWR0116"
+		(property "Reference" "#PWR0117"
 			(at 185.42 116.84 0)
 			(effects
@@
 			(project "PFC & LLC"
 				(path "/97d1a1fe-d5a5-4da8-b78a-88a9132d14ad/e834f355-1206-4dc4-b161-ae801911fe6e"
-					(reference "#PWR0116")
+					(reference "#PWR0117")
 					(unit 1)
 				)
@@
 		(dnp no)
 		(fields_autoplaced yes)
-		(property "Reference" "D16"
+		(property "Reference" "D17"
 			(at 133.35 83.8199 90)
 			(effects
@@
 			(project "PFC & LLC"
 				(path "/97d1a1fe-d5a5-4da8-b78a-88a9132d14ad/e834f355-1206-4dc4-b161-ae801911fe6e"
-					(reference "D16")
+					(reference "D17")
 					(unit 1)
 				)
@@
 		(dnp no)
 		(fields_autoplaced yes)
-		(property "Reference" "D15"
+		(property "Reference" "D16"
 			(at 101.6 83.8199 90)
 			(effects
@@
 			(project "PFC & LLC"
 				(path "/97d1a1fe-d5a5-4da8-b78a-88a9132d14ad/e834f355-1206-4dc4-b161-ae801911fe6e"
-					(reference "D15")
+					(reference "D16")
 					(unit 1)
 				)
@@
 		(dnp no)
 		(fields_autoplaced yes)
-		(property "Reference" "D17"
+		(property "Reference" "D18"
 			(at 166.37 83.8199 90)
 			(effects
@@
 			(project ""
 				(path "/97d1a1fe-d5a5-4da8-b78a-88a9132d14ad/e834f355-1206-4dc4-b161-ae801911fe6e"
-					(reference "D17")
-					(unit 1)
-				)
+					(reference "D18")
+					(unit 1)
+				)

Commit message: update LLC
Parts:
- renumbered C92 to C94, C93 to C95, C94 to C96, C95 to C97, C96 to C98
Changed lines of the file:
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@@
 		(dnp no)
 		(fields_autoplaced yes)
-		(property "Reference" "C93"
+		(property "Reference" "C95"
 			(at 120.65 83.8199 90)
 			(effects
@@
 			(project "PFC & LLC"
 				(path "/97d1a1fe-d5a5-4da8-b78a-88a9132d14ad/e834f355-1206-4dc4-b161-ae801911fe6e"
-					(reference "C93")
+					(reference "C95")
 					(unit 1)
 				)
@@
 		(on_board yes)
 		(dnp no)
-		(property "Reference" "C95"
+		(property "Reference" "C97"
 			(at 187.706 118.872 90)
 			(effects
@@
 			(project "PFC & LLC"
 				(path "/97d1a1fe-d5a5-4da8-b78a-88a9132d14ad/e834f355-1206-4dc4-b161-ae801911fe6e"
-					(reference "C95")
+					(reference "C97")
 					(unit 1)
 				)
@@
 		(on_board yes)
 		(dnp no)
-		(property "Reference" "#PWR0115"
+		(property "Reference" "#PWR0122"
 			(at 116.84 99.06 0)
 			(effects
@@
 			(project "PFC & LLC"
 				(path "/97d1a1fe-d5a5-4da8-b78a-88a9132d14ad/e834f355-1206-4dc4-b161-ae801911fe6e"
-					(reference "#PWR0115")
+					(reference "#PWR0122")
 					(unit 1)
 				)
@@
 		(on_board yes)
 		(dnp no)
-		(property "Reference" "C96"
+		(property "Reference" "C98"
 			(at 203.2 119.126 90)
 			(effects
@@
 			(project "PFC & LLC"
 				(path "/97d1a1fe-d5a5-4da8-b78a-88a9132d14ad/e834f355-1206-4dc4-b161-ae801911fe6e"
-					(reference "C96")
+					(reference "C98")
 					(unit 1)
 				)
@@
 		(dnp no)
 		(fields_autoplaced yes)
-		(property "Reference" "#PWR0120"
+		(property "Reference" "#PWR0127"
 			(at 189.23 99.06 0)
 			(effects
@@
 			(project "PFC & LLC"
 				(path "/97d1a1fe-d5a5-4da8-b78a-88a9132d14ad/e834f355-1206-4dc4-b161-ae801911fe6e"
-					(reference "#PWR0120")
+					(reference "#PWR0127")
 					(unit 1)
 				)
@@
 		(on_board yes)
 		(dnp no)
-		(property "Reference" "#PWR0119"
+		(property "Reference" "#PWR0126"
 			(at 189.23 66.04 0)
 			(effects
@@
 			(project "PFC & LLC"
 				(path "/97d1a1fe-d5a5-4da8-b78a-88a9132d14ad/e834f355-1206-4dc4-b161-ae801911fe6e"
-					(reference "#PWR0119")
+					(reference "#PWR0126")
 					(unit 1)
 				)
@@
 		(dnp no)
 		(fields_autoplaced yes)
-		(property "Reference" "C94"
+		(property "Reference" "C96"
 			(at 153.67 83.8199 90)
 			(effects
@@
 			(project "PFC & LLC"
 				(path "/97d1a1fe-d5a5-4da8-b78a-88a9132d14ad/e834f355-1206-4dc4-b161-ae801911fe6e"
-					(reference "C94")
+					(reference "C96")
 					(unit 1)
 				)
@@
 		(dnp no)
 		(fields_autoplaced yes)
-		(property "Reference" "#PWR0118"
+		(property "Reference" "#PWR0125"
 			(at 185.42 130.81 0)
 			(effects
@@
 			(project "PFC & LLC"
 				(path "/97d1a1fe-d5a5-4da8-b78a-88a9132d14ad/e834f355-1206-4dc4-b161-ae801911fe6e"
-					(reference "#PWR0118")
+					(reference "#PWR0125")
 					(unit 1)
 				)
@@
 		(on_board yes)
 		(dnp no)
-		(property "Reference" "#PWR0114"
+		(property "Reference" "#PWR0121"
 			(at 85.09 99.06 0)
 			(effects
@@
 			(project "PFC & LLC"
 				(path "/97d1a1fe-d5a5-4da8-b78a-88a9132d14ad/e834f355-1206-4dc4-b161-ae801911fe6e"
-					(reference "#PWR0114")
+					(reference "#PWR0121")
 					(unit 1)
 				)
@@
 		(dnp no)
 		(fields_autoplaced yes)
-		(property "Reference" "#PWR0121"
+		(property "Reference" "#PWR0128"
 			(at 208.28 100.33 0)
 			(effects
@@
 			(project "PFC & LLC"
 				(path "/97d1a1fe-d5a5-4da8-b78a-88a9132d14ad/e834f355-1206-4dc4-b161-ae801911fe6e"
-					(reference "#PWR0121")
+					(reference "#PWR0128")
 					(unit 1)
 				)
@@
 		(on_board yes)
 		(dnp no)
-		(property "Reference" "#PWR0116"
+		(property "Reference" "#PWR0123"
 			(at 149.86 99.06 0)
 			(effects
@@
 			(project "PFC & LLC"
 				(path "/97d1a1fe-d5a5-4da8-b78a-88a9132d14ad/e834f355-1206-4dc4-b161-ae801911fe6e"
-					(reference "#PWR0116")
+					(reference "#PWR0123")
 					(unit 1)
 				)
@@
 		(dnp no)
 		(fields_autoplaced yes)
-		(property "Reference" "C92"
+		(property "Reference" "C94"
 			(at 88.9 83.8199 90)
 			(effects
@@
 			(project ""
 				(path "/97d1a1fe-d5a5-4da8-b78a-88a9132d14ad/e834f355-1206-4dc4-b161-ae801911fe6e"
-					(reference "C92")
+					(reference "C94")
 					(unit 1)
 				)
@@
 		(on_board yes)
 		(dnp no)
-		(property "Reference" "#PWR0117"
+		(property "Reference" "#PWR0124"
 			(at 185.42 116.84 0)
 			(effects
@@
 			(project "PFC & LLC"
 				(path "/97d1a1fe-d5a5-4da8-b78a-88a9132d14ad/e834f355-1206-4dc4-b161-ae801911fe6e"
-					(reference "#PWR0117")
-					(unit 1)
-				)
+					(reference "#PWR0124")
+					(unit 1)
+				)
