File: Hardware/Source/PFC & LLC/feedback_llc.kicad_sch (KiCad schematic)
At the start: 0 parts

Commit message: update FEEDBACK, AC
Parts:
- added C64, C67, C68, C73, C79, C81, C83, C84, C87, C89, C93, C94: 10uF/16V, charge_battery_footprint_lib:Ceramic_Cap_0603, symbol charge_battery_sym_lib:Ceramic_Cap_SMD_10uF_16V
- added C65, C66, C69, C71, C74, C75, C76, C78, C80, C82, C85, C86, C90, C92: 100nF/16V, charge_battery_footprint_lib:Ceramic_Cap_0603, symbol charge_battery_sym_lib:Ceramic_Cap_SMD_100nF_16V
- added C70, C72: 1nF/50V, charge_battery_footprint_lib:Ceramic_Cap_0603, symbol charge_battery_sym_lib:Ceramic_Cap_SMD_1nF_50V
- added C77: 1pF/50V, charge_battery_footprint_lib:Ceramic_Cap_0603, symbol charge_battery_sym_lib:Ceramic_Cap_SMD_1pF_50V
- added C88, C91: 1nF/50V, charge_battery_footprint_lib:Ceramic_Cap_Hole_5mm, symbol charge_battery_sym_lib:Ceramic_Cap_Hole_1nF_50V
- added FB2, FB3: 120R, Inductor_SMD:L_0805_2012Metric, symbol Device:L_Small
- added NT4: GND_GNDAMC, NetTie:NetTie-2_SMD_Pad0.5mm, symbol Device:NetTie_2
- added NT5: GNDA_GNDPWR, NetTie:NetTie-2_SMD_Pad0.5mm, symbol Device:NetTie_2
- added R37: 15K/1%/1_10W, charge_battery_footprint_lib:Res_0603, symbol charge_battery_sym_lib:Res_15K_0603_1%
- added R38: 1K/1%/1_10W, charge_battery_footprint_lib:Res_0603, symbol charge_battery_sym_lib:Res_1K_0603_1%
- added R39, R44: 220K/1%/1_10W, charge_battery_footprint_lib:Res_0603, symbol charge_battery_sym_lib:Res_220K_0603_1%
- added R40, R41: 12K/1%/1_10W, charge_battery_footprint_lib:Res_0603, symbol charge_battery_sym_lib:Res_12K_0603_1%
- added R42, R46: 680K/1%/1_10W, charge_battery_footprint_lib:Res_0603, symbol charge_battery_sym_lib:Res_680K_0603_1%
- added R43, R45: 68K/1%/1_10W, charge_battery_footprint_lib:Res_0603, symbol charge_battery_sym_lib:Res_68K_0603_1%
- added U10: AMC1351QDWVRQ1, charge_battery_footprint_lib:SOIC_8_DWV0008A, symbol charge_battery_sym_lib:AMC1351QDWVRQ1
- added U11, U12: MCP1525T-I/TT, charge_battery_footprint_lib:SOT23, symbol charge_battery_sym_lib:MCP1525T-I_TT
- added U13, U14, U15, U16: OP07CSZ, charge_battery_footprint_lib:SOIC-8, symbol charge_battery_sym_lib:OP07CSZ
- added U9: ACS712ELCTR-05B-T, charge_battery_footprint_lib:SOIC-8, symbol charge_battery_sym_lib:ACS712ELCTR-05B-T
Connections:
- new net: C70.2, U9.6 (FILTER)
- new net: R41.1, U9.7 (VIOUT)
- new net: R41.2, R43.2, U13.3 (+)
- new net: C72.1, U10.6 (OUTN)
- new net: C72.2, R39.1, U10.7 (OUTP)
- new net: C77.2, R39.2, R42.2, U14.3 (+)
- new net: R40.2, R45.1, U13.2 (-)
- new net: R45.2, U13.6, U15.3 (+)
- new net: R46.1, U14.6, U16.3 (+)
- new net: NT4.2, U10.3 (GND1), U10.4 (GND1)
- new net: R44.2, R46.2, U14.2 (-)
- new net +3V3: U11.1 (VIN), U12.1 (VIN)
- new net +5V: C68.2, C71.2, FB3.1, U9.8 (VCC)
- new net +5V_GND: C64.2, C65.2, FB2.1
- new net +9V: C80.2, C82.2, C83.2, C84.2, C90.2, C92.2, C93.2, C94.2, U13.7 (V+), U14.7 (V+), U15.7 (V+), U16.7 (V+)
- new net -9V: C76.2, C78.2, C79.2, C81.2, C85.2, C86.2, C87.2, C89.2, U13.4 (V-), U14.4 (V-), U15.4 (V-), U16.4 (V-)
- new net ACS_OUTPUT: U9.3 (IP-), U9.4 (IP-)
- new net AMC_VDD1: C66.2, FB2.2, U10.1 (VDD1)
- new net AMC_VDD2: C74.2, FB3.2, U10.8 (VDD2)
- new net Current_ACS: C88.2, U15.2 (-), U15.6
- new net GND: C64.1, C65.1, C66.1, NT4.1, R38.1
- new net GNDA: C67.1, C68.1, C69.1, C70.1, C71.1, C73.1, C74.1, C75.1, C76.1, C77.1, C78.1, C79.1, C80.1, C81.1, C82.1, C83.1, C84.1, C85.1, C86.1, C87.1, C88.1, C89.1, C90.1, C91.1, C92.1, C93.1, C94.1, NT5.1, R42.1, R43.1, U10.5 (GND2), U11.3 (VSS), U12.3 (VSS), U9.5 (GND)
- new net GNDPWR: NT5.2
- new net LLC_FEEDBACK_VOLTAGE: R37.1, R38.2, U10.2 (IN)
- new net LLC_OUTPUT: R37.2, U9.1 (IP+), U9.2 (IP+)
- new net VREF_2.5V_2: C67.2, C69.2, R40.1, U11.2 (VOUT)
- new net VREF_2.5V_3: C73.2, C75.2, R44.1, U12.2 (VOUT)
- new net Voltage_LLC: C91.2, U16.2 (-), U16.6
- no-connect marks 0 -> 8
Other:
- note added: "CURRENT FEEDBACK"
- note added: "VOLTAGE FEEDBACK"

Commit message: update lib, LLC
Parts:
- renumbered C64 to C61, C65 to C62, C66 to C63, C67 to C64, C68 to C65, C69 to C66, C70 to C67, C71 to C68, C72 to C69, C73 to C70, C74 to C71, C75 to C72, C76 to C73, C77 to C74, C78 to C75, C79 to C76, C80 to C77, C81 to C78, C82 to C79, C83 to C80, C84 to C81, C85 to C82, C86 to C83, C87 to C84, C88 to C85, C89 to C86, C90 to C87, C91 to C88, C92 to C89, C93 to C90, C94 to C91, NT4 to NT10, NT5 to NT11, R37 to R38, R38 to R39, R39 to R40, R40 to R41, R41 to R42, R42 to R43, R43 to R44, R44 to R45, R45 to R46, R46 to R47, U12 to U10, U13 to U11, U14 to U12, U15 to U13, U16 to U14, U9 to U7, U10 to U8, U11 to U9

Commit message: update lib, LLC
Parts:
- renumbered R38 to R43, R39 to R44, R40 to R45, R41 to R46, R42 to R47, R43 to R48, R44 to R49, R45 to R50, R46 to R51, R47 to R52

Commit message: update LLC
Parts:
- removed U8: AMC1351QDWVRQ1, charge_battery_footprint_lib:SOIC_8_DWV0008A, symbol charge_battery_sym_lib:AMC1351QDWVRQ1
- added U8: AMC1350DWVR, charge_battery_footprint_lib:SOIC_8_DWV0008A, symbol charge_battery_sym_lib:AMC1350DWVR
- renumbered C61 to C63, C62 to C64, C63 to C65, C64 to C66, C65 to C67, C66 to C68, C67 to C69, C68 to C70, C69 to C71, C70 to C72, C71 to C73, C72 to C74, C73 to C75, C74 to C76, C75 to C77, C76 to C78, C77 to C79, C78 to C80, C79 to C81, C80 to C82, C81 to C83, C82 to C84, C83 to C85, C84 to C86, C85 to C87, C86 to C88, C87 to C89, C88 to C90, C89 to C91, C90 to C92, C91 to C93, R43 to R42, R44 to R43, R45 to R44, R46 to R45, R47 to R46, R48 to R47, R49 to R48, R50 to R49, R51 to R50, R52 to R51
Connections:
- net AMC_VDD1: now also U8.1 (VDD1)
- net AMC_VDD2: now also U8.8 (VDD2)
- net GNDA: now also U8.5 (GND2)
- net LLC_FEEDBACK_VOLTAGE: now also U8.2 (INN)
- net at C71.1: now also U8.6 (OUTN)
- net at C71.2, R44.1: now also U8.7 (OUTP)
- net at NT10.2: now also U8.3 (INP), U8.4 (GND1)
