File: Hardware/Source/PFC & LLC/level_shifting.kicad_sch (KiCad schematic)
At the start: 0 parts

Commit message: update FEEDBACK, AC
Parts:
- added C100, C101, C102, C106, C107, C108: 10uF/16V, charge_battery_footprint_lib:Ceramic_Cap_0603, symbol charge_battery_sym_lib:Ceramic_Cap_SMD_10uF_16V
- added C103, C104, C105, C109, C110, C111: 100nF/16V, charge_battery_footprint_lib:Ceramic_Cap_0603, symbol charge_battery_sym_lib:Ceramic_Cap_SMD_100nF_16V
- added Q6, Q7, Q8: LN2302LT1G, charge_battery_footprint_lib:SOT23, symbol charge_battery_sym_lib:LN2302LT1G
- added R47, R48, R49, R50, R51, R52: 4K7/1%/1_10W, charge_battery_footprint_lib:Res_0603, symbol charge_battery_sym_lib:Res_4K7_0603_1%
Connections:
- new net +3V3: C100.2, C101.2, C102.2, C103.2, C104.2, C105.2, Q6.1 (G), Q7.1 (G), Q8.1 (G), R47.2, R48.2, R49.2
- new net +5V: C106.2, C107.2, C108.2, C109.2, C110.2, C111.2, R50.2, R51.2, R52.2
- new net ALERT_ADS1115: Q8.3 (D), R52.1
- new net GNDD: C100.1, C101.1, C102.1, C103.1, C104.1, C105.1, C106.1, C107.1, C108.1, C109.1, C110.1, C111.1
- new net I2C_ALERT: Q8.2 (S), R49.1
- new net I2C_SCL: Q6.2 (S), R47.1
- new net I2C_SDA: Q7.2 (S), R48.1
- new net SCL_ADS1115: Q6.3 (D), R50.1
- new net SDA_ADS1115: Q7.3 (D), R51.1

Commit message: update lib, LLC
Parts:
- renumbered C103 to C100, C104 to C101, C105 to C102, C106 to C103, C107 to C104, C108 to C105, C109 to C106, C110 to C107, C111 to C108, C100 to C97, C101 to C98, C102 to C99, Q6 to Q4, Q7 to Q5, Q8 to Q6, R47 to R48, R48 to R49, R49 to R50, R50 to R51, R51 to R52, R52 to R53

Commit message: update lib, LLC
Parts:
- renumbered R48 to R53, R49 to R54, R50 to R55, R51 to R56, R52 to R57, R53 to R58
Changed lines of the file:
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@@
 		(dnp no)
 		(fields_autoplaced yes)
-		(property "Reference" "#PWR0136"
+		(property "Reference" "#PWR0137"
 			(at 193.04 104.14 0)
 			(effects
@@
 			(project "PFC & LLC"
 				(path "/97d1a1fe-d5a5-4da8-b78a-88a9132d14ad/9cd95f3e-5010-4970-88ae-b8d7b603fb03"
-					(reference "#PWR0136")
+					(reference "#PWR0137")
 					(unit 1)
 				)
@@
 		(on_board yes)
 		(dnp no)
-		(property "Reference" "#PWR0123"
+		(property "Reference" "#PWR0124"
 			(at 90.17 57.15 0)
 			(effects
@@
 			(project "PFC & LLC"
 				(path "/97d1a1fe-d5a5-4da8-b78a-88a9132d14ad/9cd95f3e-5010-4970-88ae-b8d7b603fb03"
-					(reference "#PWR0123")
+					(reference "#PWR0124")
 					(unit 1)
 				)
@@
 		(on_board yes)
 		(dnp no)
-		(property "Reference" "#PWR0125"
+		(property "Reference" "#PWR0126"
 			(at 90.17 91.44 0)
 			(effects
@@
 			(project "PFC & LLC"
 				(path "/97d1a1fe-d5a5-4da8-b78a-88a9132d14ad/9cd95f3e-5010-4970-88ae-b8d7b603fb03"
-					(reference "#PWR0125")
+					(reference "#PWR0126")
 					(unit 1)
 				)
@@
 		(on_board yes)
 		(dnp no)
-		(property "Reference" "#PWR0128"
+		(property "Reference" "#PWR0129"
 			(at 142.24 87.63 0)
 			(effects
@@
 			(project "PFC & LLC"
 				(path "/97d1a1fe-d5a5-4da8-b78a-88a9132d14ad/9cd95f3e-5010-4970-88ae-b8d7b603fb03"
-					(reference "#PWR0128")
+					(reference "#PWR0129")
 					(unit 1)
 				)
@@
 		(on_board yes)
 		(dnp no)
-		(property "Reference" "R48"
+		(property "Reference" "R53"
 			(at 137.16 61.214 90)
 			(effects
@@
 			(project "PFC & LLC"
 				(path "/97d1a1fe-d5a5-4da8-b78a-88a9132d14ad/9cd95f3e-5010-4970-88ae-b8d7b603fb03"
-					(reference "R48")
+					(reference "R53")
 					(unit 1)
 				)
@@
 		(on_board yes)
 		(dnp no)
-		(property "Reference" "R51"
+		(property "Reference" "R56"
 			(at 161.29 59.944 90)
 			(effects
@@
 			(project "PFC & LLC"
 				(path "/97d1a1fe-d5a5-4da8-b78a-88a9132d14ad/9cd95f3e-5010-4970-88ae-b8d7b603fb03"
-					(reference "R51")
+					(reference "R56")
 					(unit 1)
 				)
@@
 		(dnp no)
 		(fields_autoplaced yes)
-		(property "Reference" "#PWR0126"
+		(property "Reference" "#PWR0127"
 			(at 90.17 106.68 0)
 			(effects
@@
 			(project "PFC & LLC"
 				(path "/97d1a1fe-d5a5-4da8-b78a-88a9132d14ad/9cd95f3e-5010-4970-88ae-b8d7b603fb03"
-					(reference "#PWR0126")
+					(reference "#PWR0127")
 					(unit 1)
 				)
@@
 		(on_board yes)
 		(dnp no)
-		(property "Reference" "#PWR0121"
+		(property "Reference" "#PWR0122"
 			(at 88.9 123.19 0)
 			(effects
@@
 			(project "PFC & LLC"
 				(path "/97d1a1fe-d5a5-4da8-b78a-88a9132d14ad/9cd95f3e-5010-4970-88ae-b8d7b603fb03"
-					(reference "#PWR0121")
+					(reference "#PWR0122")
 					(unit 1)
 				)
@@
 		(on_board yes)
 		(dnp no)
-		(property "Reference" "R49"
+		(property "Reference" "R54"
 			(at 137.16 94.234 90)
 			(effects
@@
 			(project "PFC & LLC"
 				(path "/97d1a1fe-d5a5-4da8-b78a-88a9132d14ad/9cd95f3e-5010-4970-88ae-b8d7b603fb03"
-					(reference "R49")
+					(reference "R54")
 					(unit 1)
 				)
@@
 		(dnp no)
 		(fields_autoplaced yes)
-		(property "Reference" "#PWR0122"
+		(property "Reference" "#PWR0123"
 			(at 88.9 138.43 0)
 			(effects
@@
 			(project "PFC & LLC"
 				(path "/97d1a1fe-d5a5-4da8-b78a-88a9132d14ad/9cd95f3e-5010-4970-88ae-b8d7b603fb03"
-					(reference "#PWR0122")
+					(reference "#PWR0123")
 					(unit 1)
 				)
@@
 		(on_board yes)
 		(dnp no)
-		(property "Reference" "R53"
+		(property "Reference" "R58"
 			(at 161.29 125.984 90)
 			(effects
@@
 			(project "PFC & LLC"
 				(path "/97d1a1fe-d5a5-4da8-b78a-88a9132d14ad/9cd95f3e-5010-4970-88ae-b8d7b603fb03"
-					(reference "R53")
+					(reference "R58")
 					(unit 1)
 				)
@@
 		(on_board yes)
 		(dnp no)
-		(property "Reference" "#PWR0129"
+		(property "Reference" "#PWR0130"
 			(at 142.24 120.65 0)
 			(effects
@@
 			(project "PFC & LLC"
 				(path "/97d1a1fe-d5a5-4da8-b78a-88a9132d14ad/9cd95f3e-5010-4970-88ae-b8d7b603fb03"
-					(reference "#PWR0129")
+					(reference "#PWR0130")
 					(unit 1)
 				)
@@
 		(on_board yes)
 		(dnp no)
-		(property "Reference" "#PWR0127"
+		(property "Reference" "#PWR0128"
 			(at 142.24 54.61 0)
 			(effects
@@
 			(project "PFC & LLC"
 				(path "/97d1a1fe-d5a5-4da8-b78a-88a9132d14ad/9cd95f3e-5010-4970-88ae-b8d7b603fb03"
-					(reference "#PWR0127")
+					(reference "#PWR0128")
 					(unit 1)
 				)
@@
 		(dnp no)
 		(fields_autoplaced yes)
-		(property "Reference" "#PWR0130"
+		(property "Reference" "#PWR0131"
 			(at 156.21 54.61 0)
 			(effects
@@
 			(project "PFC & LLC"
 				(path "/97d1a1fe-d5a5-4da8-b78a-88a9132d14ad/9cd95f3e-5010-4970-88ae-b8d7b603fb03"
-					(reference "#PWR0130")
+					(reference "#PWR0131")
 					(unit 1)
 				)
@@
 		(dnp no)
 		(fields_autoplaced yes)
-		(property "Reference" "#PWR0138"
+		(property "Reference" "#PWR0139"
 			(at 193.04 135.89 0)
 			(effects
@@
 			(project "PFC & LLC"
 				(path "/97d1a1fe-d5a5-4da8-b78a-88a9132d14ad/9cd95f3e-5010-4970-88ae-b8d7b603fb03"
-					(reference "#PWR0138")
+					(reference "#PWR0139")
 					(unit 1)
 				)
@@
 		(on_board yes)
 		(dnp no)
-		(property "Reference" "#PWR0133"
+		(property "Reference" "#PWR0134"
 			(at 193.04 54.61 0)
 			(effects
@@
 			(project "PFC & LLC"
 				(path "/97d1a1fe-d5a5-4da8-b78a-88a9132d14ad/9cd95f3e-5010-4970-88ae-b8d7b603fb03"
-					(reference "#PWR0133")
+					(reference "#PWR0134")
 					(unit 1)
 				)
@@
 		(on_board yes)
 		(dnp no)
-		(property "Reference" "#PWR0137"
+		(property "Reference" "#PWR0138"
 			(at 193.04 120.65 0)
 			(effects
@@
 			(project "PFC & LLC"
 				(path "/97d1a1fe-d5a5-4da8-b78a-88a9132d14ad/9cd95f3e-5010-4970-88ae-b8d7b603fb03"
-					(reference "#PWR0137")
+					(reference "#PWR0138")
 					(unit 1)
 				)
@@
 		(on_board yes)
 		(dnp no)
-		(property "Reference" "#PWR0135"
+		(property "Reference" "#PWR0136"
 			(at 193.04 88.9 0)
 			(effects
@@
 			(project "PFC & LLC"
 				(path "/97d1a1fe-d5a5-4da8-b78a-88a9132d14ad/9cd95f3e-5010-4970-88ae-b8d7b603fb03"
-					(reference "#PWR0135")
+					(reference "#PWR0136")
 					(unit 1)
 				)
@@
 		(on_board yes)
 		(dnp no)
-		(property "Reference" "R50"
+		(property "Reference" "R55"
 			(at 137.16 127.254 90)
 			(effects
@@
 			(project "PFC & LLC"
 				(path "/97d1a1fe-d5a5-4da8-b78a-88a9132d14ad/9cd95f3e-5010-4970-88ae-b8d7b603fb03"
-					(reference "R50")
+					(reference "R55")
 					(unit 1)
 				)
@@
 		(dnp no)
 		(fields_autoplaced yes)
-		(property "Reference" "#PWR0131"
+		(property "Reference" "#PWR0132"
 			(at 156.21 87.63 0)
 			(effects
@@
 			(project "PFC & LLC"
 				(path "/97d1a1fe-d5a5-4da8-b78a-88a9132d14ad/9cd95f3e-5010-4970-88ae-b8d7b603fb03"
-					(reference "#PWR0131")
+					(reference "#PWR0132")
 					(unit 1)
 				)
@@
 		(on_board yes)
 		(dnp no)
-		(property "Reference" "R52"
+		(property "Reference" "R57"
 			(at 161.29 92.964 90)
 			(effects
@@
 			(project "PFC & LLC"
 				(path "/97d1a1fe-d5a5-4da8-b78a-88a9132d14ad/9cd95f3e-5010-4970-88ae-b8d7b603fb03"
-					(reference "R52")
+					(reference "R57")
 					(unit 1)
 				)
@@
 		(dnp no)
 		(fields_autoplaced yes)
-		(property "Reference" "#PWR0124"
+		(property "Reference" "#PWR0125"
 			(at 90.17 72.39 0)
 			(effects
@@
 			(project "PFC & LLC"
 				(path "/97d1a1fe-d5a5-4da8-b78a-88a9132d14ad/9cd95f3e-5010-4970-88ae-b8d7b603fb03"
-					(reference "#PWR0124")
+					(reference "#PWR0125")
 					(unit 1)
 				)
@@
 		(dnp no)
 		(fields_autoplaced yes)
-		(property "Reference" "#PWR0134"
+		(property "Reference" "#PWR0135"
 			(at 193.04 69.85 0)
 			(effects
@@
 			(project "PFC & LLC"
 				(path "/97d1a1fe-d5a5-4da8-b78a-88a9132d14ad/9cd95f3e-5010-4970-88ae-b8d7b603fb03"
-					(reference "#PWR0134")
+					(reference "#PWR0135")
 					(unit 1)
 				)
@@
 		(dnp no)
 		(fields_autoplaced yes)
-		(property "Reference" "#PWR0132"
+		(property "Reference" "#PWR0133"
 			(at 156.21 120.65 0)
 			(effects
@@
 			(project "PFC & LLC"
 				(path "/97d1a1fe-d5a5-4da8-b78a-88a9132d14ad/9cd95f3e-5010-4970-88ae-b8d7b603fb03"
-					(reference "#PWR0132")
-					(unit 1)
-				)
+					(reference "#PWR0133")
+					(unit 1)
+				)

Commit message: update LLC
Parts:
- renumbered C98 to C100, C99 to C101, C100 to C102, C101 to C103, C102 to C104, C103 to C105, C104 to C106, C105 to C107, C106 to C108, C107 to C109, C108 to C110, C97 to C99, R53 to R52, R54 to R53, R55 to R54, R56 to R55, R57 to R56, R58 to R57
