File: Hardware/Source/PFC & LLC/mcu.kicad_sch (KiCad schematic)
At the start: 1 part, among them U1 STM32F107RCT6

Commit message: update FEEDBACK, AC
Parts:
- added C31: 100nF/16V, charge_battery_footprint_lib:Ceramic_Cap_0603, symbol charge_battery_sym_lib:Ceramic_Cap_SMD_100nF_16V
- added C32, C33: 20pF/50V, charge_battery_footprint_lib:Ceramic_Cap_0603, symbol charge_battery_sym_lib:Ceramic_Cap_SMD_20pF_50V
- added C34, C35, C37: 4.7uF/25V, charge_battery_footprint_lib:Ceramic_Cap_0603, symbol charge_battery_sym_lib:Ceramic_Cap_SMD_4.7uF_25V
- added C36, C38, C39, C40, C41, C42, C43, C44, C45, C46: 100nF/50V, charge_battery_footprint_lib:Ceramic_Cap_0402, symbol charge_battery_sym_lib:Ceramic_Cap_SMD_100nF_50V_0402
- added D10, D11, D12, D9: LED_0805, charge_battery_footprint_lib:LED_0805, symbol charge_battery_sym_lib:LED_0805
- added FB1: 120R, Inductor_SMD:L_0805_2012Metric, symbol Device:L_Small
- added NT2: 3V3_VBAT, NetTie:NetTie-2_SMD_Pad0.5mm, symbol Device:NetTie_2
- added NT3: GNDA_GNDPWR, NetTie:NetTie-2_SMD_Pad0.5mm, symbol Device:NetTie_2
- added R23: 10K/1%/1_10W, charge_battery_footprint_lib:Res_0603, symbol charge_battery_sym_lib:Res_10K_0603_1%
- added R24, R25, R26, R27: 1K/1%/1_10W, charge_battery_footprint_lib:Res_0603, symbol charge_battery_sym_lib:Res_1K_0603_1%
- added R28: 47/5%/1_16W, charge_battery_footprint_lib:Res_0402, symbol charge_battery_sym_lib:Res_47_0402_5%
- added SW1: RESET, charge_battery_footprint_lib:SW_SMD, symbol charge_battery_sym_lib:SW_Push
- added Y1: Crystal_25MHz_SMD-4PIN, charge_battery_footprint_lib:Crystal_SMD_4PIN_3225, symbol charge_battery_sym_lib:Crystal_25MHz_SMD-4PIN
- renumbered U1 to U5
Connections:
- net PFC_ON/OFF: now reaches U5.15 (PA1)
- net LED_TEST: now reaches U5.22 (PA6)
- net LED_TEST: now also D12.2 (A)
- net H_Gate_Driver: now reaches U5.23 (PA7)
- net LED_WAIT: now reaches U5.26 (PB0)
- net LED_WAIT: now also D9.2 (A)
- net LED_SOFT_START: now reaches U5.27 (PB1)
- net LED_SOFT_START: now also D10.2 (A)
- net LED_PROCESS: now reaches U5.28 (PB2)
- net LED_PROCESS: now also D11.2 (A)
- net L_Gate_Driver: now reaches U5.41 (PA8)
- net UART1_TX: now reaches U5.42 (PA9)
- net UART1_RX: now reaches U5.43 (PA10)
- net SWDIO: now reaches U5.46 (PA13)
- net SWCLK: now reaches U5.49 (PA14)
- net at U5.5 (PD0): now also R28.1
- net I2C_ALERT: now reaches U5.57 (PB5)
- net I2C_SCL: now reaches U5.58 (PB6)
- net I2C_SDA: now reaches U5.59 (PB7)
- net at U5.6 (PD1): now also C33.1, Y1.1
- net BOOT0: now reaches U5.60 (BOOT0)
- net NRST: now reaches U5.7 (NRST)
- net NRST: now also C31.1, R23.1, SW1.1
- net VBAT: now reaches U5.1 (VBAT)
- net VBAT: now also C37.2, C40.2, NT2.2
- net GNDA: now reaches U5.12 (VSSA)
- net GNDA: now also C41.1, NT3.2
- net VDDA: now reaches U5.13 (VDDA)
- net VDDA: now also C41.2, FB1.2
- net GNDPWR: now reaches U5.18 (VSS)
- net GNDPWR: now also U5.31 (VSS), U5.47 (VSS), U5.63 (VSS), C34.1, C35.1, C36.1, C37.1, C38.1, C39.1, C40.1, C42.1, C43.1, C44.1, C45.1, C46.1, NT3.1
- net +3V3: now reaches U5.19 (VDD)
- net +3V3: now also U5.32 (VDD), U5.48 (VDD), U5.64 (VDD), C34.2, C35.2, C36.2, C38.2, C39.2, C42.2, C43.2, C44.2, C45.2, C46.2, FB1.1, NT2.1, R23.2
- new net: C32.1, R28.2, Y1.3
- new net: D12.1 (K), R27.1
- new net: D11.1 (K), R26.1
- new net: D10.1 (K), R25.1
- new net: D9.1 (K), R24.1
- new net GNDD: C31.2, C32.2, C33.2, R24.2, R25.2, R26.2, R27.2, SW1.2, Y1.2, Y1.4
Other:
- moved on the sheet: U5A, U5B

Commit message: update lib, LLC
Parts:
- added D14: BZT52H-C3V3, charge_battery_footprint_lib:Diode_Zener_BZT52H, symbol charge_battery_sym_lib:BZT52H-C3V3
- added J2: FLASH PROGRAM, Connector_PinHeader_2.54mm:PinHeader_1x04_P2.54mm_Vertical, symbol Connector:Conn_01x04_Pin
- added J3: COMMAND LINE, Connector_PinHeader_2.54mm:PinHeader_1x03_P2.54mm_Vertical, symbol Connector:Conn_01x03_Pin
- added NT3, NT4, NT5, NT6, NT7: GNDD_GNDPWR, NetTie:NetTie-2_SMD_Pad0.5mm, symbol Device:NetTie_2
- added R27: 10K/1%/1_16W, charge_battery_footprint_lib:Res_0402, symbol charge_battery_sym_lib:Res_10K_0402_1%
- added R28, R29: 47/5%/1_16W, charge_battery_footprint_lib:Res_0402, symbol charge_battery_sym_lib:Res_47_0402_5%
- renumbered C31 to C28, C32 to C29, C33 to C30, C34 to C31, C35 to C32, C36 to C33, C37 to C34, C38 to C35, C39 to C36, C40 to C37, C41 to C38, C42 to C39, C43 to C40, C44 to C41, C45 to C42, C46 to C43, D9 to D10, D10 to D11, D11 to D12, D12 to D13, NT2 to NT8, NT3 to NT9, R23 to R21, R24 to R22, R25 to R23, R26 to R24, R27 to R25, R28 to R26, U5 to U3
Connections:
- net +3V3: now also J2.4 (Pin_4)
- net BOOT0: now also R27.2
- net GNDD: now also D14.2 (A), J3.3 (Pin_3), NT3.1, NT4.1, NT5.1, NT6.1, NT7.1, R27.1
- net GNDPWR: now also J2.1 (Pin_1), NT3.2, NT4.2, NT5.2, NT6.2, NT7.2
- net SWCLK: now also R29.2
- net SWDIO: now also R28.2
- net UART1_RX: now also J3.2 (Pin_2)
- net UART1_TX: now also J3.1 (Pin_1)
- net DETECT_BATTERY: now reaches U3.14 (PA0)
- net DETECT_BATTERY: now also D14.1 (K)
- new net: J2.2 (Pin_2), R29.1
- new net: J2.3 (Pin_3), R28.1
- no-connect marks 0 -> 34
Other:
- moved on the sheet: C28, C29, C30, C32, C33, C34, C36, C37, C39, C40, C41, C42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

Commit message: update lib, LLC
Parts:
- removed R22, R23, R24, R25: 1K/1%/1_10W, charge_battery_footprint_lib:Res_0603, symbol charge_battery_sym_lib:Res_1K_0603_1%
- added D15: BZT52H-C3V3, charge_battery_footprint_lib:Diode_Zener_BZT52H, symbol charge_battery_sym_lib:BZT52H-C3V3
- added R27, R28, R29, R30: 1K/1%/1_10W, charge_battery_footprint_lib:Res_0603, symbol charge_battery_sym_lib:Res_1K_0603_1%
- added R33, R34: 10K/1%/1_10W, charge_battery_footprint_lib:Res_0603, symbol charge_battery_sym_lib:Res_10K_0603_1%
- renumbered R21 to R24, R28 to R25, R29 to R26, R26 to R31, R27 to R32
Connections:
- net +3V3: now also R33.2, R34.2
- net GNDD: now also D15.2 (A), R27.2, R28.2, R29.2, R30.2
- net PFC_ON/OFF: now also U3.16 (PA2); no longer U3.15 (PA1)
- net UART1_RX: now also R33.1
- net UART1_TX: now also R34.1
- net at D13.1 (K): now also R30.1
- net at D12.1 (K): now also R29.1
- net at D11.1 (K): now also R28.1
- net at D10.1 (K): now also R27.1
- net CONTROL_CHARGER: now reaches U3.17 (PA3)
- new net PFC_OPERATION: D15.1 (K), U3.15 (PA1)
- no-connect marks 34 -> 32
Other:
- moved on the sheet: C28, C29, C30, D11, D12, D13, D14, J2, J3, NT3, NT4, NT5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

Commit message: update LLC
Parts:
- renumbered C28 to C30, C29 to C31, C30 to C32, C31 to C33, C32 to C34, C33 to C35, C34 to C36, C35 to C37, C36 to C38, C37 to C39, C38 to C40, C39 to C41, C40 to C42, C41 to C43, C42 to C44, C43 to C45, R24 to R23, R25 to R24, R26 to R25, R27 to R26, R28 to R27, R29 to R28, R30 to R29, R31 to R30, R32 to R31, R33 to R32, R34 to R33

Commit message: update lib
Changed lines of the file:
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@@
 (kicad_sch
-	(version 20231120)
+	(version 20250114)
 	(generator "eeschema")
-	(generator_version "8.0")
+	(generator_version "9.0")
 	(paper "A3")
 	(title_block
