File: Hardware/Source/BATTERY_CONVERTER/charge_pump.kicad_sch (KiCad schematic)
At the start: 3 parts, among them U6 ICL7662CBA

Commit message: update bat
Parts:
- renumbered C33 to C32, C34 to C33
Changed lines of the file:
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@@
 		(on_board yes)
 		(dnp no)
-		(property "Reference" "C33"
+		(property "Reference" "C32"
 			(at 115.316 93.218 90)
 			(effects
@@
 			(project "BATTERY_CONVERTER"
 				(path "/518c170c-c465-4532-a1cc-dfde0d4d70b3/82a5c018-41ff-42c0-b129-fd1671b16d38"
-					(reference "C33")
+					(reference "C32")
 					(unit 1)
 				)
@@
 		(on_board yes)
 		(dnp no)
-		(property "Reference" "C34"
+		(property "Reference" "C33"
 			(at 171.196 95.25 90)
 			(effects
@@
 			(project "BATTERY_CONVERTER"
 				(path "/518c170c-c465-4532-a1cc-dfde0d4d70b3/82a5c018-41ff-42c0-b129-fd1671b16d38"
-					(reference "C34")
+					(reference "C33")
 					(unit 1)
 				)
