File: Hardware/Source/BATTERY_CONVERTER/ldo_3v3.kicad_sch (KiCad schematic)
At the start: 10 parts, among them U3 LD1117S33CTR_SOT223, U4 LD1117S33CTR_SOT223

Commit message: update bat
Parts:
- renumbered C21 to C20, C22 to C21, C23 to C22, C24 to C23, C25 to C24, C26 to C25, C27 to C26, C28 to C27
Changed lines of the file:
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@@
 		(on_board yes)
 		(dnp no)
-		(property "Reference" "C22"
+		(property "Reference" "C21"
 			(at 117.094 117.602 90)
 			(effects
@@
 			(project "BATTERY_CONVERTER"
 				(path "/518c170c-c465-4532-a1cc-dfde0d4d70b3/b067cfa2-b17d-4705-b89a-fb5960338b81"
-					(reference "C22")
+					(reference "C21")
 					(unit 1)
 				)
@@
 		(on_board yes)
 		(dnp no)
-		(property "Reference" "C21"
+		(property "Reference" "C20"
 			(at 117.094 79.502 90)
 			(effects
@@
 			(project "BATTERY_CONVERTER"
 				(path "/518c170c-c465-4532-a1cc-dfde0d4d70b3/b067cfa2-b17d-4705-b89a-fb5960338b81"
-					(reference "C21")
+					(reference "C20")
 					(unit 1)
 				)
@@
 		(on_board yes)
 		(dnp no)
-		(property "Reference" "C23"
+		(property "Reference" "C22"
 			(at 130.048 79.248 90)
 			(effects
@@
 			(project "BATTERY_CONVERTER"
 				(path "/518c170c-c465-4532-a1cc-dfde0d4d70b3/b067cfa2-b17d-4705-b89a-fb5960338b81"
-					(reference "C23")
+					(reference "C22")
 					(unit 1)
 				)
@@
 		(on_board yes)
 		(dnp no)
-		(property "Reference" "C26"
+		(property "Reference" "C25"
 			(at 167.894 117.602 90)
 			(effects
@@
 			(project "BATTERY_CONVERTER"
 				(path "/518c170c-c465-4532-a1cc-dfde0d4d70b3/b067cfa2-b17d-4705-b89a-fb5960338b81"
-					(reference "C26")
+					(reference "C25")
 					(unit 1)
 				)
@@
 		(on_board yes)
 		(dnp no)
-		(property "Reference" "C27"
+		(property "Reference" "C26"
 			(at 180.848 80.518 90)
 			(effects
@@
 			(project "BATTERY_CONVERTER"
 				(path "/518c170c-c465-4532-a1cc-dfde0d4d70b3/b067cfa2-b17d-4705-b89a-fb5960338b81"
-					(reference "C27")
+					(reference "C26")
 					(unit 1)
 				)
@@
 		(on_board yes)
 		(dnp no)
-		(property "Reference" "C25"
+		(property "Reference" "C24"
 			(at 166.624 80.772 90)
 			(effects
@@
 			(project "BATTERY_CONVERTER"
 				(path "/518c170c-c465-4532-a1cc-dfde0d4d70b3/b067cfa2-b17d-4705-b89a-fb5960338b81"
-					(reference "C25")
+					(reference "C24")
 					(unit 1)
 				)
@@
 		(on_board yes)
 		(dnp no)
-		(property "Reference" "C28"
+		(property "Reference" "C27"
 			(at 180.848 117.348 90)
 			(effects
@@
 			(project "BATTERY_CONVERTER"
 				(path "/518c170c-c465-4532-a1cc-dfde0d4d70b3/b067cfa2-b17d-4705-b89a-fb5960338b81"
-					(reference "C28")
+					(reference "C27")
 					(unit 1)
 				)
@@
 		(on_board yes)
 		(dnp no)
-		(property "Reference" "C24"
+		(property "Reference" "C23"
 			(at 130.048 117.348 90)
 			(effects
@@
 			(project "BATTERY_CONVERTER"
 				(path "/518c170c-c465-4532-a1cc-dfde0d4d70b3/b067cfa2-b17d-4705-b89a-fb5960338b81"
-					(reference "C24")
-					(unit 1)
-				)
+					(reference "C23")
+					(unit 1)
+				)
