File: Hardware/Source/BATTERY_CONVERTER/Liner_Voltage_9V.kicad_sch (KiCad schematic)
At the start: 5 parts, among them U5 L7809CV

Commit message: update bat
Parts:
- renumbered C29 to C28, C30 to C29, C31 to C30, C32 to C31
Changed lines of the file:
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@@
 		(on_board yes)
 		(dnp no)
-		(property "Reference" "C32"
+		(property "Reference" "C31"
 			(at 181.356 83.312 90)
 			(effects
@@
 			(project "BATTERY_CONVERTER"
 				(path "/518c170c-c465-4532-a1cc-dfde0d4d70b3/615e3a1f-00ea-4f8b-87b9-21b5b209977b"
-					(reference "C32")
+					(reference "C31")
 					(unit 1)
 				)
@@
 		(on_board yes)
 		(dnp no)
-		(property "Reference" "C31"
+		(property "Reference" "C30"
 			(at 168.402 83.058 90)
 			(effects
@@
 			(project "BATTERY_CONVERTER"
 				(path "/518c170c-c465-4532-a1cc-dfde0d4d70b3/615e3a1f-00ea-4f8b-87b9-21b5b209977b"
-					(reference "C31")
+					(reference "C30")
 					(unit 1)
 				)
@@
 		(on_board yes)
 		(dnp no)
-		(property "Reference" "C29"
+		(property "Reference" "C28"
 			(at 112.268 83.566 90)
 			(effects
@@
 			(project "BATTERY_CONVERTER"
 				(path "/518c170c-c465-4532-a1cc-dfde0d4d70b3/615e3a1f-00ea-4f8b-87b9-21b5b209977b"
-					(reference "C29")
+					(reference "C28")
 					(unit 1)
 				)
@@
 		(on_board yes)
 		(dnp no)
-		(property "Reference" "C30"
+		(property "Reference" "C29"
 			(at 124.968 83.058 90)
 			(effects
@@
 			(project "BATTERY_CONVERTER"
 				(path "/518c170c-c465-4532-a1cc-dfde0d4d70b3/615e3a1f-00ea-4f8b-87b9-21b5b209977b"
-					(reference "C30")
-					(unit 1)
-				)
+					(reference "C29")
+					(unit 1)
+				)

Commit message: Update Battery Converter Project
Parts:
- U5: Supply name TME -> tme
Changed lines of the file:
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@@
 			)
 		)
-		(property "Supply name" "TME"
+		(property "Supply name" "tme"
 			(at 150.876 90.932 0)
 			(effects
