File: Hardware/Source/BATTERY_CONVERTER/dc_dc_converter_5v.kicad_sch (KiCad schematic)
At the start: 18 parts, among them U2 TPS54331DR

Commit message: update bat
Parts:
- renumbered C13 to C12, C14 to C13, C15 to C14, C16 to C15, C17 to C16, C18 to C17, C19 to C18, C20 to C19
Changed lines of the file:
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@@
 		(on_board yes)
 		(dnp no)
-		(property "Reference" "C13"
+		(property "Reference" "C12"
 			(at 55.626 60.198 90)
 			(effects
@@
 			(project "BATTERY_CONVERTER"
 				(path "/518c170c-c465-4532-a1cc-dfde0d4d70b3/9a5087fa-0efc-4e35-a4c0-e5c486dda67f"
-					(reference "C13")
+					(reference "C12")
 					(unit 1)
 				)
@@
 		(on_board yes)
 		(dnp no)
-		(property "Reference" "C19"
+		(property "Reference" "C18"
 			(at 196.85 72.39 90)
 			(effects
@@
 			(project "BATTERY_CONVERTER"
 				(path "/518c170c-c465-4532-a1cc-dfde0d4d70b3/9a5087fa-0efc-4e35-a4c0-e5c486dda67f"
-					(reference "C19")
+					(reference "C18")
 					(unit 1)
 				)
@@
 		(on_board yes)
 		(dnp no)
-		(property "Reference" "C18"
+		(property "Reference" "C17"
 			(at 161.29 55.88 0)
 			(effects
@@
 			(project "BATTERY_CONVERTER"
 				(path "/518c170c-c465-4532-a1cc-dfde0d4d70b3/9a5087fa-0efc-4e35-a4c0-e5c486dda67f"
-					(reference "C18")
+					(reference "C17")
 					(unit 1)
 				)
@@
 		(on_board yes)
 		(dnp no)
-		(property "Reference" "C14"
+		(property "Reference" "C13"
 			(at 73.152 59.69 90)
 			(effects
@@
 			(project ""
 				(path "/518c170c-c465-4532-a1cc-dfde0d4d70b3/9a5087fa-0efc-4e35-a4c0-e5c486dda67f"
-					(reference "C14")
+					(reference "C13")
 					(unit 1)
 				)
@@
 		(on_board yes)
 		(dnp no)
-		(property "Reference" "C16"
+		(property "Reference" "C15"
 			(at 125.222 84.582 90)
 			(effects
@@
 			(project "BATTERY_CONVERTER"
 				(path "/518c170c-c465-4532-a1cc-dfde0d4d70b3/9a5087fa-0efc-4e35-a4c0-e5c486dda67f"
-					(reference "C16")
+					(reference "C15")
 					(unit 1)
 				)
@@
 		(on_board yes)
 		(dnp no)
-		(property "Reference" "C20"
+		(property "Reference" "C19"
 			(at 214.376 72.39 90)
 			(effects
@@
 			(project "BATTERY_CONVERTER"
 				(path "/518c170c-c465-4532-a1cc-dfde0d4d70b3/9a5087fa-0efc-4e35-a4c0-e5c486dda67f"
-					(reference "C20")
+					(reference "C19")
 					(unit 1)
 				)
@@
 		(on_board yes)
 		(dnp no)
-		(property "Reference" "C15"
+		(property "Reference" "C14"
 			(at 106.172 77.47 90)
 			(effects
@@
 			(project "BATTERY_CONVERTER"
 				(path "/518c170c-c465-4532-a1cc-dfde0d4d70b3/9a5087fa-0efc-4e35-a4c0-e5c486dda67f"
-					(reference "C15")
+					(reference "C14")
 					(unit 1)
 				)
@@
 		(on_board yes)
 		(dnp no)
-		(property "Reference" "C17"
+		(property "Reference" "C16"
 			(at 141.732 81.534 90)
 			(effects
@@
 			(project "BATTERY_CONVERTER"
 				(path "/518c170c-c465-4532-a1cc-dfde0d4d70b3/9a5087fa-0efc-4e35-a4c0-e5c486dda67f"
-					(reference "C17")
-					(unit 1)
-				)
+					(reference "C16")
+					(unit 1)
+				)

Commit message: Update Battery Converter Project
Parts:
- L2: Supply name (none) -> tme
Changed lines of the file:
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@@
 			)
 		)
-		(property "Description" " 4.5V to 28V Input, 3A, Synchronous Step-Down Converter with Eco-mode(tm)"
+		(property "Description" "4.5V to 28V Input, 3A, Synchronous Step-Down Converter with Eco-mode(tm)"
 			(at 141.732 94.742 0)
 			(effects
@@
 			(at 171.45 66.04 0)
 			(effects
+				(font
+					(size 1.27 1.27)
+				)
+				(hide yes)
+			)
+		)
+		(property "Supply name" "tme"
+			(at 171.45 66.04 0)
+			(effects
