File: Hardware/Source/BATTERY_CONVERTER/dc_dc_converter_battery.kicad_sch (KiCad schematic)
At the start: 21 parts, among them U1 LM5576MHX/NOPB

Commit message: update bat
Parts:
- removed C4: 2.2uF/100V, Capacitor_SMD:CP_Elec_6.3x5.4, symbol charge_battery_sym_lib:Cap_Polarized_SMD_2.2uF_100V
- renumbered C11 to C10, C12 to C11, C5 to C4, C6 to C5, C7 to C6, C8 to C7, C9 to C8, C10 to C9
Changed lines of the file:
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@@
 	)
 	(junction
-		(at 67.31 67.31)
-		(diameter 0)
-		(color 0 0 0 0)
-	)
-	(junction
 		(at 162.56 87.63)
 		(diameter 0)
@@
 	)
 	(junction
-		(at 83.82 58.42)
-		(diameter 0)
-		(color 0 0 0 0)
-	)
-	(junction
 		(at 248.92 72.39)
 		(diameter 0)
@@
 	(wire
 		(pts
-			(xy 67.31 67.31) (xy 67.31 68.58)
-		)
-		(stroke
-			(width 0)
-			(type default)
-		)
-	)
-	(wire
-		(pts
 			(xy 116.84 114.3) (xy 125.73 114.3)
 		)
@@
 	(wire
 		(pts
-			(xy 83.82 58.42) (xy 83.82 60.96)
-		)
-		(stroke
-			(width 0)
-			(type default)
-		)
-	)
-	(wire
-		(pts
 			(xy 167.64 77.47) (xy 167.64 76.2)
 		)
@@
 	(wire
 		(pts
-			(xy 83.82 58.42) (xy 129.54 58.42)
+			(xy 67.31 58.42) (xy 129.54 58.42)
 		)
 		(stroke
@@
 	(wire
 		(pts
-			(xy 83.82 66.04) (xy 83.82 67.31)
-		)
-		(stroke
-			(width 0)
-			(type default)
-		)
-	)
-	(wire
-		(pts
 			(xy 111.76 69.85) (xy 129.54 69.85)
 		)
@@
 	(wire
 		(pts
-			(xy 67.31 66.04) (xy 67.31 67.31)
+			(xy 67.31 66.04) (xy 67.31 68.58)
 		)
 		(stroke
@@
 	(wire
 		(pts
-			(xy 83.82 58.42) (xy 67.31 58.42)
-		)
-		(stroke
-			(width 0)
-			(type default)
-		)
-	)
-	(wire
-		(pts
 			(xy 157.48 54.61) (xy 157.48 52.07)
 		)
@@
 	(wire
 		(pts
-			(xy 83.82 67.31) (xy 67.31 67.31)
-		)
-		(stroke
-			(width 0)
-			(type default)
-		)
-	)
-	(wire
-		(pts
 			(xy 54.61 104.14) (xy 54.61 100.33)
 		)
@@
 		(dnp no)
 		(fields_autoplaced yes)
-		(property "Reference" "C11"
+		(property "Reference" "C10"
 			(at 219.71 75.7681 90)
 			(effects
@@
 			(project "BATTERY_CONVERTER"
 				(path "/518c170c-c465-4532-a1cc-dfde0d4d70b3/ef158934-4c2e-46c0-b577-2a60bdf42815"
-					(reference "C11")
+					(reference "C10")
 					(unit 1)
 				)
@@
 		(dnp no)
 		(fields_autoplaced yes)
-		(property "Reference" "C5"
+		(property "Reference" "C4"
 			(at 99.06 104.1399 90)
 			(effects
@@
 			(project "BATTERY_CONVERTER"
 				(path "/518c170c-c465-4532-a1cc-dfde0d4d70b3/ef158934-4c2e-46c0-b577-2a60bdf42815"
-					(reference "C5")
+					(reference "C4")
 					(unit 1)
 				)
@@
 	)
 	(symbol
-		(lib_id "charge_battery_sym_lib:Cap_Polarized_SMD_2.2uF_100V")
-		(at 83.82 60.96 270)
-		(unit 1)
-		(exclude_from_sim no)
-		(in_bom yes)
-		(on_board yes)
-		(dnp no)
-		(fields_autoplaced yes)
-		(property "Reference" "C4"
-			(at 86.36 61.7981 90)
-			(effects
-				(font
-					(size 1.27 1.27)
-				)
-				(justify left)
-			)
-		)
-		(property "Value" "2.2uF/100V"
-			(at 86.36 64.3381 90)
-			(effects
-				(font
-					(size 1.27 1.27)
-				)
-				(justify left)
-			)
-		)
-		(property "Footprint" "Capacitor_SMD:CP_Elec_6.3x5.4"
-			(at 96.52 64.262 0)
-			(effects
-				(font
-					(size 1.27 1.27)
-				)
-				(hide yes)
-			)
-		)
-		(property "Datasheet" ""
-			(at 96.266 61.722 0)
-			(effects
-				(font
-					(size 1.27 1.27)
-				)
-				(hide yes)
-			)
-		)
-		(property "Description" "Polarized capacitor 2.2uF 100V, 20%"
-			(at 96.012 60.198 0)
-			(effects
-				(font
-					(size 1.27 1.27)
-				)
-				(hide yes)
-			)
-		)
-		(property "Supply name" "Thegioiic"
-			(at 96.266 62.992 0)
-			(effects
-				(font
-					(size 1.27 1.27)
-				)
-				(hide yes)
-			)
-		)
-		(property "Supply part number" "Tụ Nhôm SMD 2.2uF 100V 6.3x5.4mm"
-			(at 96.266 62.23 0)
-			(effects
-				(font
-					(size 1.27 1.27)
-				)
-				(hide yes)
-			)
-		)
-		(property "Supply URL" "https://www.thegioiic.com/tu-nhom-smd-2-2uf-100v-6-3x5-4mm"
-			(at 96.52 62.992 0)
-			(effects
-				(font
-					(size 1.27 1.27)
-				)
-				(hide yes)
-			)
-		)
-		(pin "2"
-		)
-		(pin "1"
-		)
-		(instances
-			(project ""
-				(path "/518c170c-c465-4532-a1cc-dfde0d4d70b3/ef158934-4c2e-46c0-b577-2a60bdf42815"
-					(reference "C4")
-					(unit 1)
-				)
-			)
-		)
-	)
-	(symbol
 		(lib_id "charge_battery_sym_lib:Ceramic_Cap_SMD_10nF_100V")
 		(at 116.84 107.95 90)
@@
 		(dnp no)
 		(fields_autoplaced yes)
-		(property "Reference" "C7"
+		(property "Reference" "C6"
 			(at 120.65 102.8699 90)
 			(effects
@@
 			(project "BATTERY_CONVERTER"
 				(path "/518c170c-c465-4532-a1cc-dfde0d4d70b3/ef158934-4c2e-46c0-b577-2a60bdf42815"
-					(reference "C7")
+					(reference "C6")
 					(unit 1)
 				)
@@
 		(dnp no)
 		(fields_autoplaced yes)
-		(property "Reference" "C6"
+		(property "Reference" "C5"
 			(at 115.57 73.6599 90)
 			(effects
@@
 			(project ""
 				(path "/518c170c-c465-4532-a1cc-dfde0d4d70b3/ef158934-4c2e-46c0-b577-2a60bdf42815"
-					(reference "C6")
+					(reference "C5")
 					(unit 1)
 				)
@@
 		(dnp no)
 		(fields_autoplaced yes)
-		(property "Reference" "C9"
+		(property "Reference" "C8"
 			(at 173.99 66.04 0)
 			(effects
@@
 			(project ""
 				(path "/518c170c-c465-4532-a1cc-dfde0d4d70b3/ef158934-4c2e-46c0-b577-2a60bdf42815"
-					(reference "C9")
+					(reference "C8")
 					(unit 1)
 				)
@@
 		(dnp no)
 		(fields_autoplaced yes)
-		(property "Reference" "C12"
+		(property "Reference" "C11"
 			(at 237.49 76.1999 90)
 			(effects
@@
 			(project "BATTERY_CONVERTER"
 				(path "/518c170c-c465-4532-a1cc-dfde0d4d70b3/ef158934-4c2e-46c0-b577-2a60bdf42815"
-					(reference "C12")
+					(reference "C11")
 					(unit 1)
 				)
@@
 		(dnp no)
 		(fields_autoplaced yes)
-		(property "Reference" "C8"
+		(property "Reference" "C7"
 			(at 166.37 55.8799 90)
 			(effects
@@
 			(project ""
 				(path "/518c170c-c465-4532-a1cc-dfde0d4d70b3/ef158934-4c2e-46c0-b577-2a60bdf42815"
-					(reference "C8")
+					(reference "C7")
 					(unit 1)
 				)
@@
 		(dnp no)
 		(fields_autoplaced yes)
-		(property "Reference" "C10"
+		(property "Reference" "C9"
 			(at 195.58 76.1999 90)
 			(effects
@@
 			(project ""
 				(path "/518c170c-c465-4532-a1cc-dfde0d4d70b3/ef158934-4c2e-46c0-b577-2a60bdf42815"
-					(reference "C10")
+					(reference "C9")
 					(unit 1)
 				)

Commit message: Update Battery Converter Project
Parts:
- C10, R3: Supply name (none) -> Thegioiic
- L1: Supply URL (none) -> https://www.thegioiic.com/cuon-cam-dan-smd-cdrh127-1280-680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; Supply name (none) -> Thegioiic
- U1: Supply name TME -> tme
Changed lines of the file:
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@@
+			)
+		)
+		(property "Supply name" "Thegioiic"
+			(at 220.98 77.47 0)
+			(effects
+				(font
+					(size 1.27 1.27)
+				)
+				(hide yes)
 			)
 		)
@@
 			)
 		)
-		(property "Supply name" "TME"
+		(property "Supply name" "tme"
 			(at 108.204 122.174 0)
 			(effects
@@
 			)
 		)
+		(property "Supply URL" "https://www.thegioiic.com/cuon-cam-dan-smd-cdrh127-1280-680-68uh-3-2a"
+			(at 196.85 72.39 0)
+			(effects
+				(font
+					(size 1.27 1.27)
+				)
+				(hide yes)
+			)
+		)
+		(property "Supply name" "Thegioiic"
+			(at 196.85 72.39 0)
+			(effects
+				(font
+					(size 1.27 1.27)
+				)
+				(hide yes)
+			)
+		)
 		(pin "2"
 		)
@@
 			(effects
 				(font
+					(size 1.27 1.27)
+				)
+				(hide yes)
+			)
+		)
+		(property "Supply name" "Thegioiic"
+			(at 191.77 91.44 0)
+			(effects
+				(font
