File: Hardware/Test Board/Test_Gate_Driver/Test_Gate_Driver.kicad_sch (KiCad schematic)
At the start: 19 parts, among them J1 Conn_01x02_Socket, J2 Conn_01x03_Socket, J3 Conn_01x02_Socket, Q1 IPP60R125CP, Q2 IPP60R125CP, U1 IR2110STRPBF

Commit message: update
Parts:
- removed J1: Conn_01x02_Socket, Connector_PinHeader_2.54mm:PinHeader_1x02_P2.54mm_Vertical, symbol Connector:Conn_01x02_Socket
- removed Q1, Q2: IPP60R125CP, charge_battery_footprint_lib:TO-220-3, symbol charge_battery_sym_lib:IPP60R125CP
- removed R2: 10K/1%/1_10W, charge_battery_footprint_lib:Res_0603, symbol charge_battery_sym_lib:Res_10K_0603_1%
- added R5: 10K/1%/1_4W, charge_battery_footprint_lib:Res_1206, symbol charge_battery_sym_lib:Res_10K_1206_1%
Connections:
- net at D3.1 (A), R1.2: now also R5.2
