File: Hardware/Test Board/Test_Gate_Driver/Test_Gate_Driver.kicad_pcb (KiCad board)
At the start: 2 copper layers, 42 x 30 mm, 19 parts, among them J1 Conn_01x04_Pin, J3 Conn_01x02_Socket, U1 IR2110STRPBF

Commit message: update test gate driver
Parts:
- moved J3 85.1 mm to (106.3, 101.0), turned to -90 degrees
- moved J1 81.2 mm to (98.0, 88.8), turned to 180 degrees
- moved U1 51.8 mm to (108.1, 85.2)
- moved TP1 49.6 mm to (135.8, 97.1)
- moved R1 45.8 mm to (114.1, 92.3), turned to 0 degrees
- moved C1 44.4 mm to (104.5, 96.4)
- moved R3 41.8 mm to (114.1, 77.4), turned to 0 degrees
- moved TP2 41.5 mm to (135.8, 92.3)
- moved C2 39.9 mm to (102.6, 91.3), turned to 0 degrees
- moved D1 38.5 mm to (118.8, 84.9), turned to -90 degrees
- moved D3 37.7 mm to (115.1, 95.5), turned to 0 degrees
- moved R5 35.4 mm to (121.9, 92.3)
- moved R2 34.1 mm to (121.7, 75.9), turned to -90 degrees
- moved C3 32.8 mm to (128.4, 86.6), turned to 90 degrees
- moved D2 29.8 mm to (115.1, 74.2), turned to 0 degrees
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Routing:
- net GND: track 0.00 -> 119.1 mm
- net +12V: track 0.00 -> 54.4 mm, vias 0 -> 2
- net VS: track 0.00 -> 45.1 mm
- net Net-(D3-A): track 0.00 -> 27.1 mm
- net Net-(D2-A): track 0.00 -> 23.4 mm
- net VB: track 0.00 -> 16.4 mm
- net Net-(D2-K): track 0.00 -> 6.66 mm
- net Net-(J1-Pin_4): track 0.00 -> 6.24 mm
- net +3.3V: track 0.00 -> 6.09 mm
- net Net-(D3-K): track 0.00 -> 6.02 mm
- net Net-(J1-Pin_3): track 0.00 -> 5.70 mm
- net Net-(J1-Pin_2): track 0.00 -> 5.57 mm
- added copper zone on B.Cu, net +12V
- added copper zone on B.Cu, net Net-(D2-K)
- added copper zone on B.Cu, net Net-(D3-K)
Other:
- board size 42 x 30 mm -> 47.7 x 33.4 mm
- rule pad_to_mask_clearance: 0 -> 0.0508
